File: hardware/calcumaker-display/display.kicad_sch (KiCad schematic)
At the start: 19 parts, among them U1 TM1640, U2 TM1640, U3 TM1640

Commit message: Add 5V display rail: EN-gated boost + 74HCT125 level shifter
Display chosen to run at 5V (TM1640 is 5V-nominal; VIH 3.5V > the STM32's 3.3V).
Rather than upsizing the 3V3 buck-boost, split the rails:

- Keep the ULP TPS63900 at 3V3 for the MCU only (always-on, low-Iq for sleep).
- Add an EN-gated 5V boost for the display LED load (off in sleep via DISP_PWR_EN).
- Add a 74HCT125 quad buffer @5V to translate CLK + DIN1/2/3 from 3V3 to 5V.
- Interconnect now carries +5V + 5V-logic; main-board "display_if" sheet holds
  the boost + shifter + J3. Display board regenerated for the 5V note.

Boost (+inductor) and 74HCT125 LCSC parts are being picked by availability.
Updated both manifests, DESIGN.md (power tree/sheet plan/parts), README, PARTS.md.

Co-Authored-By: Claude Opus 4.8 (1M context) <noreply@anthropic.com>
Changed lines of the file:
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@@
 		(instances
 			(project "calcumaker-display"
-				(path "/ca1c0000-0000-4000-8000-0000000d1501/90740d87-7211-4fa0-b59b-73c565908d04"
+				(path "/ca1c0000-0000-4000-8000-0000000d1501/bff2c2c9-e03f-4398-9f4c-6cb350699cef"
 					(reference "U1")
 					(unit 1)
@@
 		(instances
 			(project "calcumaker-display"
-				(path "/ca1c0000-0000-4000-8000-0000000d1501/90740d87-7211-4fa0-b59b-73c565908d04"
+				(path "/ca1c0000-0000-4000-8000-0000000d1501/bff2c2c9-e03f-4398-9f4c-6cb350699cef"
 					(reference "U2")
 					(unit 1)
@@
 		(instances
 			(project "calcumaker-display"
-				(path "/ca1c0000-0000-4000-8000-0000000d1501/90740d87-7211-4fa0-b59b-73c565908d04"
+				(path "/ca1c0000-0000-4000-8000-0000000d1501/bff2c2c9-e03f-4398-9f4c-6cb350699cef"
 					(reference "U3")
 					(unit 1)
@@
 		(instances
 			(project "calcumaker-display"
-				(path "/ca1c0000-0000-4000-8000-0000000d1501/90740d87-7211-4fa0-b59b-73c565908d04"
+				(path "/ca1c0000-0000-4000-8000-0000000d1501/bff2c2c9-e03f-4398-9f4c-6cb350699cef"
 					(reference "DS1")
 					(unit 1)
@@
 		(instances
 			(project "calcumaker-display"
-				(path "/ca1c0000-0000-4000-8000-0000000d1501/90740d87-7211-4fa0-b59b-73c565908d04"
+				(path "/ca1c0000-0000-4000-8000-0000000d1501/bff2c2c9-e03f-4398-9f4c-6cb350699cef"
 					(reference "DS2")
 					(unit 1)
@@
 		(instances
 			(project "calcumaker-display"
-				(path "/ca1c0000-0000-4000-8000-0000000d1501/90740d87-7211-4fa0-b59b-73c565908d04"
+				(path "/ca1c0000-0000-4000-8000-0000000d1501/bff2c2c9-e03f-4398-9f4c-6cb350699cef"
 					(reference "DS3")
 					(unit 1)
@@
 		(instances
 			(project "calcumaker-display"
-				(path "/ca1c0000-0000-4000-8000-0000000d1501/90740d87-7211-4fa0-b59b-73c565908d04"
+				(path "/ca1c0000-0000-4000-8000-0000000d1501/bff2c2c9-e03f-4398-9f4c-6cb350699cef"
 					(reference "DS4")
 					(unit 1)
@@
 		(instances
 			(project "calcumaker-display"
-				(path "/ca1c0000-0000-4000-8000-0000000d1501/90740d87-7211-4fa0-b59b-73c565908d04"
+				(path "/ca1c0000-0000-4000-8000-0000000d1501/bff2c2c9-e03f-4398-9f4c-6cb350699cef"
 					(reference "DS5")
 					(unit 1)
@@
 		(instances
 			(project "calcumaker-display"
-				(path "/ca1c0000-0000-4000-8000-0000000d1501/90740d87-7211-4fa0-b59b-73c565908d04"
+				(path "/ca1c0000-0000-4000-8000-0000000d1501/bff2c2c9-e03f-4398-9f4c-6cb350699cef"
 					(reference "DS6")
 					(unit 1)
@@
 		(instances
 			(project "calcumaker-display"
-				(path "/ca1c0000-0000-4000-8000-0000000d1501/90740d87-7211-4fa0-b59b-73c565908d04"
+				(path "/ca1c0000-0000-4000-8000-0000000d1501/bff2c2c9-e03f-4398-9f4c-6cb350699cef"
 					(reference "DS7")
 					(unit 1)
@@
 		(instances
 			(project "calcumaker-display"
-				(path "/ca1c0000-0000-4000-8000-0000000d1501/90740d87-7211-4fa0-b59b-73c565908d04"
+				(path "/ca1c0000-0000-4000-8000-0000000d1501/bff2c2c9-e03f-4398-9f4c-6cb350699cef"
 					(reference "DS8")
 					(unit 1)
@@
 		(instances
 			(project "calcumaker-display"
-				(path "/ca1c0000-0000-4000-8000-0000000d1501/90740d87-7211-4fa0-b59b-73c565908d04"
+				(path "/ca1c0000-0000-4000-8000-0000000d1501/bff2c2c9-e03f-4398-9f4c-6cb350699cef"
 					(reference "DS9")
 					(unit 1)
@@
 		(instances
 			(project "calcumaker-display"
-				(path "/ca1c0000-0000-4000-8000-0000000d1501/90740d87-7211-4fa0-b59b-73c565908d04"
+				(path "/ca1c0000-0000-4000-8000-0000000d1501/bff2c2c9-e03f-4398-9f4c-6cb350699cef"
 					(reference "DS10")
 					(unit 1)
@@
 		(instances
 			(project "calcumaker-display"
-				(path "/ca1c0000-0000-4000-8000-0000000d1501/90740d87-7211-4fa0-b59b-73c565908d04"
+				(path "/ca1c0000-0000-4000-8000-0000000d1501/bff2c2c9-e03f-4398-9f4c-6cb350699cef"
 					(reference "DS11")
 					(unit 1)
@@
 		(instances
 			(project "calcumaker-display"
-				(path "/ca1c0000-0000-4000-8000-0000000d1501/90740d87-7211-4fa0-b59b-73c565908d04"
+				(path "/ca1c0000-0000-4000-8000-0000000d1501/bff2c2c9-e03f-4398-9f4c-6cb350699cef"
 					(reference "DS12")
 					(unit 1)
@@
 		(instances
 			(project "calcumaker-display"
-				(path "/ca1c0000-0000-4000-8000-0000000d1501/90740d87-7211-4fa0-b59b-73c565908d04"
+				(path "/ca1c0000-0000-4000-8000-0000000d1501/bff2c2c9-e03f-4398-9f4c-6cb350699cef"
 					(reference "C1")
 					(unit 1)
@@
 		(instances
 			(project "calcumaker-display"
-				(path "/ca1c0000-0000-4000-8000-0000000d1501/90740d87-7211-4fa0-b59b-73c565908d04"
+				(path "/ca1c0000-0000-4000-8000-0000000d1501/bff2c2c9-e03f-4398-9f4c-6cb350699cef"
 					(reference "C2")
 					(unit 1)
@@
 		(instances
 			(project "calcumaker-display"
-				(path "/ca1c0000-0000-4000-8000-0000000d1501/90740d87-7211-4fa0-b59b-73c565908d04"
+				(path "/ca1c0000-0000-4000-8000-0000000d1501/bff2c2c9-e03f-4398-9f4c-6cb350699cef"
 					(reference "C3")
 					(unit 1)
@@
 		(instances
 			(project "calcumaker-display"
-				(path "/ca1c0000-0000-4000-8000-0000000d1501/90740d87-7211-4fa0-b59b-73c565908d04"
+				(path "/ca1c0000-0000-4000-8000-0000000d1501/bff2c2c9-e03f-4398-9f4c-6cb350699cef"
 					(reference "C4")
 					(unit 1)
@@
 		)
 	)
-	(text "Calcumaker 16 display — 7-seg RPN stack. 3 rows x 16 digits (top row U3/DS9-12 optional => 2- or 3-row build). PER ROW: 1x TM1640 (C5337152) drives 4x FJ5161AH 0.56\" 4-digit common-cathode (C8093) over a 2-wire bus. *** DIGITS ARE THROUGH-HOLE (no SMD multi-digit 7-seg on LCSC) -> THT assembly. *** TM1640: shared CLK, per-chip DIN (DIN1/2/3) from the interconnect; GRID->digit commons, SEG->segments. LED current dominates active power (drawn from +3V3 across the interconnect) -> gates the main buck-boost sizing. Use brightness (TM1640 dimming) + blank-on-idle."
+	(text "Calcumaker 16 display — 7-seg RPN stack. 3 rows x 16 digits (top row U3/DS9-12 optional => 2- or 3-row build). PER ROW: 1x TM1640 (C5337152) drives 4x FJ5161AH 0.56\" 4-digit common-cathode (C8093) over a 2-wire bus. *** DIGITS ARE THROUGH-HOLE (no SMD multi-digit 7-seg on LCSC) -> THT assembly. *** TM1640: shared CLK, per-chip DIN (DIN1/2/3) from the interconnect; GRID->digit commons, SEG->segments. Runs at +5V (VDD + LED) from the main-board EN-gated 5V boost across the interconnect -> sized on that boost, not the 3V3 rail. Use brightness (TM1640 dimming) + blank-on-idle."
 		(exclude_from_sim no)
 		(at 15.00 120.00 0)

Commit message: 5V-rail BOM (TPS61022 + SN74HCT125) + 0402/0603 passive & small-magnetics policy
Sourced via the LCSC/jlcsearch skill, applying the 0402-passives / smallest-
reasonable-magnetics directive:

- 5V boost: TPS61022RWUR (C915088, EN-gated, VQFN-7) + FB divider (732k/100k→5V)
  + 1µH FTC201610S1R0MBCA (C5832342, 2.0×1.6mm) + 0603 caps (10µF in, 2×22µF out).
- Level shifter: SN74HCT125DR (C352957); KiCad symbol = stock 74xx:74AHCT125
  (pin-identical), value 74HCT125; footprint Texas_RWU0007A_VQFN-7 confirmed for
  the boost (its symbol is a TODO, batched with the MCU symbol).
- Passive policy: 0402 for R + decoupling; 0603 for bulk MLCCs (true-0402 10µF is
  6.3V-only, too low for 5V). 3V3 buck-boost inductor downsized to 0805/2016.
- Display board regenerated (0603 bulk); structure check still passes.
- DESIGN.md / PARTS.md updated with parts, LCSC#s, and the size policy.

Co-Authored-By: Claude Opus 4.8 (1M context) <noreply@anthropic.com>
Parts:
- C4: footprint Capacitor_SMD:C_0805_2012Metric -> Capacitor_SMD:C_0603_1608Metric; LCSC C15850 -> (none)
Changed lines of the file:
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@@
 		(instances
 			(project "calcumaker-display"
-				(path "/ca1c0000-0000-4000-8000-0000000d1501/bff2c2c9-e03f-4398-9f4c-6cb350699cef"
+				(path "/ca1c0000-0000-4000-8000-0000000d1501/5655df7c-81b1-4acd-8ecd-e82f9f427e94"
 					(reference "U1")
 					(unit 1)
@@
 		(instances
 			(project "calcumaker-display"
-				(path "/ca1c0000-0000-4000-8000-0000000d1501/bff2c2c9-e03f-4398-9f4c-6cb350699cef"
+				(path "/ca1c0000-0000-4000-8000-0000000d1501/5655df7c-81b1-4acd-8ecd-e82f9f427e94"
 					(reference "U2")
 					(unit 1)
@@
 		(instances
 			(project "calcumaker-display"
-				(path "/ca1c0000-0000-4000-8000-0000000d1501/bff2c2c9-e03f-4398-9f4c-6cb350699cef"
+				(path "/ca1c0000-0000-4000-8000-0000000d1501/5655df7c-81b1-4acd-8ecd-e82f9f427e94"
 					(reference "U3")
 					(unit 1)
@@
 		(instances
 			(project "calcumaker-display"
-				(path "/ca1c0000-0000-4000-8000-0000000d1501/bff2c2c9-e03f-4398-9f4c-6cb350699cef"
+				(path "/ca1c0000-0000-4000-8000-0000000d1501/5655df7c-81b1-4acd-8ecd-e82f9f427e94"
 					(reference "DS1")
 					(unit 1)
@@
 		(instances
 			(project "calcumaker-display"
-				(path "/ca1c0000-0000-4000-8000-0000000d1501/bff2c2c9-e03f-4398-9f4c-6cb350699cef"
+				(path "/ca1c0000-0000-4000-8000-0000000d1501/5655df7c-81b1-4acd-8ecd-e82f9f427e94"
 					(reference "DS2")
 					(unit 1)
@@
 		(instances
 			(project "calcumaker-display"
-				(path "/ca1c0000-0000-4000-8000-0000000d1501/bff2c2c9-e03f-4398-9f4c-6cb350699cef"
+				(path "/ca1c0000-0000-4000-8000-0000000d1501/5655df7c-81b1-4acd-8ecd-e82f9f427e94"
 					(reference "DS3")
 					(unit 1)
@@
 		(instances
 			(project "calcumaker-display"
-				(path "/ca1c0000-0000-4000-8000-0000000d1501/bff2c2c9-e03f-4398-9f4c-6cb350699cef"
+				(path "/ca1c0000-0000-4000-8000-0000000d1501/5655df7c-81b1-4acd-8ecd-e82f9f427e94"
 					(reference "DS4")
 					(unit 1)
@@
 		(instances
 			(project "calcumaker-display"
-				(path "/ca1c0000-0000-4000-8000-0000000d1501/bff2c2c9-e03f-4398-9f4c-6cb350699cef"
+				(path "/ca1c0000-0000-4000-8000-0000000d1501/5655df7c-81b1-4acd-8ecd-e82f9f427e94"
 					(reference "DS5")
 					(unit 1)
@@
 		(instances
 			(project "calcumaker-display"
-				(path "/ca1c0000-0000-4000-8000-0000000d1501/bff2c2c9-e03f-4398-9f4c-6cb350699cef"
+				(path "/ca1c0000-0000-4000-8000-0000000d1501/5655df7c-81b1-4acd-8ecd-e82f9f427e94"
 					(reference "DS6")
 					(unit 1)
@@
 		(instances
 			(project "calcumaker-display"
-				(path "/ca1c0000-0000-4000-8000-0000000d1501/bff2c2c9-e03f-4398-9f4c-6cb350699cef"
+				(path "/ca1c0000-0000-4000-8000-0000000d1501/5655df7c-81b1-4acd-8ecd-e82f9f427e94"
 					(reference "DS7")
 					(unit 1)
@@
 		(instances
 			(project "calcumaker-display"
-				(path "/ca1c0000-0000-4000-8000-0000000d1501/bff2c2c9-e03f-4398-9f4c-6cb350699cef"
+				(path "/ca1c0000-0000-4000-8000-0000000d1501/5655df7c-81b1-4acd-8ecd-e82f9f427e94"
 					(reference "DS8")
 					(unit 1)
@@
 		(instances
 			(project "calcumaker-display"
-				(path "/ca1c0000-0000-4000-8000-0000000d1501/bff2c2c9-e03f-4398-9f4c-6cb350699cef"
+				(path "/ca1c0000-0000-4000-8000-0000000d1501/5655df7c-81b1-4acd-8ecd-e82f9f427e94"
 					(reference "DS9")
 					(unit 1)
@@
 		(instances
 			(project "calcumaker-display"
-				(path "/ca1c0000-0000-4000-8000-0000000d1501/bff2c2c9-e03f-4398-9f4c-6cb350699cef"
+				(path "/ca1c0000-0000-4000-8000-0000000d1501/5655df7c-81b1-4acd-8ecd-e82f9f427e94"
 					(reference "DS10")
 					(unit 1)
@@
 		(instances
 			(project "calcumaker-display"
-				(path "/ca1c0000-0000-4000-8000-0000000d1501/bff2c2c9-e03f-4398-9f4c-6cb350699cef"
+				(path "/ca1c0000-0000-4000-8000-0000000d1501/5655df7c-81b1-4acd-8ecd-e82f9f427e94"
 					(reference "DS11")
 					(unit 1)
@@
 		(instances
 			(project "calcumaker-display"
-				(path "/ca1c0000-0000-4000-8000-0000000d1501/bff2c2c9-e03f-4398-9f4c-6cb350699cef"
+				(path "/ca1c0000-0000-4000-8000-0000000d1501/5655df7c-81b1-4acd-8ecd-e82f9f427e94"
 					(reference "DS12")
 					(unit 1)
@@
 		(instances
 			(project "calcumaker-display"
-				(path "/ca1c0000-0000-4000-8000-0000000d1501/bff2c2c9-e03f-4398-9f4c-6cb350699cef"
+				(path "/ca1c0000-0000-4000-8000-0000000d1501/5655df7c-81b1-4acd-8ecd-e82f9f427e94"
 					(reference "C1")
 					(unit 1)
@@
 		(instances
 			(project "calcumaker-display"
-				(path "/ca1c0000-0000-4000-8000-0000000d1501/bff2c2c9-e03f-4398-9f4c-6cb350699cef"
+				(path "/ca1c0000-0000-4000-8000-0000000d1501/5655df7c-81b1-4acd-8ecd-e82f9f427e94"
 					(reference "C2")
 					(unit 1)
@@
 		(instances
 			(project "calcumaker-display"
-				(path "/ca1c0000-0000-4000-8000-0000000d1501/bff2c2c9-e03f-4398-9f4c-6cb350699cef"
+				(path "/ca1c0000-0000-4000-8000-0000000d1501/5655df7c-81b1-4acd-8ecd-e82f9f427e94"
 					(reference "C3")
 					(unit 1)
@@
 			(effects (font (size 1.27 1.27)) (justify left))
 		)
-		(property "Footprint" "Capacitor_SMD:C_0805_2012Metric"
+		(property "Footprint" "Capacitor_SMD:C_0603_1608Metric"
 			(at 144.7800 121.9200 0)
 			(effects (font (size 1.27 1.27))) (hide yes)
@@
 			(effects (font (size 1.27 1.27))) (hide yes)
 		)
-		(property "LCSC" "C15850"
-			(at 144.7800 121.9200 0)
-			(effects (font (size 1.27 1.27))) (hide yes)
-		)
-		(pin "1")
-		(pin "2")
-		(instances
-			(project "calcumaker-display"
-				(path "/ca1c0000-0000-4000-8000-0000000d1501/bff2c2c9-e03f-4398-9f4c-6cb350699cef"
+		(pin "1")
+		(pin "2")
+		(instances
+			(project "calcumaker-display"
+				(path "/ca1c0000-0000-4000-8000-0000000d1501/5655df7c-81b1-4acd-8ecd-e82f9f427e94"
 					(reference "C4")
 					(unit 1)
