File: hardware/calcumaker-display/aux.kicad_sch (KiCad schematic)
At the start: 1 part, among them J2 OLED 128x32 (DNP)

Commit message: hardware: 3-board split (MCU + keyboard + display), wired display, real connectors
Split the single logic board into three, wire the display as a KiCad
multi-channel design, and settle every interconnect on real, in-stock parts.

Three-board split (was two):
- Rename calcumaker-main -> calcumaker-mcu (brain/PSU logic board).
- New calcumaker-keyboard board: 50-key Cherry MX matrix + its own
  STM32G031K8U6 scanner (LCSC C432207, UFQFPN-32) + annunciator LEDs,
  mezzanine-stacked above the MCU board. Keyscanning is off the main board;
  only an I2C + UART link + KB_IRQ wake + power cross the mezzanine.

Display board (calcumaker-display):
- Corrected FJ5161AH to a SINGLE-digit 0.56" common-cathode part (C8093) --
  it is NOT a 4-digit module; 48 single digits (16/row x 3), authored symbol
  + 0.56" LTS6760 land. The old 4-digit CC56-12 mapping (and its 3D model)
  was the phantom "clock colon".
- Rebuilt as a KiCad multi-channel design: one reusable display_row.kicad_sch
  (1 TM1640 + 16 digits, fully wired) instantiated x3. Extended kschgen.py
  with wiring primitives + reused-sheet (multi-channel) support.

Connectors (real, verified LCSC / DigiKey parts):
- Display link -> 0.5mm 12P FFC: AFC01-S12FCA-00 (LCSC C262661) on both
  boards; cable = GCT FFC05-TIN 05-12-A-<len>-A-4-06-4-T (DigiKey accessory,
  length TBD). +5V/GND conductors doubled for the display LED current.
- Keyboard mezzanine -> low-profile Hirose DF40 (0.4mm, 2x5, 1.5mm stack):
  DF40C-10DS (C424636) + DF40C-10DP (C424635) -- dedicated KiCad footprint
  + 3D model, unlike the datasheet-less generic parts first considered.

Low-power & wake documented (two Stop domains; keypress -> G0 EXTI wake ->
KB_IRQ -> U575 WKUP; G0 also wakes on I2C address-match). calcumaker-core
is unchanged -- App still consumes (row,col).

All three boards generate + pass the structure check (mcu 52 / keyboard 119 /
display 60 components, all footprints assigned, no duplicate refs). Docs
(DESIGN.md, PARTS.md incl. a Non-B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
Parts:
- J2: now not fitted
Connections:
- net +3V3: now reaches J2.1 (Pin_1)
- net GND: now reaches J2.2 (Pin_2)
- net SCL: now reaches J2.3 (Pin_3)
- net SDA: now reaches J2.4 (Pin_4)
Other:
- note added: "Calcumaker 16 display — OPTIONAL aux OLED (DNP by default). J2 receives a standard 0.91" SSD1306 128x32 I2C module (VCC GND SCL SDA; sourced separately, hand-placed with the THT digits). Wiring: J2.1 VCC<-+3V3, J2.2 GND, J2.3 SCL, J2.4 SDA. I2C at 3V3 straight from the MCU (pull-ups on the MCU board, DNP alongside). Shows full error text / SETUP / STATUS; the 7-seg glass stays primary."
- note removed: "Calcumaker 16 display — OPTIONAL aux OLED (DNP by default). J2 receives a standard 0.91" SSD1306 128x32 I2C module (VCC GND SCL SDA; module sourced separately, hand-placed with the THT digits). Wiring: J2.1 VCC <- J1.8 (+3V3), J2.2 GND, J2.3 SCL <- J1.10, J2.4 SDA <- J1.9. I2C runs at 3V3 straight from the MCU (pull-ups on the main board, DNP alongside). Firmware sleeps the panel in idle (~10uA).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"
Changed lines of the file:
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@@
 	(title_block
 		(title "Calcumaker 16 — Display — Aux OLED 128x32 (SSD1306 I2C) — DNP-optional")
-		(date "2026-06-21")
-		(rev "0.1")
+		(date "2026-07-04")
+		(rev "0.2")
 		(company "calcumaker authors")
 	)
 	(symbol
 		(lib_id "Connector_Generic:Conn_01x04")
-		(at 45.7200 55.8800 0)
+		(at 71.1200 71.1200 0)
 		(unit 1)
 		(exclude_from_sim no)
 		(in_bom yes)
 		(on_board yes)
-		(dnp no)
+		(dnp yes)
 		(property "Reference" "J2"
-			(at 49.5300 53.3400 0)
+			(at 74.9300 68.5800 0)
 			(effects (font (size 1.27 1.27)) (justify left))
 		)
 		(property "Value" "OLED 128x32 (DNP)"
-			(at 49.5300 58.4200 0)
+			(at 74.9300 73.6600 0)
 			(effects (font (size 1.27 1.27)) (justify left))
 		)
 		(property "Footprint" "Connector_PinHeader_2.54mm:PinHeader_1x04_P2.54mm_Vertical"
-			(at 45.7200 55.8800 0)
+			(at 71.1200 71.1200 0)
 			(effects (font (size 1.27 1.27))) (hide yes)
 		)
 		(property "Datasheet" "~"
-			(at 45.7200 55.8800 0)
+			(at 71.1200 71.1200 0)
 			(effects (font (size 1.27 1.27))) (hide yes)
 		)
 		(property "LCSC" "C2691448"
-			(at 45.7200 55.8800 0)
+			(at 71.1200 71.1200 0)
 			(effects (font (size 1.27 1.27))) (hide yes)
 		)
 		(property "MPN" "PZ254V-11-04P"
-			(at 45.7200 55.8800 0)
+			(at 71.1200 71.1200 0)
 			(effects (font (size 1.27 1.27))) (hide yes)
 		)
 		(property "Manufacturer" "XKB"
-			(at 45.7200 55.8800 0)
+			(at 71.1200 71.1200 0)
 			(effects (font (size 1.27 1.27))) (hide yes)
 		)
@@
 		(instances
 			(project "calcumaker-display"
-				(path "/ca1c0000-0000-4000-8000-0000000d1501/a66aef50-7a52-4b48-b96b-ed0e80888573"
+				(path "/ca1c0000-0000-4000-8000-0000000d1501/ca1c0000-0000-4000-8000-0000000d1530"
 					(reference "J2")
 					(unit 1)
@@
 		)
 	)
-	(text "Calcumaker 16 display — OPTIONAL aux OLED (DNP by default). J2 receives a standard 0.91\" SSD1306 128x32 I2C module (VCC GND SCL SDA; module sourced separately, hand-placed with the THT digits). Wiring: J2.1 VCC <- J1.8 (+3V3), J2.2 GND, J2.3 SCL <- J1.10, J2.4 SDA <- J1.9. I2C runs at 3V3 straight from the MCU (pull-ups on the main board, DNP alongside). Firmware sleeps the panel in idle (~10uA). Shows full error text / SETUP / STATUS; the 7-seg glass stays primary (Error N codes)."
+	(wire (pts (xy 66.0400 68.5800) (xy 63.5000 68.5800))
+		(stroke (width 0) (type default))
+	)
+	(global_label "+3V3"
+		(shape input)
+		(at 63.5000 68.5800 180)
+		(fields_autoplaced yes)
+		(effects (font (size 1.27 1.27)) (justify left))
+	)
+	(wire (pts (xy 66.0400 71.1200) (xy 63.5000 71.1200))
+		(stroke (width 0) (type default))
+	)
+	(global_label "GND"
+		(shape input)
+		(at 63.5000 71.1200 180)
+		(fields_autoplaced yes)
+		(effects (font (size 1.27 1.27)) (justify left))
+	)
+	(wire (pts (xy 66.0400 73.6600) (xy 63.5000 73.6600))
+		(stroke (width 0) (type default))
+	)
+	(global_label "SCL"
+		(shape input)
+		(at 63.5000 73.6600 180)
+		(fields_autoplaced yes)
+		(effects (font (size 1.27 1.27)) (justify left))
+	)
+	(wire (pts (xy 66.0400 76.2000) (xy 63.5000 76.2000))
+		(stroke (width 0) (type default))
+	)
+	(global_label "SDA"
+		(shape input)
+		(at 63.5000 76.2000 180)
+		(fields_autoplaced yes)
+		(effects (font (size 1.27 1.27)) (justify left))
+	)
+	(text "Calcumaker 16 display — OPTIONAL aux OLED (DNP by default). J2 receives a standard 0.91\" SSD1306 128x32 I2C module (VCC GND SCL SDA; sourced separately, hand-placed with the THT digits). Wiring: J2.1 VCC<-+3V3, J2.2 GND, J2.3 SCL, J2.4 SDA. I2C at 3V3 straight from the MCU (pull-ups on the MCU board, DNP alongside). Shows full error text / SETUP / STATUS; the 7-seg glass stays primary."
 		(exclude_from_sim no)
-		(at 15.00 80.00 0)
+		(at 20.00 110.00 0)
 		(effects (font (size 1.5 1.5)) (justify left top))
 	)
 	(sheet_instances
 		(path "/"
-			(page "4")
+			(page "7")
 		)
 	)

Commit message: hardware: MCU -> STM32U575RGT6 (LQFP-64) + 4MB QSPI flash; monospace wiring notes
MCU package + external flash
- Swap U1 STM32U575ZGT6 (LQFP-144) -> STM32U575RGT6 (LQFP-64, LCSC C5270980).
  The firmware links at ~323 KB so 1 MB flash is ample (~3x headroom), and with
  the key matrix scanned off-board the LQFP-64 has enough GPIO — smaller/cheaper.
- Correct the flash size everywhere: the STM32 `G` code = 1 MB (not 2 MB; the
  `I` parts are 2 MB). memory.x FLASH 2048K -> 1024K; .cargo runner -> RGTx.
- Add U7 W25Q32JVSSIQ, a 4 MB (32 Mbit) quad-SPI NOR (LCSC C179173, SOIC-8) on
  OCTOSPI1 as a new QSPIFlash sheet (+ R9 CS# pull-up + C26 decoupling) for
  memory-mapped (XIP) constants + state/program storage.
- mcu board 52 -> 55 components / 7 sheets. Docs (DESIGN.md, PARTS.md, READMEs,
  CLAUDE/AGENTS) updated; availability ladder now lists RGT6/VGT6/ZGT6.

Monospace, multi-line schematic wiring notes
- kschgen text_note() now renders notes in a monospace font (Courier New) so
  tables/columns line up; add note_block() + pin_table() helpers.
- Reformat all 14 per-sheet notes into titled, multi-line, aligned blocks —
  connector pinouts as PIN/SIGNAL tables, power/MCU sheets as wiring blocks.

The regenerated schematics carry both changes, so this is one commit. All three
boards regenerate + pass the structure check (mcu 55 / keyboard 119 / display
60, no duplicate refs).

Co-Authored-By: Claude Opus 4.8 (1M context) <noreply@anthropic.com>
Other:
- note added: "AUX OLED - J2 (OPTIONAL, DNP by default) Receives a 0.91" SSD1306 128x32 I2C module (sourced separately, hand-placed with the THT digits). I2C at 3V3 straight from the MCU (pull-ups on the MCU board, DNP alongside). PIN SIGNAL 1 VCC <- +3V3 2 GND 3 SCL 4 SDA Shows full error text / SETUP / STATUS; the 7-seg glass stays primary."
- note removed: "Calcumaker 16 display — OPTIONAL aux OLED (DNP by default). J2 receives a standard 0.91" SSD1306 128x32 I2C module (VCC GND SCL SDA; sourced separately, hand-placed with the THT digits). Wiring: J2.1 VCC<-+3V3, J2.2 GND, J2.3 SCL, J2.4 SDA. I2C at 3V3 straight from the MCU (pull-ups on the MCU board, DNP alongside). Shows full error text / SETUP / STATUS; the 7-seg glass stays primary."
Changed lines of the file:
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@@
 		(effects (font (size 1.27 1.27)) (justify left))
 	)
-	(text "Calcumaker 16 display — OPTIONAL aux OLED (DNP by default). J2 receives a standard 0.91\" SSD1306 128x32 I2C module (VCC GND SCL SDA; sourced separately, hand-placed with the THT digits). Wiring: J2.1 VCC<-+3V3, J2.2 GND, J2.3 SCL, J2.4 SDA. I2C at 3V3 straight from the MCU (pull-ups on the MCU board, DNP alongside). Shows full error text / SETUP / STATUS; the 7-seg glass stays primary."
+	(text "AUX OLED  -  J2   (OPTIONAL, DNP by default)\nReceives a 0.91\" SSD1306 128x32 I2C module (sourced separately,\nhand-placed with the THT digits).  I2C at 3V3 straight from the MCU\n(pull-ups on the MCU board, DNP alongside).\n\n  PIN  SIGNAL     \n    1  VCC <- +3V3\n    2  GND        \n    3  SCL        \n    4  SDA\n\nShows full error text / SETUP / STATUS; the 7-seg glass stays primary."
 		(exclude_from_sim no)
 		(at 20.00 110.00 0)
-		(effects (font (size 1.5 1.5)) (justify left top))
+		(effects (font (face "Courier New") (size 1.27 1.27)) (justify left top))
 	)
 	(sheet_instances
