File: hardware/calcumaker-display/interconnect.kicad_sch (KiCad schematic)
At the start: 2 parts, among them J1 TO MAIN

Commit message: Add 5V display rail: EN-gated boost + 74HCT125 level shifter
Display chosen to run at 5V (TM1640 is 5V-nominal; VIH 3.5V > the STM32's 3.3V).
Rather than upsizing the 3V3 buck-boost, split the rails:

- Keep the ULP TPS63900 at 3V3 for the MCU only (always-on, low-Iq for sleep).
- Add an EN-gated 5V boost for the display LED load (off in sleep via DISP_PWR_EN).
- Add a 74HCT125 quad buffer @5V to translate CLK + DIN1/2/3 from 3V3 to 5V.
- Interconnect now carries +5V + 5V-logic; main-board "display_if" sheet holds
  the boost + shifter + J3. Display board regenerated for the 5V note.

Boost (+inductor) and 74HCT125 LCSC parts are being picked by availability.
Updated both manifests, DESIGN.md (power tree/sheet plan/parts), README, PARTS.md.

Co-Authored-By: Claude Opus 4.8 (1M context) <noreply@anthropic.com>
Other:
- note added: "Calcumaker 16 display — Interconnect to the main board. J1 pinout (MUST match calcumaker-main J3): 1=+5V, 2=GND, 3=CLK (shared), 4=DIN1, 5=DIN2, 6=DIN3, 7=GND, 8=spare. Display runs at +5V (TM1640 VDD + LED); CLK/DIN are 5V-logic from the main-board 74HCT125 level shifter. Wide +5V/GND for LED current. 2.54mm 1x8 header (C492407); short cable to the angled display. See DESIGN.md Board Partition."
- note removed: "Calcumaker 16 display — Interconnect to the main board. J1 pinout (MUST match calcumaker-main J3): 1=+3V3, 2=GND, 3=CLK (shared), 4=DIN1, 5=DIN2, 6=DIN3, 7=GND, 8=spare. (TM1640 2-wire: one shared CLK + one DIN per row driver U1/U2/U3.) Wide +3V3/GND for LED current. 2.54mm 1x8 header (C492407); short cable to the angled display. See DESIGN.md Board Partition."
Changed lines of the file:
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@@
 		(instances
 			(project "calcumaker-display"
-				(path "/ca1c0000-0000-4000-8000-0000000d1501/003235e3-d05f-48ee-ae76-22965c0677c8"
+				(path "/ca1c0000-0000-4000-8000-0000000d1501/f2c009b6-dba2-43d5-a6f1-690da8662fd2"
 					(reference "J1")
 					(unit 1)
@@
 		(instances
 			(project "calcumaker-display"
-				(path "/ca1c0000-0000-4000-8000-0000000d1501/003235e3-d05f-48ee-ae76-22965c0677c8"
+				(path "/ca1c0000-0000-4000-8000-0000000d1501/f2c009b6-dba2-43d5-a6f1-690da8662fd2"
 					(reference "C5")
 					(unit 1)
@@
 		)
 	)
-	(text "Calcumaker 16 display — Interconnect to the main board. J1 pinout (MUST match calcumaker-main J3): 1=+3V3, 2=GND, 3=CLK (shared), 4=DIN1, 5=DIN2, 6=DIN3, 7=GND, 8=spare. (TM1640 2-wire: one shared CLK + one DIN per row driver U1/U2/U3.) Wide +3V3/GND for LED current. 2.54mm 1x8 header (C492407); short cable to the angled display. See DESIGN.md Board Partition."
+	(text "Calcumaker 16 display — Interconnect to the main board. J1 pinout (MUST match calcumaker-main J3): 1=+5V, 2=GND, 3=CLK (shared), 4=DIN1, 5=DIN2, 6=DIN3, 7=GND, 8=spare. Display runs at +5V (TM1640 VDD + LED); CLK/DIN are 5V-logic from the main-board 74HCT125 level shifter. Wide +5V/GND for LED current. 2.54mm 1x8 header (C492407); short cable to the angled display. See DESIGN.md Board Partition."
 		(exclude_from_sim no)
 		(at 15.00 95.00 0)

Commit message: 5V-rail BOM (TPS61022 + SN74HCT125) + 0402/0603 passive & small-magnetics policy
Sourced via the LCSC/jlcsearch skill, applying the 0402-passives / smallest-
reasonable-magnetics directive:

- 5V boost: TPS61022RWUR (C915088, EN-gated, VQFN-7) + FB divider (732k/100k→5V)
  + 1µH FTC201610S1R0MBCA (C5832342, 2.0×1.6mm) + 0603 caps (10µF in, 2×22µF out).
- Level shifter: SN74HCT125DR (C352957); KiCad symbol = stock 74xx:74AHCT125
  (pin-identical), value 74HCT125; footprint Texas_RWU0007A_VQFN-7 confirmed for
  the boost (its symbol is a TODO, batched with the MCU symbol).
- Passive policy: 0402 for R + decoupling; 0603 for bulk MLCCs (true-0402 10µF is
  6.3V-only, too low for 5V). 3V3 buck-boost inductor downsized to 0805/2016.
- Display board regenerated (0603 bulk); structure check still passes.
- DESIGN.md / PARTS.md updated with parts, LCSC#s, and the size policy.

Co-Authored-By: Claude Opus 4.8 (1M context) <noreply@anthropic.com>
Parts:
- C5: footprint Capacitor_SMD:C_0805_2012Metric -> Capacitor_SMD:C_0603_1608Metric; LCSC C15850 -> (none)
Changed lines of the file:
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@@
 		(instances
 			(project "calcumaker-display"
-				(path "/ca1c0000-0000-4000-8000-0000000d1501/f2c009b6-dba2-43d5-a6f1-690da8662fd2"
+				(path "/ca1c0000-0000-4000-8000-0000000d1501/c4c3c015-b6ba-4dbd-a6a4-490d09c995d8"
 					(reference "J1")
 					(unit 1)
@@
 			(effects (font (size 1.27 1.27)) (justify left))
 		)
-		(property "Footprint" "Capacitor_SMD:C_0805_2012Metric"
+		(property "Footprint" "Capacitor_SMD:C_0603_1608Metric"
 			(at 30.4800 121.9200 0)
 			(effects (font (size 1.27 1.27))) (hide yes)
@@
 			(effects (font (size 1.27 1.27))) (hide yes)
 		)
-		(property "LCSC" "C15850"
-			(at 30.4800 121.9200 0)
-			(effects (font (size 1.27 1.27))) (hide yes)
-		)
 		(pin "1")
 		(pin "2")
 		(instances
 			(project "calcumaker-display"
-				(path "/ca1c0000-0000-4000-8000-0000000d1501/f2c009b6-dba2-43d5-a6f1-690da8662fd2"
+				(path "/ca1c0000-0000-4000-8000-0000000d1501/c4c3c015-b6ba-4dbd-a6a4-490d09c995d8"
 					(reference "C5")
 					(unit 1)

Commit message: Error handling: HP-style glass codes + DNP-optional aux OLED (display board)
Two layers, per design discussion:

ENGINE/APP — CalcError restructured: TypeError(&str) becomes Op(code, msg)
with class constructors at every site; code() gives the HP-16C-style glass
class (0 math domain, 1 register/flag, 2 bits/shift/word, 3 mode ranges,
4 too large, 5 no solution, 6 stack/entry, 7 dates, 8 statistics, 9 reserved
for crash recovery), text() the full string. App shows a transient 'Error N'
on the X row (cleared by the next key, like SHOW) and keeps the full text on
the status line — the duplicated error-string mapping in run_owned/flush is
now one report() helper. All of 'Error N' renders on the 7-seg. 211 tests.

HARDWARE — the aux OLED lands on the DISPLAY board (user decision): new
AuxDisplay sheet with J2, a 1x4 socket (PZ254V-11-04P C2691448) receiving a
standard 0.91in SSD1306 128x32 I2C module, DNP by default, hand-placed with
the THT digits. Interconnect grows 1x8 -> 1x10 (PZ254V-11-10P C492409, both
boards, pinout now ... 8=+3V3 9=SDA 10=SCL); I2C pull-ups R14/R15 4.7k on
the main board, DNP with the OLED. Both boards regenerate + check clean
(main 161, display 22 components). DESIGN.md documents the layered error
story and names the reusable 'DNP-optional aux' pattern; PARTS.md updated.

Co-Authored-By: Claude Fable 5 <noreply@anthropic.com>
Parts:
- removed J1: TO MAIN, Connector_PinHeader_2.54mm:PinHeader_1x08_P2.54mm_Vertical, symbol Connector_Generic:Conn_01x08
- added J1: TO MAIN, Connector_PinHeader_2.54mm:PinHeader_1x10_P2.54mm_Vertical, symbol Connector_Generic:Conn_01x10
Other:
- note added: "Calcumaker 16 display — Interconnect to the main board. J1 pinout (MUST match calcumaker-main J3): 1=+5V, 2=GND, 3=CLK (shared), 4=DIN1, 5=DIN2, 6=DIN3, 7=GND, 8=+3V3, 9=SDA, 10=SCL. Display runs at +5V (TM1640 VDD + LED); CLK/DIN are 5V-logic from the main-board 74HCT125. Pins 8-10 feed the OPTIONAL aux OLED (AuxDisplay sheet) at 3V3 I2C — unused when the OLED is not populated. Wide +5V/GND for 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"
- note removed: "Calcumaker 16 display — Interconnect to the main board. J1 pinout (MUST match calcumaker-main J3): 1=+5V, 2=GND, 3=CLK (shared), 4=DIN1, 5=DIN2, 6=DIN3, 7=GND, 8=spare. Display runs at +5V (TM1640 VDD + LED); CLK/DIN are 5V-logic from the main-board 74HCT125 level shifter. Wide +5V/GND for LED current. 2.54mm 1x8 header (C492407); short cable to the angled display. See DESIGN.md Board Partition."
Changed lines of the file:
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@@
 	)
 	(symbol
-		(lib_id "Connector_Generic:Conn_01x08")
+		(lib_id "Connector_Generic:Conn_01x10")
 		(at 45.7200 55.8800 0)
 		(unit 1)
@@
 			(effects (font (size 1.27 1.27)) (justify left))
 		)
-		(property "Footprint" "Connector_PinHeader_2.54mm:PinHeader_1x08_P2.54mm_Vertical"
+		(property "Footprint" "Connector_PinHeader_2.54mm:PinHeader_1x10_P2.54mm_Vertical"
 			(at 45.7200 55.8800 0)
 			(effects (font (size 1.27 1.27))) (hide yes)
@@
 			(effects (font (size 1.27 1.27))) (hide yes)
 		)
-		(property "LCSC" "C492407"
+		(property "LCSC" "C492409"
 			(at 45.7200 55.8800 0)
 			(effects (font (size 1.27 1.27))) (hide yes)
 		)
-		(property "MPN" "PZ254V-11-08P"
+		(property "MPN" "PZ254V-11-10P"
 			(at 45.7200 55.8800 0)
 			(effects (font (size 1.27 1.27))) (hide yes)
@@
 		(pin "7")
 		(pin "8")
+		(pin "9")
+		(pin "10")
 		(instances
 			(project "calcumaker-display"
-				(path "/ca1c0000-0000-4000-8000-0000000d1501/c4c3c015-b6ba-4dbd-a6a4-490d09c995d8"
+				(path "/ca1c0000-0000-4000-8000-0000000d1501/6885ee80-e191-4b5d-9a90-d31ab546f2b5"
 					(reference "J1")
 					(unit 1)
@@
 		(instances
 			(project "calcumaker-display"
-				(path "/ca1c0000-0000-4000-8000-0000000d1501/c4c3c015-b6ba-4dbd-a6a4-490d09c995d8"
+				(path "/ca1c0000-0000-4000-8000-0000000d1501/6885ee80-e191-4b5d-9a90-d31ab546f2b5"
 					(reference "C5")
 					(unit 1)
@@
 		)
 	)
-	(text "Calcumaker 16 display — Interconnect to the main board. J1 pinout (MUST match calcumaker-main J3): 1=+5V, 2=GND, 3=CLK (shared), 4=DIN1, 5=DIN2, 6=DIN3, 7=GND, 8=spare. Display runs at +5V (TM1640 VDD + LED); CLK/DIN are 5V-logic from the main-board 74HCT125 level shifter. Wide +5V/GND for LED current. 2.54mm 1x8 header (C492407); short cable to the angled display. See DESIGN.md Board Partition."
+	(text "Calcumaker 16 display — Interconnect to the main board. J1 pinout (MUST match calcumaker-main J3): 1=+5V, 2=GND, 3=CLK (shared), 4=DIN1, 5=DIN2, 6=DIN3, 7=GND, 8=+3V3, 9=SDA, 10=SCL. Display runs at +5V (TM1640 VDD + LED); CLK/DIN are 5V-logic from the main-board 74HCT125. Pins 8-10 feed the OPTIONAL aux OLED (AuxDisplay sheet) at 3V3 I2C — unused when the OLED is not populated. Wide +5V/GND for LED current. 2.54mm 1x10 header (C492409); short cable to the angled display. See DESIGN.md Board Partition."
 		(exclude_from_sim no)
 		(at 15.00 95.00 0)

Commit message: hardware: 3-board split (MCU + keyboard + display), wired display, real connectors
Split the single logic board into three, wire the display as a KiCad
multi-channel design, and settle every interconnect on real, in-stock parts.

Three-board split (was two):
- Rename calcumaker-main -> calcumaker-mcu (brain/PSU logic board).
- New calcumaker-keyboard board: 50-key Cherry MX matrix + its own
  STM32G031K8U6 scanner (LCSC C432207, UFQFPN-32) + annunciator LEDs,
  mezzanine-stacked above the MCU board. Keyscanning is off the main board;
  only an I2C + UART link + KB_IRQ wake + power cross the mezzanine.

Display board (calcumaker-display):
- Corrected FJ5161AH to a SINGLE-digit 0.56" common-cathode part (C8093) --
  it is NOT a 4-digit module; 48 single digits (16/row x 3), authored symbol
  + 0.56" LTS6760 land. The old 4-digit CC56-12 mapping (and its 3D model)
  was the phantom "clock colon".
- Rebuilt as a KiCad multi-channel design: one reusable display_row.kicad_sch
  (1 TM1640 + 16 digits, fully wired) instantiated x3. Extended kschgen.py
  with wiring primitives + reused-sheet (multi-channel) support.

Connectors (real, verified LCSC / DigiKey parts):
- Display link -> 0.5mm 12P FFC: AFC01-S12FCA-00 (LCSC C262661) on both
  boards; cable = GCT FFC05-TIN 05-12-A-<len>-A-4-06-4-T (DigiKey accessory,
  length TBD). +5V/GND conductors doubled for the display LED current.
- Keyboard mezzanine -> low-profile Hirose DF40 (0.4mm, 2x5, 1.5mm stack):
  DF40C-10DS (C424636) + DF40C-10DP (C424635) -- dedicated KiCad footprint
  + 3D model, unlike the datasheet-less generic parts first considered.

Low-power & wake documented (two Stop domains; keypress -> G0 EXTI wake ->
KB_IRQ -> U575 WKUP; G0 also wakes on I2C address-match). calcumaker-core
is unchanged -- App still consumes (row,col).

All three boards generate + pass the structure check (mcu 52 / keyboard 119 /
display 60 components, all footprints assigned, no duplicate refs). Docs
(DESIGN.md, PARTS.md incl. a Non-B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
Parts:
- removed C5: 10uF, Capacitor_SMD:C_0603_1608Metric, symbol Device:C
- removed J1: TO MAIN, Connector_PinHeader_2.54mm:PinHeader_1x10_P2.54mm_Vertical, symbol Connector_Generic:Conn_01x10
- added C7: 10uF, Capacitor_SMD:C_0603_1608Metric, symbol Device:C
- added J1: TO MCU (FFC), Connector_FFC-FPC:Hirose_FH12-12S-0.5SH_1x12-1MP_P0.50mm_Horizontal, symbol Connector_Generic:Conn_01x12
Connections:
- new net +3V3: J1.9 (Pin_9)
- new net +5V: C7.1, J1.1 (Pin_1), J1.2 (Pin_2)
- new net DIN1: J1.5 (Pin_5)
- new net DIN2: J1.6 (Pin_6)
- new net DIN3: J1.7 (Pin_7)
- new net DISP_CLK: J1.4 (Pin_4)
- new net GND: C7.2, J1.12 (Pin_12), J1.3 (Pin_3), J1.8 (Pin_8)
- new net SCL: J1.11 (Pin_11)
- new net SDA: J1.10 (Pin_10)
Other:
- note added: "Calcumaker 16 display — Interconnect to the MCU board = 0.5mm 12P FFC (J1 AFC01-S12FCA-00, LCSC C262661; the flat-flex CABLE = GCT FFC05-TIN 05-12-A-<len>-A-4-06-4-T, DigiKey, length TBD @ layout, NOT assembled). Pinout (MUST match calcumaker-mcu J3): 1=+5V, 2=+5V, 3=GND, 4=CLK (shared), 5=DIN1, 6=DIN2, 7=DIN3, 8=GND, 9=+3V3, 10=SDA, 11=SCL, 12=GND. +5V + GND are DOUBLED/TRIPLED for the display L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"
- note removed: "Calcumaker 16 display — Interconnect to the main board. J1 pinout (MUST match calcumaker-main J3): 1=+5V, 2=GND, 3=CLK (shared), 4=DIN1, 5=DIN2, 6=DIN3, 7=GND, 8=+3V3, 9=SDA, 10=SCL. Display runs at +5V (TM1640 VDD + LED); CLK/DIN are 5V-logic from the main-board 74HCT125. Pins 8-10 feed the OPTIONAL aux OLED (AuxDisplay sheet) at 3V3 I2C — unused when the OLED is not populated. Wide +5V/GND for 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"
- title: Calcumaker 16 — Display — Main board interconnect -> Calcumaker 16 — Display — MCU board interconnect (0.5mm FFC)
Changed lines of the file:
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@@
 	(paper "A3")
 	(title_block
-		(title "Calcumaker 16 — Display — Main board interconnect")
-		(date "2026-06-21")
-		(rev "0.1")
+		(title "Calcumaker 16 — Display — MCU board interconnect (0.5mm FFC)")
+		(date "2026-07-04")
+		(rev "0.2")
 		(company "calcumaker authors")
 	)
 	(symbol
-		(lib_id "Connector_Generic:Conn_01x10")
-		(at 45.7200 55.8800 0)
+		(lib_id "Connector_Generic:Conn_01x12")
+		(at 71.1200 71.1200 0)
 		(unit 1)
 		(exclude_from_sim no)
@@
 		(dnp no)
 		(property "Reference" "J1"
-			(at 49.5300 53.3400 0)
-			(effects (font (size 1.27 1.27)) (justify left))
-		)
-		(property "Value" "TO MAIN"
-			(at 49.5300 58.4200 0)
-			(effects (font (size 1.27 1.27)) (justify left))
-		)
-		(property "Footprint" "Connector_PinHeader_2.54mm:PinHeader_1x10_P2.54mm_Vertical"
-			(at 45.7200 55.8800 0)
+			(at 74.9300 68.5800 0)
+			(effects (font (size 1.27 1.27)) (justify left))
+		)
+		(property "Value" "TO MCU (FFC)"
+			(at 74.9300 73.6600 0)
+			(effects (font (size 1.27 1.27)) (justify left))
+		)
+		(property "Footprint" "Connector_FFC-FPC:Hirose_FH12-12S-0.5SH_1x12-1MP_P0.50mm_Horizontal"
+			(at 71.1200 71.1200 0)
 			(effects (font (size 1.27 1.27))) (hide yes)
 		)
 		(property "Datasheet" "~"
-			(at 45.7200 55.8800 0)
-			(effects (font (size 1.27 1.27))) (hide yes)
-		)
-		(property "LCSC" "C492409"
-			(at 45.7200 55.8800 0)
-			(effects (font (size 1.27 1.27))) (hide yes)
-		)
-		(property "MPN" "PZ254V-11-10P"
-			(at 45.7200 55.8800 0)
-			(effects (font (size 1.27 1.27))) (hide yes)
-		)
-		(property "Manufacturer" "XKB"
-			(at 45.7200 55.8800 0)
+			(at 71.1200 71.1200 0)
+			(effects (font (size 1.27 1.27))) (hide yes)
+		)
+		(property "LCSC" "C262661"
+			(at 71.1200 71.1200 0)
+			(effects (font (size 1.27 1.27))) (hide yes)
+		)
+		(property "MPN" "AFC01-S12FCA-00"
+			(at 71.1200 71.1200 0)
+			(effects (font (size 1.27 1.27))) (hide yes)
+		)
+		(property "Manufacturer" "JUSHUO"
+			(at 71.1200 71.1200 0)
 			(effects (font (size 1.27 1.27))) (hide yes)
 		)
@@
 		(pin "9")
 		(pin "10")
+		(pin "11")
+		(pin "12")
 		(instances
 			(project "calcumaker-display"
-				(path "/ca1c0000-0000-4000-8000-0000000d1501/6885ee80-e191-4b5d-9a90-d31ab546f2b5"
+				(path "/ca1c0000-0000-4000-8000-0000000d1501/ca1c0000-0000-4000-8000-0000000d1520"
 					(reference "J1")
 					(unit 1)
@@
 	(symbol
 		(lib_id "Device:C")
-		(at 30.4800 121.9200 0)
+		(at 121.9200 71.1200 0)
 		(unit 1)
 		(exclude_from_sim no)
@@
 		(on_board yes)
 		(dnp no)
-		(property "Reference" "C5"
-			(at 34.2900 119.3800 0)
+		(property "Reference" "C7"
+			(at 125.7300 68.5800 0)
 			(effects (font (size 1.27 1.27)) (justify left))
 		)
 		(property "Value" "10uF"
-			(at 34.2900 124.4600 0)
+			(at 125.7300 73.6600 0)
 			(effects (font (size 1.27 1.27)) (justify left))
 		)
 		(property "Footprint" "Capacitor_SMD:C_0603_1608Metric"
-			(at 30.4800 121.9200 0)
+			(at 121.9200 71.1200 0)
 			(effects (font (size 1.27 1.27))) (hide yes)
 		)
 		(property "Datasheet" "~"
-			(at 30.4800 121.9200 0)
+			(at 121.9200 71.1200 0)
+			(effects (font (size 1.27 1.27))) (hide yes)
+		)
+		(property "LCSC" "C15850"
+			(at 121.9200 71.1200 0)
 			(effects (font (size 1.27 1.27))) (hide yes)
 		)
@@
 		(instances
 			(project "calcumaker-display"
-				(path "/ca1c0000-0000-4000-8000-0000000d1501/6885ee80-e191-4b5d-9a90-d31ab546f2b5"
-					(reference "C5")
+				(path "/ca1c0000-0000-4000-8000-0000000d1501/ca1c0000-0000-4000-8000-0000000d1520"
+					(reference "C7")
 					(unit 1)
 				)
@@
 		)
 	)
-	(text "Calcumaker 16 display — Interconnect to the main board. J1 pinout (MUST match calcumaker-main J3): 1=+5V, 2=GND, 3=CLK (shared), 4=DIN1, 5=DIN2, 6=DIN3, 7=GND, 8=+3V3, 9=SDA, 10=SCL. Display runs at +5V (TM1640 VDD + LED); CLK/DIN are 5V-logic from the main-board 74HCT125. Pins 8-10 feed the OPTIONAL aux OLED (AuxDisplay sheet) at 3V3 I2C — unused when the OLED is not populated. Wide +5V/GND for LED current. 2.54mm 1x10 header (C492409); short cable to the angled display. See DESIGN.md Board Partition."
+	(wire (pts (xy 66.0400 58.4200) (xy 63.5000 58.4200))
+		(stroke (width 0) (type default))
+	)
+	(global_label "+5V"
+		(shape input)
+		(at 63.5000 58.4200 180)
+		(fields_autoplaced yes)
+		(effects (font (size 1.27 1.27)) (justify left))
+	)
+	(wire (pts (xy 66.0400 60.9600) (xy 63.5000 60.9600))
+		(stroke (width 0) (type default))
+	)
+	(global_label "+5V"
+		(shape input)
+		(at 63.5000 60.9600 180)
+		(fields_autoplaced yes)
+		(effects (font (size 1.27 1.27)) (justify left))
+	)
+	(wire (pts (xy 66.0400 63.5000) (xy 63.5000 63.5000))
+		(stroke (width 0) (type default))
+	)
+	(global_label "GND"
+		(shape input)
+		(at 63.5000 63.5000 180)
+		(fields_autoplaced yes)
+		(effects (font (size 1.27 1.27)) (justify left))
+	)
+	(wire (pts (xy 66.0400 66.0400) (xy 63.5000 66.0400))
+		(stroke (width 0) (type default))
+	)
+	(global_label "DISP_CLK"
+		(shape input)
+		(at 63.5000 66.0400 180)
+		(fields_autoplaced yes)
+		(effects (font (size 1.27 1.27)) (justify left))
+	)
+	(wire (pts (xy 66.0400 68.5800) (xy 63.5000 68.5800))
+		(stroke (width 0) (type default))
+	)
+	(global_label "DIN1"
+		(shape input)
+		(at 63.5000 68.5800 180)
+		(fields_autoplaced yes)
+		(effects (font (size 1.27 1.27)) (justify left))
+	)
+	(wire (pts (xy 66.0400 71.1200) (xy 63.5000 71.1200))
+		(stroke (width 0) (type default))
+	)
+	(global_label "DIN2"
+		(shape input)
+		(at 63.5000 71.1200 180)
+		(fields_autoplaced yes)
+		(effects (font (size 1.27 1.27)) (justify left))
+	)
+	(wire (pts (xy 66.0400 73.6600) (xy 63.5000 73.6600))
+		(stroke (width 0) (type default))
+	)
+	(global_label "DIN3"
+		(shape input)
+		(at 63.5000 73.6600 180)
+		(fields_autoplaced yes)
+		(effects (font (size 1.27 1.27)) (justify left))
+	)
+	(wire (pts (xy 66.0400 76.2000) (xy 63.5000 76.2000))
+		(stroke (width 0) (type default))
+	)
+	(global_label "GND"
+		(shape input)
+		(at 63.5000 76.2000 180)
+		(fields_autoplaced yes)
+		(effects (font (size 1.27 1.27)) (justify left))
+	)
+	(wire (pts (xy 66.0400 78.7400) (xy 63.5000 78.7400))
+		(stroke (width 0) (type default))
+	)
+	(global_label "+3V3"
+		(shape input)
+		(at 63.5000 78.7400 180)
+		(fields_autoplaced yes)
+		(effects (font (size 1.27 1.27)) (justify left))
+	)
+	(wire (pts (xy 66.0400 81.2800) (xy 63.5000 81.2800))
+		(stroke (width 0) (type default))
+	)
+	(global_label "SDA"
+		(shape input)
+		(at 63.5000 81.2800 180)
+		(fields_autoplaced yes)
+		(effects (font (size 1.27 1.27)) (justify left))
+	)
+	(wire (pts (xy 66.0400 83.8200) (xy 63.5000 83.8200))
+		(stroke (width 0) (type default))
+	)
+	(global_label "SCL"
+		(shape input)
+		(at 63.5000 83.8200 180)
+		(fields_autoplaced yes)
+		(effects (font (size 1.27 1.27)) (justify left))
+	)
+	(wire (pts (xy 66.0400 86.3600) (xy 63.5000 86.3600))
+		(stroke (width 0) (type default))
+	)
+	(global_label "GND"
+		(shape input)
+		(at 63.5000 86.3600 180)
+		(fields_autoplaced yes)
+		(effects (font (size 1.27 1.27)) (justify left))
+	)
+	(wire (pts (xy 121.9200 67.3100) (xy 121.9200 64.7700))
+		(stroke (width 0) (type default))
+	)
+	(global_label "+5V"
+		(shape input)
+		(at 121.9200 64.7700 270)
+		(fields_autoplaced yes)
+		(effects (font (size 1.27 1.27)) (justify left))
+	)
+	(wire (pts (xy 121.9200 74.9300) (xy 121.9200 77.4700))
+		(stroke (width 0) (type default))
+	)
+	(global_label "GND"
+		(shape input)
+		(at 121.9200 77.4700 90)
+		(fields_autoplaced yes)
+		(effects (font (size 1.27 1.27)) (justify left))
+	)
+	(text "Calcumaker 16 display — Interconnect to the MCU board = 0.5mm 12P FFC (J1 AFC01-S12FCA-00, LCSC C262661; the flat-flex CABLE = GCT FFC05-TIN 05-12-A-<len>-A-4-06-4-T, DigiKey, length TBD @ layout, NOT assembled). Pinout (MUST match calcumaker-mcu J3): 1=+5V, 2=+5V, 3=GND, 4=CLK (shared), 5=DIN1, 6=DIN2, 7=DIN3, 8=GND, 9=+3V3, 10=SDA, 11=SCL, 12=GND. +5V + GND are DOUBLED/TRIPLED for the display LED current (a 0.5mm FFC conductor is ~0.4A; 3 TM1640s peak ~0.3-0.5A on +5V, less with brightness capping). CLK/DIN are 5V-logic from the MCU-board 74HCT125; DIN1/2/3 fan out to Row1/2/3; DISP_CLK is shared. Pins 9-11 feed the OPTIONAL aux OLED (AuxDisplay) at 3V3 I2C. Verify the FFC land + contact orientation (top/bottom, same/opposite end) vs the AFC01 datasheet at layout. See DESIGN.md."
 		(exclude_from_sim no)
-		(at 15.00 95.00 0)
+		(at 20.00 120.00 0)
 		(effects (font (size 1.5 1.5)) (justify left top))
 	)
 	(sheet_instances
 		(path "/"
-			(page "3")
-		)
-	)
+			(page "6")
+		)
+	)
