File: hardware/calcumaker-display/interconnect.kicad_sch (KiCad schematic)
At the start: 2 parts, among them J1 TO MCU (FFC)

Commit message: hardware: MCU -> STM32U575RGT6 (LQFP-64) + 4MB QSPI flash; monospace wiring notes
MCU package + external flash
- Swap U1 STM32U575ZGT6 (LQFP-144) -> STM32U575RGT6 (LQFP-64, LCSC C5270980).
  The firmware links at ~323 KB so 1 MB flash is ample (~3x headroom), and with
  the key matrix scanned off-board the LQFP-64 has enough GPIO — smaller/cheaper.
- Correct the flash size everywhere: the STM32 `G` code = 1 MB (not 2 MB; the
  `I` parts are 2 MB). memory.x FLASH 2048K -> 1024K; .cargo runner -> RGTx.
- Add U7 W25Q32JVSSIQ, a 4 MB (32 Mbit) quad-SPI NOR (LCSC C179173, SOIC-8) on
  OCTOSPI1 as a new QSPIFlash sheet (+ R9 CS# pull-up + C26 decoupling) for
  memory-mapped (XIP) constants + state/program storage.
- mcu board 52 -> 55 components / 7 sheets. Docs (DESIGN.md, PARTS.md, READMEs,
  CLAUDE/AGENTS) updated; availability ladder now lists RGT6/VGT6/ZGT6.

Monospace, multi-line schematic wiring notes
- kschgen text_note() now renders notes in a monospace font (Courier New) so
  tables/columns line up; add note_block() + pin_table() helpers.
- Reformat all 14 per-sheet notes into titled, multi-line, aligned blocks —
  connector pinouts as PIN/SIGNAL tables, power/MCU sheets as wiring blocks.

The regenerated schematics carry both changes, so this is one commit. All three
boards regenerate + pass the structure check (mcu 55 / keyboard 119 / display
60, no duplicate refs).

Co-Authored-By: Claude Opus 4.8 (1M context) <noreply@anthropic.com>
Other:
- note added: "DISPLAY INTERCONNECT - J1 AFC01-S12FCA-00 (LCSC C262661) 0.5mm 12-pos FFC to the MCU board. Pinout MUST match mcu J3. PIN SIGNAL PIN SIGNAL 1 +5V 7 DIN3 2 +5V 8 GND 3 GND 9 +3V3 4 CLK (shared) 10 SDA 5 DIN1 11 SCL 6 DIN2 12 GND +5V/GND doubled: a 0.5mm FFC conductor is ~0.4A; 3x TM1640 peak ~0.3-0.5A on +5V (less with brightness capping). CLK/DIN1-3 are 5V-logic from the MCU-board 74HCT125. Pins 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"
- note removed: "Calcumaker 16 display — Interconnect to the MCU board = 0.5mm 12P FFC (J1 AFC01-S12FCA-00, LCSC C262661; the flat-flex CABLE = GCT FFC05-TIN 05-12-A-<len>-A-4-06-4-T, DigiKey, length TBD @ layout, NOT assembled). Pinout (MUST match calcumaker-mcu J3): 1=+5V, 2=+5V, 3=GND, 4=CLK (shared), 5=DIN1, 6=DIN2, 7=DIN3, 8=GND, 9=+3V3, 10=SDA, 11=SCL, 12=GND. +5V + GND are DOUBLED/TRIPLED for the display L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"
Changed lines of the file:
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@@
 		(effects (font (size 1.27 1.27)) (justify left))
 	)
-	(text "Calcumaker 16 display — Interconnect to the MCU board = 0.5mm 12P FFC (J1 AFC01-S12FCA-00, LCSC C262661; the flat-flex CABLE = GCT FFC05-TIN 05-12-A-<len>-A-4-06-4-T, DigiKey, length TBD @ layout, NOT assembled). Pinout (MUST match calcumaker-mcu J3): 1=+5V, 2=+5V, 3=GND, 4=CLK (shared), 5=DIN1, 6=DIN2, 7=DIN3, 8=GND, 9=+3V3, 10=SDA, 11=SCL, 12=GND. +5V + GND are DOUBLED/TRIPLED for the display LED current (a 0.5mm FFC conductor is ~0.4A; 3 TM1640s peak ~0.3-0.5A on +5V, less with brightness capping). CLK/DIN are 5V-logic from the MCU-board 74HCT125; DIN1/2/3 fan out to Row1/2/3; DISP_CLK is shared. Pins 9-11 feed the OPTIONAL aux OLED (AuxDisplay) at 3V3 I2C. Verify the FFC land + contact orientation (top/bottom, same/opposite end) vs the AFC01 datasheet at layout. See DESIGN.md."
+	(text "DISPLAY INTERCONNECT  -  J1  AFC01-S12FCA-00  (LCSC C262661)\n0.5mm 12-pos FFC to the MCU board.  Pinout MUST match mcu J3.\n\n  PIN  SIGNAL          PIN  SIGNAL      \n    1  +5V               7  DIN3        \n    2  +5V               8  GND         \n    3  GND               9  +3V3        \n    4  CLK (shared)     10  SDA         \n    5  DIN1             11  SCL         \n    6  DIN2             12  GND\n\n+5V/GND doubled: a 0.5mm FFC conductor is ~0.4A; 3x TM1640 peak\n~0.3-0.5A on +5V (less with brightness capping).\nCLK/DIN1-3 are 5V-logic from the MCU-board 74HCT125.\nPins 9-11 (+3V3/SDA/SCL) feed the DNP aux OLED (unused if bare).\n\nCABLE (non-BOM): GCT FFC05-TIN  05-12-A-<len>-A-4-06-4-T  (DigiKey);\n                 length + A(same-side)/D(opposite) contacts TBD @ layout.\nVerify the FFC land vs the AFC01 datasheet at layout.  See DESIGN.md."
 		(exclude_from_sim no)
 		(at 20.00 120.00 0)
-		(effects (font (size 1.5 1.5)) (justify left top))
+		(effects (font (face "Courier New") (size 1.27 1.27)) (justify left top))
 	)
 	(sheet_instances
