File: hardware/calcumaker-display/display_row.kicad_sch (KiCad schematic)
At the start: 19 parts, among them U1 TM1640

Commit message: hardware: MCU -> STM32U575RGT6 (LQFP-64) + 4MB QSPI flash; monospace wiring notes
MCU package + external flash
- Swap U1 STM32U575ZGT6 (LQFP-144) -> STM32U575RGT6 (LQFP-64, LCSC C5270980).
  The firmware links at ~323 KB so 1 MB flash is ample (~3x headroom), and with
  the key matrix scanned off-board the LQFP-64 has enough GPIO — smaller/cheaper.
- Correct the flash size everywhere: the STM32 `G` code = 1 MB (not 2 MB; the
  `I` parts are 2 MB). memory.x FLASH 2048K -> 1024K; .cargo runner -> RGTx.
- Add U7 W25Q32JVSSIQ, a 4 MB (32 Mbit) quad-SPI NOR (LCSC C179173, SOIC-8) on
  OCTOSPI1 as a new QSPIFlash sheet (+ R9 CS# pull-up + C26 decoupling) for
  memory-mapped (XIP) constants + state/program storage.
- mcu board 52 -> 55 components / 7 sheets. Docs (DESIGN.md, PARTS.md, READMEs,
  CLAUDE/AGENTS) updated; availability ladder now lists RGT6/VGT6/ZGT6.

Monospace, multi-line schematic wiring notes
- kschgen text_note() now renders notes in a monospace font (Courier New) so
  tables/columns line up; add note_block() + pin_table() helpers.
- Reformat all 14 per-sheet notes into titled, multi-line, aligned blocks —
  connector pinouts as PIN/SIGNAL tables, power/MCU sheets as wiring blocks.

The regenerated schematics carry both changes, so this is one commit. All three
boards regenerate + pass the structure check (mcu 55 / keyboard 119 / display
60, no duplicate refs).

Co-Authored-By: Claude Opus 4.8 (1M context) <noreply@anthropic.com>
Other:
- note added: "REUSABLE ROW (multi-channel: instantiated x3 as Row1/Row2/Row3) Row1 -> U1 / DS1-16 Row2 -> U2 / DS17-32 Row3 -> U3 / DS33-48 One TM1640 (C5337152) drives 16x FJ5161AH single-digit 0.56" common- cathode (C8093, THROUGH-HOLE): SEG1..8 (a..g,dp) - shared 8-line bus to all 16 digits' segments GRID1..16 - one per digit (GRID k -> digit k cathode) VDD -> +5V VSS -> GND SCLK -> DISP_CLK (global net, sh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"
- note removed: "Calcumaker 16 display — REUSABLE ROW (multi-channel: instantiated x3 as Row1/Row2/Row3 => U1/DS1-16, U2/DS17-32, U3/DS33-48). One TM1640 (C5337152) drives 16x FJ5161AH single-digit 0.56" common-cathode (C8093, THROUGH-HOLE) over a shared 8-line SEG bus (SEG1..8 = a..g,dp) + 16 GRID lines (GRID k -> digit k cathode). Runs at +5V (VDD + LED) from the MCU-board EN-gated 5V boost. Shared across all r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"
Changed lines of the file:
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@@
 		(effects (font (size 1.27 1.27)) (justify left))
 	)
-	(text "Calcumaker 16 display — REUSABLE ROW (multi-channel: instantiated x3 as Row1/Row2/Row3 => U1/DS1-16, U2/DS17-32, U3/DS33-48). One TM1640 (C5337152) drives 16x FJ5161AH single-digit 0.56\" common-cathode (C8093, THROUGH-HOLE) over a shared 8-line SEG bus (SEG1..8 = a..g,dp) + 16 GRID lines (GRID k -> digit k cathode). Runs at +5V (VDD + LED) from the MCU-board EN-gated 5V boost. Shared across all rows via global nets: +5V, GND, DISP_CLK. Per-row DIN is a hierarchical pin (Row1<-DIN1, Row2<-DIN2, Row3<-DIN3 at the root). Digit->GRID mapping is 1:1 and sequential; firmware seg7/App is the source of truth — keep them in step. *** THT digits: no SMD multi-digit 7-seg on LCSC. *** Verify FJ5161AH pad map vs the LTS6760 0.56\" land before fab."
+	(text "REUSABLE ROW  (multi-channel: instantiated x3 as Row1/Row2/Row3)\n  Row1 -> U1 / DS1-16     Row2 -> U2 / DS17-32     Row3 -> U3 / DS33-48\n\nOne TM1640 (C5337152) drives 16x FJ5161AH single-digit 0.56\" common-\ncathode (C8093, THROUGH-HOLE):\n  SEG1..8 (a..g,dp)  -  shared 8-line bus to all 16 digits' segments\n  GRID1..16          -  one per digit  (GRID k -> digit k cathode)\n  VDD  -> +5V              VSS  -> GND\n  SCLK -> DISP_CLK (global net, shared by all 3 rows)\n  DIN  -> hierarchical pin (Row1<-DIN1, Row2<-DIN2, Row3<-DIN3 @ root)\n\nRuns at +5V (VDD + LED) from the MCU-board EN-gated 5V boost.\nDigit->GRID is 1:1 sequential; firmware seg7/App is the source of truth.\n*** THT digits (no SMD multi-digit 7-seg on LCSC). ***\nVerify FJ5161AH pad map vs the LTS6760 0.56\" land before fab."
 		(exclude_from_sim no)
 		(at 20.00 240.00 0)
-		(effects (font (size 1.5 1.5)) (justify left top))
+		(effects (font (face "Courier New") (size 1.27 1.27)) (justify left top))
 	)
 	(sheet_instances
