File: hardware/calcumaker-display/display_row.kicad_sch (KiCad schematic)
At the start: 19 parts, among them U1 TM1640

Commit message: Floorplan both display PCBs and verify their schematic nets
Other:
- title: Calcumaker 16 — Display — Reusable 7-seg row (1x TM1640 + 16 digits) -> Calcumaker 16 / 16-digit row
