File: hardware/calcumaker-display/disp_power.kicad_sch (KiCad schematic)
At the start: 15 parts, among them U5 TPS61022RWUR, U6 74HCT1G125, U7 74HCT1G125, U8 74HCT1G125, U9 74HCT1G125

Commit message: Floorplan both display PCBs and verify their schematic nets
Parts:
- U6, U7, U8, U9: footprint Package_TO_SOT_SMD:SOT-23-5 -> Package_TO_SOT_SMD:SOT-353_SC-70-5
