File: hardware/calcumaker-mcu/mcu.kicad_sch (KiCad schematic)
At the start: 14 parts, among them U1 STM32U575ZGT6

Commit message: hardware: 3-board split (MCU + keyboard + display), wired display, real connectors
Split the single logic board into three, wire the display as a KiCad
multi-channel design, and settle every interconnect on real, in-stock parts.

Three-board split (was two):
- Rename calcumaker-main -> calcumaker-mcu (brain/PSU logic board).
- New calcumaker-keyboard board: 50-key Cherry MX matrix + its own
  STM32G031K8U6 scanner (LCSC C432207, UFQFPN-32) + annunciator LEDs,
  mezzanine-stacked above the MCU board. Keyscanning is off the main board;
  only an I2C + UART link + KB_IRQ wake + power cross the mezzanine.

Display board (calcumaker-display):
- Corrected FJ5161AH to a SINGLE-digit 0.56" common-cathode part (C8093) --
  it is NOT a 4-digit module; 48 single digits (16/row x 3), authored symbol
  + 0.56" LTS6760 land. The old 4-digit CC56-12 mapping (and its 3D model)
  was the phantom "clock colon".
- Rebuilt as a KiCad multi-channel design: one reusable display_row.kicad_sch
  (1 TM1640 + 16 digits, fully wired) instantiated x3. Extended kschgen.py
  with wiring primitives + reused-sheet (multi-channel) support.

Connectors (real, verified LCSC / DigiKey parts):
- Display link -> 0.5mm 12P FFC: AFC01-S12FCA-00 (LCSC C262661) on both
  boards; cable = GCT FFC05-TIN 05-12-A-<len>-A-4-06-4-T (DigiKey accessory,
  length TBD). +5V/GND conductors doubled for the display LED current.
- Keyboard mezzanine -> low-profile Hirose DF40 (0.4mm, 2x5, 1.5mm stack):
  DF40C-10DS (C424636) + DF40C-10DP (C424635) -- dedicated KiCad footprint
  + 3D model, unlike the datasheet-less generic parts first considered.

Low-power & wake documented (two Stop domains; keypress -> G0 EXTI wake ->
KB_IRQ -> U575 WKUP; G0 also wakes on I2C address-match). calcumaker-core
is unchanged -- App still consumes (row,col).

All three boards generate + pass the structure check (mcu 52 / keyboard 119 /
display 60 components, all footprints assigned, no duplicate refs). Docs
(DESIGN.md, PARTS.md incl. a Non-B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
Other:
- title: Calcumaker 16 — Main — MCU core (STM32U575) -> Calcumaker 16 — MCU — MCU core (STM32U575)
Changed lines of the file:
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@@
 	(paper "A3")
 	(title_block
-		(title "Calcumaker 16 — Main — MCU core (STM32U575)")
-		(date "2026-06-21")
-		(rev "0.1")
+		(title "Calcumaker 16 — MCU — MCU core (STM32U575)")
+		(date "2026-07-05")
+		(rev "0.2")
 		(company "calcumaker authors")
 	)
@@
 		(pin "144")
 		(instances
-			(project "calcumaker-main"
-				(path "/ca1c0000-0000-4000-8000-00000000ma01/da764cdd-8caf-4481-b72a-cf9dd25cafa9"
+			(project "calcumaker-mcu"
+				(path "/ca1c0000-0000-4000-8000-00000000ma01/23aa651c-01ea-4ee3-bb12-f879a30c281f"
 					(reference "U1")
 					(unit 1)
@@
 		(pin "2")
 		(instances
-			(project "calcumaker-main"
-				(path "/ca1c0000-0000-4000-8000-00000000ma01/da764cdd-8caf-4481-b72a-cf9dd25cafa9"
+			(project "calcumaker-mcu"
+				(path "/ca1c0000-0000-4000-8000-00000000ma01/23aa651c-01ea-4ee3-bb12-f879a30c281f"
 					(reference "C12")
 					(unit 1)
@@
 		(pin "2")
 		(instances
-			(project "calcumaker-main"
-				(path "/ca1c0000-0000-4000-8000-00000000ma01/da764cdd-8caf-4481-b72a-cf9dd25cafa9"
+			(project "calcumaker-mcu"
+				(path "/ca1c0000-0000-4000-8000-00000000ma01/23aa651c-01ea-4ee3-bb12-f879a30c281f"
 					(reference "C13")
 					(unit 1)
@@
 		(pin "2")
 		(instances
-			(project "calcumaker-main"
-				(path "/ca1c0000-0000-4000-8000-00000000ma01/da764cdd-8caf-4481-b72a-cf9dd25cafa9"
+			(project "calcumaker-mcu"
+				(path "/ca1c0000-0000-4000-8000-00000000ma01/23aa651c-01ea-4ee3-bb12-f879a30c281f"
 					(reference "C14")
 					(unit 1)
@@
 		(pin "2")
 		(instances
-			(project "calcumaker-main"
-				(path "/ca1c0000-0000-4000-8000-00000000ma01/da764cdd-8caf-4481-b72a-cf9dd25cafa9"
+			(project "calcumaker-mcu"
+				(path "/ca1c0000-0000-4000-8000-00000000ma01/23aa651c-01ea-4ee3-bb12-f879a30c281f"
 					(reference "C15")
 					(unit 1)
@@
 		(pin "2")
 		(instances
-			(project "calcumaker-main"
-				(path "/ca1c0000-0000-4000-8000-00000000ma01/da764cdd-8caf-4481-b72a-cf9dd25cafa9"
+			(project "calcumaker-mcu"
+				(path "/ca1c0000-0000-4000-8000-00000000ma01/23aa651c-01ea-4ee3-bb12-f879a30c281f"
 					(reference "C16")
 					(unit 1)
@@
 		(pin "2")
 		(instances
-			(project "calcumaker-main"
-				(path "/ca1c0000-0000-4000-8000-00000000ma01/da764cdd-8caf-4481-b72a-cf9dd25cafa9"
+			(project "calcumaker-mcu"
+				(path "/ca1c0000-0000-4000-8000-00000000ma01/23aa651c-01ea-4ee3-bb12-f879a30c281f"
 					(reference "C17")
 					(unit 1)
@@
 		(pin "2")
 		(instances
-			(project "calcumaker-main"
-				(path "/ca1c0000-0000-4000-8000-00000000ma01/da764cdd-8caf-4481-b72a-cf9dd25cafa9"
+			(project "calcumaker-mcu"
+				(path "/ca1c0000-0000-4000-8000-00000000ma01/23aa651c-01ea-4ee3-bb12-f879a30c281f"
 					(reference "C18")
 					(unit 1)
@@
 		(pin "2")
 		(instances
-			(project "calcumaker-main"
-				(path "/ca1c0000-0000-4000-8000-00000000ma01/da764cdd-8caf-4481-b72a-cf9dd25cafa9"
+			(project "calcumaker-mcu"
+				(path "/ca1c0000-0000-4000-8000-00000000ma01/23aa651c-01ea-4ee3-bb12-f879a30c281f"
 					(reference "C19")
 					(unit 1)
@@
 		(pin "2")
 		(instances
-			(project "calcumaker-main"
-				(path "/ca1c0000-0000-4000-8000-00000000ma01/da764cdd-8caf-4481-b72a-cf9dd25cafa9"
+			(project "calcumaker-mcu"
+				(path "/ca1c0000-0000-4000-8000-00000000ma01/23aa651c-01ea-4ee3-bb12-f879a30c281f"
 					(reference "C20")
 					(unit 1)
@@
 		(pin "2")
 		(instances
-			(project "calcumaker-main"
-				(path "/ca1c0000-0000-4000-8000-00000000ma01/da764cdd-8caf-4481-b72a-cf9dd25cafa9"
+			(project "calcumaker-mcu"
+				(path "/ca1c0000-0000-4000-8000-00000000ma01/23aa651c-01ea-4ee3-bb12-f879a30c281f"
 					(reference "C21")
 					(unit 1)
@@
 		(pin "2")
 		(instances
-			(project "calcumaker-main"
-				(path "/ca1c0000-0000-4000-8000-00000000ma01/da764cdd-8caf-4481-b72a-cf9dd25cafa9"
+			(project "calcumaker-mcu"
+				(path "/ca1c0000-0000-4000-8000-00000000ma01/23aa651c-01ea-4ee3-bb12-f879a30c281f"
 					(reference "R8")
 					(unit 1)
@@
 		(pin "2")
 		(instances
-			(project "calcumaker-main"
-				(path "/ca1c0000-0000-4000-8000-00000000ma01/da764cdd-8caf-4481-b72a-cf9dd25cafa9"
+			(project "calcumaker-mcu"
+				(path "/ca1c0000-0000-4000-8000-00000000ma01/23aa651c-01ea-4ee3-bb12-f879a30c281f"
 					(reference "C22")
 					(unit 1)
@@
 		(pin "2")
 		(instances
-			(project "calcumaker-main"
-				(path "/ca1c0000-0000-4000-8000-00000000ma01/da764cdd-8caf-4481-b72a-cf9dd25cafa9"
+			(project "calcumaker-mcu"
+				(path "/ca1c0000-0000-4000-8000-00000000ma01/23aa651c-01ea-4ee3-bb12-f879a30c281f"
 					(reference "C23")
 					(unit 1)
@@
 		)
 	)
-	(text "Calcumaker 16 main — MCU core (U1 STM32U575ZGTx, LQFP-144). POWER: VDD pins -> +3V3 (5x 100nF C12-C16 + C17 10uF bulk); VDDA/VREF+ -> C18 1uF + C19 100nF; VDDUSB -> C20 100nF; EP/VSS -> GND. VCORE: choose LDO or internal SMPS — SMPS needs an inductor on VLXSMPS + VDD12; C22/C23 are VCAP placeholders (set per mode, datasheet). RESET/BOOT: NRST + C21 100nF; BOOT0 -> R8 10k to GND. OFF-SHEET: USB PA11/PA12 -> PSU ESD; SWD PA13/PA14 + NRST -> Programming; LSE OSC32_IN/OUT -> Clock; display bus (CLK+DIN1/2/3) + DISP_PWR_EN -> DisplayIF; 5 rows + 10 cols -> Keypad (one col -> EXTI wake)."
+	(text "Calcumaker 16 main — MCU core (U1 STM32U575ZGTx, LQFP-144). POWER: VDD pins -> +3V3 (5x 100nF C12-C16 + C17 10uF bulk); VDDA/VREF+ -> C18 1uF + C19 100nF; VDDUSB -> C20 100nF; EP/VSS -> GND. VCORE: choose LDO or internal SMPS — SMPS needs an inductor on VLXSMPS + VDD12; C22/C23 are VCAP placeholders (set per mode, datasheet). RESET/BOOT: NRST + C21 100nF; BOOT0 -> R8 10k to GND. OFF-SHEET: USB PA11/PA12 -> PSU ESD; SWD PA13/PA14 + NRST -> Programming; LSE OSC32_IN/OUT -> Clock; display bus (CLK+DIN1/2/3) + DISP_PWR_EN -> DisplayIF; 5 rows + 10 cols + 5 annunciator drives -> KeyboardIF mezzanine J5 (one col -> EXTI wake)."
 		(exclude_from_sim no)
 		(at 15.00 150.00 0)

Commit message: docs: accuracy cleanup across README/DESIGN/PARTS + firmware/schgen comments
Sweep the docs and code comments to the three-board reality. Reviewed for
accuracy against the schematics/parts — no factual fixes were needed; this
also corrected several stale spots left over from the split:

- README / DESIGN.md / PARTS.md / reference: three-board split, 0.5mm FFC
  display link, Hirose DF40 mezzanine, STM32G0 keyboard scanner; drop stale
  "main board" phrasing; populate reference/README.md's datasheet table with
  the real parts (STM32G031K8U6, TM1640, FJ5161AH, AFC01-S12FCA-00 + GCT FFC,
  DF40C-10DS/DP).
- DESIGN.md Annunciators corrected to the keyboard board (D51-55 / R1-5,
  driven by the keyboard G0); Open Questions renumbered sequentially.
- firmware comments (keypad.rs / main.rs / Cargo.toml / README): keyboard-event
  intake over the mezzanine link + wake on KB_IRQ; fixed the wrong "host-tested
  with rug" note (it is the gmp-mpfr-nostd FFI). Comment-only, no logic change.
- schgen + .kicad_sch notes: "main" -> "MCU board", FFC/mezzanine references,
  TPS61022/MCU "no custom symbol".

All three boards still pass the structure check (mcu 52 / keyboard 119 /
display 60 components, no duplicate refs); the generator still compiles.

Co-Authored-By: Claude Opus 4.8 (1M context) <noreply@anthropic.com>
Other:
- note added: "Calcumaker 16 MCU board — MCU core (U1 STM32U575ZGTx, LQFP-144). POWER: VDD pins -> +3V3 (5x 100nF C12-C16 + C17 10uF bulk); VDDA/VREF+ -> C18 1uF + C19 100nF; VDDUSB -> C20 100nF; EP/VSS -> GND. VCORE: choose LDO or internal SMPS — SMPS needs an inductor on VLXSMPS + VDD12; C22/C23 are VCAP placeholders (set per mode, datasheet). RESET/BOOT: NRST + C21 100nF; BOOT0 -> R8 10k to GND. OFF-SHEET: U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"
- note removed: "Calcumaker 16 main — MCU core (U1 STM32U575ZGTx, LQFP-144). POWER: VDD pins -> +3V3 (5x 100nF C12-C16 + C17 10uF bulk); VDDA/VREF+ -> C18 1uF + C19 100nF; VDDUSB -> C20 100nF; EP/VSS -> GND. VCORE: choose LDO or internal SMPS — SMPS needs an inductor on VLXSMPS + VDD12; C22/C23 are VCAP placeholders (set per mode, datasheet). RESET/BOOT: NRST + C21 100nF; BOOT0 -> R8 10k to GND. OFF-SHEET: USB PA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"
Changed lines of the file:
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@@
 		)
 	)
-	(text "Calcumaker 16 main — MCU core (U1 STM32U575ZGTx, LQFP-144). POWER: VDD pins -> +3V3 (5x 100nF C12-C16 + C17 10uF bulk); VDDA/VREF+ -> C18 1uF + C19 100nF; VDDUSB -> C20 100nF; EP/VSS -> GND. VCORE: choose LDO or internal SMPS — SMPS needs an inductor on VLXSMPS + VDD12; C22/C23 are VCAP placeholders (set per mode, datasheet). RESET/BOOT: NRST + C21 100nF; BOOT0 -> R8 10k to GND. OFF-SHEET: USB PA11/PA12 -> PSU ESD; SWD PA13/PA14 + NRST -> Programming; LSE OSC32_IN/OUT -> Clock; display bus (CLK+DIN1/2/3) + DISP_PWR_EN -> DisplayIF; 5 rows + 10 cols + 5 annunciator drives -> KeyboardIF mezzanine J5 (one col -> EXTI wake)."
+	(text "Calcumaker 16 MCU board — MCU core (U1 STM32U575ZGTx, LQFP-144). POWER: VDD pins -> +3V3 (5x 100nF C12-C16 + C17 10uF bulk); VDDA/VREF+ -> C18 1uF + C19 100nF; VDDUSB -> C20 100nF; EP/VSS -> GND. VCORE: choose LDO or internal SMPS — SMPS needs an inductor on VLXSMPS + VDD12; C22/C23 are VCAP placeholders (set per mode, datasheet). RESET/BOOT: NRST + C21 100nF; BOOT0 -> R8 10k to GND. OFF-SHEET: USB PA11/PA12 -> PSU ESD; SWD PA13/PA14 + NRST -> Programming; LSE OSC32_IN/OUT -> Clock; display bus (CLK+DIN1/2/3) + DISP_PWR_EN -> DisplayIF; keyboard-board link (I2C+UART+KB_IRQ/NRST/BOOT0) -> KeyboardIF mezzanine J5."
 		(exclude_from_sim no)
 		(at 15.00 150.00 0)
