File: hardware/calcumaker-mcu/mcu.kicad_sch (KiCad schematic)
At the start: 14 parts, among them U1 STM32U575ZGT6

Commit message: hardware: 3-board split (MCU + keyboard + display), wired display, real connectors (#1)
* hardware: 3-board split (MCU + keyboard + display), wired display, real connectors

Split the single logic board into three, wire the display as a KiCad
multi-channel design, and settle every interconnect on real, in-stock parts.

Three-board split (was two):
- Rename calcumaker-main -> calcumaker-mcu (brain/PSU logic board).
- New calcumaker-keyboard board: 50-key Cherry MX matrix + its own
  STM32G031K8U6 scanner (LCSC C432207, UFQFPN-32) + annunciator LEDs,
  mezzanine-stacked above the MCU board. Keyscanning is off the main board;
  only an I2C + UART link + KB_IRQ wake + power cross the mezzanine.

Display board (calcumaker-display):
- Corrected FJ5161AH to a SINGLE-digit 0.56" common-cathode part (C8093) --
  it is NOT a 4-digit module; 48 single digits (16/row x 3), authored symbol
  + 0.56" LTS6760 land. The old 4-digit CC56-12 mapping (and its 3D model)
  was the phantom "clock colon".
- Rebuilt as a KiCad multi-channel design: one reusable display_row.kicad_sch
  (1 TM1640 + 16 digits, fully wired) instantiated x3. Extended kschgen.py
  with wiring primitives + reused-sheet (multi-channel) support.

Connectors (real, verified LCSC / DigiKey parts):
- Display link -> 0.5mm 12P FFC: AFC01-S12FCA-00 (LCSC C262661) on both
  boards; cable = GCT FFC05-TIN 05-12-A-<len>-A-4-06-4-T (DigiKey accessory,
  length TBD). +5V/GND conductors doubled for the display LED current.
- Keyboard mezzanine -> low-profile Hirose DF40 (0.4mm, 2x5, 1.5mm stack):
  DF40C-10DS (C424636) + DF40C-10DP (C424635) -- dedicated KiCad footprint
  + 3D model, unlike the datasheet-less generic parts first considered.

Low-power & wake documented (two Stop domains; keypress -> G0 EXTI wake ->
KB_IRQ -> U575 WKUP; G0 also wakes on I2C address-match). calcumaker-core
is unchanged -- App still consumes (row,col).

All three boards generate + pass the structure check (mcu 52 / keyboard 119 /
display 60 compo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
Other:
- note added: "Calcumaker 16 MCU board — MCU core (U1 STM32U575ZGTx, LQFP-144). POWER: VDD pins -> +3V3 (5x 100nF C12-C16 + C17 10uF bulk); VDDA/VREF+ -> C18 1uF + C19 100nF; VDDUSB -> C20 100nF; EP/VSS -> GND. VCORE: choose LDO or internal SMPS — SMPS needs an inductor on VLXSMPS + VDD12; C22/C23 are VCAP placeholders (set per mode, datasheet). RESET/BOOT: NRST + C21 100nF; BOOT0 -> R8 10k to GND. OFF-SHEET: U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"
- note removed: "Calcumaker 16 main — MCU core (U1 STM32U575ZGTx, LQFP-144). POWER: VDD pins -> +3V3 (5x 100nF C12-C16 + C17 10uF bulk); VDDA/VREF+ -> C18 1uF + C19 100nF; VDDUSB -> C20 100nF; EP/VSS -> GND. VCORE: choose LDO or internal SMPS — SMPS needs an inductor on VLXSMPS + VDD12; C22/C23 are VCAP placeholders (set per mode, datasheet). RESET/BOOT: NRST + C21 100nF; BOOT0 -> R8 10k to GND. OFF-SHEET: USB PA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"
- title: Calcumaker 16 — Main — MCU core (STM32U575) -> Calcumaker 16 — MCU — MCU core (STM32U575)
Changed lines of the file:
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@@
 	(paper "A3")
 	(title_block
-		(title "Calcumaker 16 — Main — MCU core (STM32U575)")
-		(date "2026-06-21")
-		(rev "0.1")
+		(title "Calcumaker 16 — MCU — MCU core (STM32U575)")
+		(date "2026-07-05")
+		(rev "0.2")
 		(company "calcumaker authors")
 	)
@@
 		(pin "144")
 		(instances
-			(project "calcumaker-main"
-				(path "/ca1c0000-0000-4000-8000-00000000ma01/da764cdd-8caf-4481-b72a-cf9dd25cafa9"
+			(project "calcumaker-mcu"
+				(path "/ca1c0000-0000-4000-8000-00000000ma01/23aa651c-01ea-4ee3-bb12-f879a30c281f"
 					(reference "U1")
 					(unit 1)
@@
 		(pin "2")
 		(instances
-			(project "calcumaker-main"
-				(path "/ca1c0000-0000-4000-8000-00000000ma01/da764cdd-8caf-4481-b72a-cf9dd25cafa9"
+			(project "calcumaker-mcu"
+				(path "/ca1c0000-0000-4000-8000-00000000ma01/23aa651c-01ea-4ee3-bb12-f879a30c281f"
 					(reference "C12")
 					(unit 1)
@@
 		(pin "2")
 		(instances
-			(project "calcumaker-main"
-				(path "/ca1c0000-0000-4000-8000-00000000ma01/da764cdd-8caf-4481-b72a-cf9dd25cafa9"
+			(project "calcumaker-mcu"
+				(path "/ca1c0000-0000-4000-8000-00000000ma01/23aa651c-01ea-4ee3-bb12-f879a30c281f"
 					(reference "C13")
 					(unit 1)
@@
 		(pin "2")
 		(instances
-			(project "calcumaker-main"
-				(path "/ca1c0000-0000-4000-8000-00000000ma01/da764cdd-8caf-4481-b72a-cf9dd25cafa9"
+			(project "calcumaker-mcu"
+				(path "/ca1c0000-0000-4000-8000-00000000ma01/23aa651c-01ea-4ee3-bb12-f879a30c281f"
 					(reference "C14")
 					(unit 1)
@@
 		(pin "2")
 		(instances
-			(project "calcumaker-main"
-				(path "/ca1c0000-0000-4000-8000-00000000ma01/da764cdd-8caf-4481-b72a-cf9dd25cafa9"
+			(project "calcumaker-mcu"
+				(path "/ca1c0000-0000-4000-8000-00000000ma01/23aa651c-01ea-4ee3-bb12-f879a30c281f"
 					(reference "C15")
 					(unit 1)
@@
 		(pin "2")
 		(instances
-			(project "calcumaker-main"
-				(path "/ca1c0000-0000-4000-8000-00000000ma01/da764cdd-8caf-4481-b72a-cf9dd25cafa9"
+			(project "calcumaker-mcu"
+				(path "/ca1c0000-0000-4000-8000-00000000ma01/23aa651c-01ea-4ee3-bb12-f879a30c281f"
 					(reference "C16")
 					(unit 1)
@@
 		(pin "2")
 		(instances
-			(project "calcumaker-main"
-				(path "/ca1c0000-0000-4000-8000-00000000ma01/da764cdd-8caf-4481-b72a-cf9dd25cafa9"
+			(project "calcumaker-mcu"
+				(path "/ca1c0000-0000-4000-8000-00000000ma01/23aa651c-01ea-4ee3-bb12-f879a30c281f"
 					(reference "C17")
 					(unit 1)
@@
 		(pin "2")
 		(instances
-			(project "calcumaker-main"
-				(path "/ca1c0000-0000-4000-8000-00000000ma01/da764cdd-8caf-4481-b72a-cf9dd25cafa9"
+			(project "calcumaker-mcu"
+				(path "/ca1c0000-0000-4000-8000-00000000ma01/23aa651c-01ea-4ee3-bb12-f879a30c281f"
 					(reference "C18")
 					(unit 1)
@@
 		(pin "2")
 		(instances
-			(project "calcumaker-main"
-				(path "/ca1c0000-0000-4000-8000-00000000ma01/da764cdd-8caf-4481-b72a-cf9dd25cafa9"
+			(project "calcumaker-mcu"
+				(path "/ca1c0000-0000-4000-8000-00000000ma01/23aa651c-01ea-4ee3-bb12-f879a30c281f"
 					(reference "C19")
 					(unit 1)
@@
 		(pin "2")
 		(instances
-			(project "calcumaker-main"
-				(path "/ca1c0000-0000-4000-8000-00000000ma01/da764cdd-8caf-4481-b72a-cf9dd25cafa9"
+			(project "calcumaker-mcu"
+				(path "/ca1c0000-0000-4000-8000-00000000ma01/23aa651c-01ea-4ee3-bb12-f879a30c281f"
 					(reference "C20")
 					(unit 1)
@@
 		(pin "2")
 		(instances
-			(project "calcumaker-main"
-				(path "/ca1c0000-0000-4000-8000-00000000ma01/da764cdd-8caf-4481-b72a-cf9dd25cafa9"
+			(project "calcumaker-mcu"
+				(path "/ca1c0000-0000-4000-8000-00000000ma01/23aa651c-01ea-4ee3-bb12-f879a30c281f"
 					(reference "C21")
 					(unit 1)
@@
 		(pin "2")
 		(instances
-			(project "calcumaker-main"
-				(path "/ca1c0000-0000-4000-8000-00000000ma01/da764cdd-8caf-4481-b72a-cf9dd25cafa9"
+			(project "calcumaker-mcu"
+				(path "/ca1c0000-0000-4000-8000-00000000ma01/23aa651c-01ea-4ee3-bb12-f879a30c281f"
 					(reference "R8")
 					(unit 1)
@@
 		(pin "2")
 		(instances
-			(project "calcumaker-main"
-				(path "/ca1c0000-0000-4000-8000-00000000ma01/da764cdd-8caf-4481-b72a-cf9dd25cafa9"
+			(project "calcumaker-mcu"
+				(path "/ca1c0000-0000-4000-8000-00000000ma01/23aa651c-01ea-4ee3-bb12-f879a30c281f"
 					(reference "C22")
 					(unit 1)
@@
 		(pin "2")
 		(instances
-			(project "calcumaker-main"
-				(path "/ca1c0000-0000-4000-8000-00000000ma01/da764cdd-8caf-4481-b72a-cf9dd25cafa9"
+			(project "calcumaker-mcu"
+				(path "/ca1c0000-0000-4000-8000-00000000ma01/23aa651c-01ea-4ee3-bb12-f879a30c281f"
 					(reference "C23")
 					(unit 1)
@@
 		)
 	)
-	(text "Calcumaker 16 main — MCU core (U1 STM32U575ZGTx, LQFP-144). POWER: VDD pins -> +3V3 (5x 100nF C12-C16 + C17 10uF bulk); VDDA/VREF+ -> C18 1uF + C19 100nF; VDDUSB -> C20 100nF; EP/VSS -> GND. VCORE: choose LDO or internal SMPS — SMPS needs an inductor on VLXSMPS + VDD12; C22/C23 are VCAP placeholders (set per mode, datasheet). RESET/BOOT: NRST + C21 100nF; BOOT0 -> R8 10k to GND. OFF-SHEET: USB PA11/PA12 -> PSU ESD; SWD PA13/PA14 + NRST -> Programming; LSE OSC32_IN/OUT -> Clock; display bus (CLK+DIN1/2/3) + DISP_PWR_EN -> DisplayIF; 5 rows + 10 cols -> Keypad (one col -> EXTI wake)."
+	(text "Calcumaker 16 MCU board — MCU core (U1 STM32U575ZGTx, LQFP-144). POWER: VDD pins -> +3V3 (5x 100nF C12-C16 + C17 10uF bulk); VDDA/VREF+ -> C18 1uF + C19 100nF; VDDUSB -> C20 100nF; EP/VSS -> GND. VCORE: choose LDO or internal SMPS — SMPS needs an inductor on VLXSMPS + VDD12; C22/C23 are VCAP placeholders (set per mode, datasheet). RESET/BOOT: NRST + C21 100nF; BOOT0 -> R8 10k to GND. OFF-SHEET: USB PA11/PA12 -> PSU ESD; SWD PA13/PA14 + NRST -> Programming; LSE OSC32_IN/OUT -> Clock; display bus (CLK+DIN1/2/3) + DISP_PWR_EN -> DisplayIF; keyboard-board link (I2C+UART+KB_IRQ/NRST/BOOT0) -> KeyboardIF mezzanine J5."
 		(exclude_from_sim no)
 		(at 15.00 150.00 0)

Commit message: hardware: MCU -> STM32U575RGT6 (LQFP-64) + 4MB QSPI flash; monospace wiring notes
MCU package + external flash
- Swap U1 STM32U575ZGT6 (LQFP-144) -> STM32U575RGT6 (LQFP-64, LCSC C5270980).
  The firmware links at ~323 KB so 1 MB flash is ample (~3x headroom), and with
  the key matrix scanned off-board the LQFP-64 has enough GPIO — smaller/cheaper.
- Correct the flash size everywhere: the STM32 `G` code = 1 MB (not 2 MB; the
  `I` parts are 2 MB). memory.x FLASH 2048K -> 1024K; .cargo runner -> RGTx.
- Add U7 W25Q32JVSSIQ, a 4 MB (32 Mbit) quad-SPI NOR (LCSC C179173, SOIC-8) on
  OCTOSPI1 as a new QSPIFlash sheet (+ R9 CS# pull-up + C26 decoupling) for
  memory-mapped (XIP) constants + state/program storage.
- mcu board 52 -> 55 components / 7 sheets. Docs (DESIGN.md, PARTS.md, READMEs,
  CLAUDE/AGENTS) updated; availability ladder now lists RGT6/VGT6/ZGT6.

Monospace, multi-line schematic wiring notes
- kschgen text_note() now renders notes in a monospace font (Courier New) so
  tables/columns line up; add note_block() + pin_table() helpers.
- Reformat all 14 per-sheet notes into titled, multi-line, aligned blocks —
  connector pinouts as PIN/SIGNAL tables, power/MCU sheets as wiring blocks.

The regenerated schematics carry both changes, so this is one commit. All three
boards regenerate + pass the structure check (mcu 55 / keyboard 119 / display
60, no duplicate refs).

Co-Authored-By: Claude Opus 4.8 (1M context) <noreply@anthropic.com>
Parts:
- removed U1: STM32U575ZGT6, Package_QFP:LQFP-144_20x20mm_P0.5mm, symbol MCU_ST_STM32U5:STM32U575ZGTx
- added U1: STM32U575RGT6, Package_QFP:LQFP-64_10x10mm_P0.5mm, symbol MCU_ST_STM32U5:STM32U575RGTx
Connections:
- new net: U1.18 (VSS), U1.31 (VSS), U1.47 (VSS), U1.63 (VSS)
Other:
- note added: "MCU CORE - U1 STM32U575RGT6 (LQFP-64, Cortex-M33) Smaller pkg now the key matrix scans on the keyboard G0, not here. POWER VDD (each pin) -> +3V3 C12-C16 100nF + C17 10uF bulk (LQFP-64 has fewer VDD than the 5 caps; spares are extra bypass, trim @ layout) VDDA / VREF+ -> +3V3 C18 1uF + C19 100nF VDDUSB -> +3V3 C20 100nF VSS / EP -> GND VCORE -> LDO or internal SMPS (SMPS: L on VLXSMPS + VDD12); C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"
- note removed: "Calcumaker 16 MCU board — MCU core (U1 STM32U575ZGTx, LQFP-144). POWER: VDD pins -> +3V3 (5x 100nF C12-C16 + C17 10uF bulk); VDDA/VREF+ -> C18 1uF + C19 100nF; VDDUSB -> C20 100nF; EP/VSS -> GND. VCORE: choose LDO or internal SMPS — SMPS needs an inductor on VLXSMPS + VDD12; C22/C23 are VCAP placeholders (set per mode, datasheet). RESET/BOOT: NRST + C21 100nF; BOOT0 -> R8 10k to GND. OFF-SHEET: U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"
Changed lines of the file:
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@@
 	(title_block
 		(title "Calcumaker 16 — MCU — MCU core (STM32U575)")
-		(date "2026-07-05")
-		(rev "0.2")
+		(date "2026-07-06")
+		(rev "0.3")
 		(company "calcumaker authors")
 	)
 	(symbol
-		(lib_id "MCU_ST_STM32U5:STM32U575ZGTx")
+		(lib_id "MCU_ST_STM32U5:STM32U575RGTx")
 		(at 45.7200 55.8800 0)
 		(unit 1)
@@
 			(effects (font (size 1.27 1.27)) (justify left))
 		)
-		(property "Value" "STM32U575ZGT6"
+		(property "Value" "STM32U575RGT6"
 			(at 49.5300 58.4200 0)
 			(effects (font (size 1.27 1.27)) (justify left))
 		)
-		(property "Footprint" "Package_QFP:LQFP-144_20x20mm_P0.5mm"
+		(property "Footprint" "Package_QFP:LQFP-64_10x10mm_P0.5mm"
 			(at 45.7200 55.8800 0)
 			(effects (font (size 1.27 1.27))) (hide yes)
@@
 			(effects (font (size 1.27 1.27))) (hide yes)
 		)
-		(property "LCSC" "C5271004"
+		(property "LCSC" "C5270980"
 			(at 45.7200 55.8800 0)
 			(effects (font (size 1.27 1.27))) (hide yes)
 		)
-		(property "MPN" "STM32U575ZGT6"
+		(property "MPN" "STM32U575RGT6"
 			(at 45.7200 55.8800 0)
 			(effects (font (size 1.27 1.27))) (hide yes)
@@
 		(pin "63")
 		(pin "64")
-		(pin "65")
-		(pin "66")
-		(pin "67")
-		(pin "68")
-		(pin "69")
-		(pin "70")
-		(pin "71")
-		(pin "72")
-		(pin "73")
-		(pin "74")
-		(pin "75")
-		(pin "76")
-		(pin "77")
-		(pin "78")
-		(pin "79")
-		(pin "80")
-		(pin "81")
-		(pin "82")
-		(pin "83")
-		(pin "84")
-		(pin "85")
-		(pin "86")
-		(pin "87")
-		(pin "88")
-		(pin "89")
-		(pin "90")
-		(pin "91")
-		(pin "92")
-		(pin "93")
-		(pin "94")
-		(pin "95")
-		(pin "96")
-		(pin "97")
-		(pin "98")
-		(pin "99")
-		(pin "100")
-		(pin "101")
-		(pin "102")
-		(pin "103")
-		(pin "104")
-		(pin "105")
-		(pin "106")
-		(pin "107")
-		(pin "108")
-		(pin "109")
-		(pin "110")
-		(pin "111")
-		(pin "112")
-		(pin "113")
-		(pin "114")
-		(pin "115")
-		(pin "116")
-		(pin "117")
-		(pin "118")
-		(pin "119")
-		(pin "120")
-		(pin "121")
-		(pin "122")
-		(pin "123")
-		(pin "124")
-		(pin "125")
-		(pin "126")
-		(pin "127")
-		(pin "128")
-		(pin "129")
-		(pin "130")
-		(pin "131")
-		(pin "132")
-		(pin "133")
-		(pin "134")
-		(pin "135")
-		(pin "136")
-		(pin "137")
-		(pin "138")
-		(pin "139")
-		(pin "140")
-		(pin "141")
-		(pin "142")
-		(pin "143")
-		(pin "144")
-		(instances
-			(project "calcumaker-mcu"
-				(path "/ca1c0000-0000-4000-8000-00000000ma01/23aa651c-01ea-4ee3-bb12-f879a30c281f"
+		(instances
+			(project "calcumaker-mcu"
+				(path "/ca1c0000-0000-4000-8000-00000000ma01/77d1e065-260c-4e9e-b78f-2ca7ebacff25"
 					(reference "U1")
 					(unit 1)
@@
 		(instances
 			(project "calcumaker-mcu"
-				(path "/ca1c0000-0000-4000-8000-00000000ma01/23aa651c-01ea-4ee3-bb12-f879a30c281f"
+				(path "/ca1c0000-0000-4000-8000-00000000ma01/77d1e065-260c-4e9e-b78f-2ca7ebacff25"
 					(reference "C12")
 					(unit 1)
@@
 		(instances
 			(project "calcumaker-mcu"
-				(path "/ca1c0000-0000-4000-8000-00000000ma01/23aa651c-01ea-4ee3-bb12-f879a30c281f"
+				(path "/ca1c0000-0000-4000-8000-00000000ma01/77d1e065-260c-4e9e-b78f-2ca7ebacff25"
 					(reference "C13")
 					(unit 1)
@@
 		(instances
 			(project "calcumaker-mcu"
-				(path "/ca1c0000-0000-4000-8000-00000000ma01/23aa651c-01ea-4ee3-bb12-f879a30c281f"
+				(path "/ca1c0000-0000-4000-8000-00000000ma01/77d1e065-260c-4e9e-b78f-2ca7ebacff25"
 					(reference "C14")
 					(unit 1)
@@
 		(instances
 			(project "calcumaker-mcu"
-				(path "/ca1c0000-0000-4000-8000-00000000ma01/23aa651c-01ea-4ee3-bb12-f879a30c281f"
+				(path "/ca1c0000-0000-4000-8000-00000000ma01/77d1e065-260c-4e9e-b78f-2ca7ebacff25"
 					(reference "C15")
 					(unit 1)
@@
 		(instances
 			(project "calcumaker-mcu"
-				(path "/ca1c0000-0000-4000-8000-00000000ma01/23aa651c-01ea-4ee3-bb12-f879a30c281f"
+				(path "/ca1c0000-0000-4000-8000-00000000ma01/77d1e065-260c-4e9e-b78f-2ca7ebacff25"
 					(reference "C16")
 					(unit 1)
@@
 		(instances
 			(project "calcumaker-mcu"
-				(path "/ca1c0000-0000-4000-8000-00000000ma01/23aa651c-01ea-4ee3-bb12-f879a30c281f"
+				(path "/ca1c0000-0000-4000-8000-00000000ma01/77d1e065-260c-4e9e-b78f-2ca7ebacff25"
 					(reference "C17")
 					(unit 1)
@@
 		(instances
 			(project "calcumaker-mcu"
-				(path "/ca1c0000-0000-4000-8000-00000000ma01/23aa651c-01ea-4ee3-bb12-f879a30c281f"
+				(path "/ca1c0000-0000-4000-8000-00000000ma01/77d1e065-260c-4e9e-b78f-2ca7ebacff25"
 					(reference "C18")
 					(unit 1)
@@
 		(instances
 			(project "calcumaker-mcu"
-				(path "/ca1c0000-0000-4000-8000-00000000ma01/23aa651c-01ea-4ee3-bb12-f879a30c281f"
+				(path "/ca1c0000-0000-4000-8000-00000000ma01/77d1e065-260c-4e9e-b78f-2ca7ebacff25"
 					(reference "C19")
 					(unit 1)
@@
 		(instances
 			(project "calcumaker-mcu"
-				(path "/ca1c0000-0000-4000-8000-00000000ma01/23aa651c-01ea-4ee3-bb12-f879a30c281f"
+				(path "/ca1c0000-0000-4000-8000-00000000ma01/77d1e065-260c-4e9e-b78f-2ca7ebacff25"
 					(reference "C20")
 					(unit 1)
@@
 		(instances
 			(project "calcumaker-mcu"
-				(path "/ca1c0000-0000-4000-8000-00000000ma01/23aa651c-01ea-4ee3-bb12-f879a30c281f"
+				(path "/ca1c0000-0000-4000-8000-00000000ma01/77d1e065-260c-4e9e-b78f-2ca7ebacff25"
 					(reference "C21")
 					(unit 1)
@@
 		(instances
 			(project "calcumaker-mcu"
-				(path "/ca1c0000-0000-4000-8000-00000000ma01/23aa651c-01ea-4ee3-bb12-f879a30c281f"
+				(path "/ca1c0000-0000-4000-8000-00000000ma01/77d1e065-260c-4e9e-b78f-2ca7ebacff25"
 					(reference "R8")
 					(unit 1)
@@
 		(instances
 			(project "calcumaker-mcu"
-				(path "/ca1c0000-0000-4000-8000-00000000ma01/23aa651c-01ea-4ee3-bb12-f879a30c281f"
+				(path "/ca1c0000-0000-4000-8000-00000000ma01/77d1e065-260c-4e9e-b78f-2ca7ebacff25"
 					(reference "C22")
 					(unit 1)
@@
 		(instances
 			(project "calcumaker-mcu"
-				(path "/ca1c0000-0000-4000-8000-00000000ma01/23aa651c-01ea-4ee3-bb12-f879a30c281f"
+				(path "/ca1c0000-0000-4000-8000-00000000ma01/77d1e065-260c-4e9e-b78f-2ca7ebacff25"
 					(reference "C23")
 					(unit 1)
@@
 		)
 	)
-	(text "Calcumaker 16 MCU board — MCU core (U1 STM32U575ZGTx, LQFP-144). POWER: VDD pins -> +3V3 (5x 100nF C12-C16 + C17 10uF bulk); VDDA/VREF+ -> C18 1uF + C19 100nF; VDDUSB -> C20 100nF; EP/VSS -> GND. VCORE: choose LDO or internal SMPS — SMPS needs an inductor on VLXSMPS + VDD12; C22/C23 are VCAP placeholders (set per mode, datasheet). RESET/BOOT: NRST + C21 100nF; BOOT0 -> R8 10k to GND. OFF-SHEET: USB PA11/PA12 -> PSU ESD; SWD PA13/PA14 + NRST -> Programming; LSE OSC32_IN/OUT -> Clock; display bus (CLK+DIN1/2/3) + DISP_PWR_EN -> DisplayIF; keyboard-board link (I2C+UART+KB_IRQ/NRST/BOOT0) -> KeyboardIF mezzanine J5."
+	(text "MCU CORE  -  U1  STM32U575RGT6   (LQFP-64, Cortex-M33)\nSmaller pkg now the key matrix scans on the keyboard G0, not here.\n\nPOWER\n  VDD (each pin) -> +3V3   C12-C16 100nF + C17 10uF bulk\n                           (LQFP-64 has fewer VDD than the 5 caps;\n                            spares are extra bypass, trim @ layout)\n  VDDA / VREF+   -> +3V3   C18 1uF + C19 100nF\n  VDDUSB         -> +3V3   C20 100nF\n  VSS / EP       -> GND\n  VCORE          -> LDO or internal SMPS (SMPS: L on VLXSMPS + VDD12);\n                    C22/C23 = VCAP placeholders (set per mode)\nRESET / BOOT\n  NRST -> C21 100nF          BOOT0 -> R8 10k to GND\n\nOFF-SHEET\n  USB   PA11/PA12  -> PSU ESD (U3)\n  SWD   PA13/PA14  -> Programming J4  (+ NRST)\n  LSE   OSC32      -> Clock Y1\n  DISP  CLK+DIN1-3 + DISP_PWR_EN   -> DisplayIF\n  KBD   I2C+UART+KB_IRQ/NRST/BOOT0 -> KeyboardIF J5\n  QSPI  OCTOSPI1 CLK/NCS/IO0-3     -> QSPIFlash U7\n\nVerify OCTOSPI1 pin mapping is available on LQFP-64."
 		(exclude_from_sim no)
 		(at 15.00 150.00 0)
-		(effects (font (size 1.5 1.5)) (justify left top))
+		(effects (font (face "Courier New") (size 1.27 1.27)) (justify left top))
 	)
 	(sheet_instances
