File: hardware/calcumaker-mcu/mcu.kicad_sch (KiCad schematic)
At the start: 20 parts, among them J3 TO DISPLAY (unified SPI FFC), J4 SWD TC2030-NL, J7 VSYS -> matrix LED pwr, U1 STM32U575RGT6, Y1 32.768kHz

Commit message: Checkpoint
Changed lines of the file:
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@@
 		)
 	)
-	(text "MCU CORE  -  U1  STM32U575RGT6   (LQFP-64, Cortex-M33)\nSmaller pkg now the key matrix scans on the keyboard G0, not here.\n\nPOWER\n  VDD (each pin) -> +3V3   C12-C16 100nF + C17 10uF bulk\n                           (LQFP-64 has fewer VDD than the 5 caps;\n                            spares are extra bypass, trim @ layout)\n  VDDA / VREF+   -> +3V3   C18 1uF + C19 100nF\n  VDDUSB         -> +3V3   C20 100nF\n  VSS / EP       -> GND\n  VCORE          -> LDO or internal SMPS (SMPS: L on VLXSMPS + VDD12);\n                    C22/C23 = VCAP placeholders (set per mode)\nRESET / BOOT\n  NRST -> C21 100nF          BOOT0 -> R8 10k to GND\n\nPIN MAP  (verified vs the ST CubeMX pin DB for LQFP-64)\n  OCTOSPI1 -> U7      OCTOSPIM Port 1; IO0-3 forced, 1 pin each\n    CLK  PB10 AF10 p29      IO0  PB1  AF10 p27\n    NCS  PA4  AF3  p20      IO1  PB0  AF10 p26\n                            IO2  PA7  AF10 p23\n                            IO3  PA6  AF10 p22\n  SPI1 -> display J3  (PA6/PA7 are QSPI now; the FFC has no MISO)\n    SCK  PA5  AF5  p21      MOSI PB5  AF5  p57\n    CS   PA15 AF5  p50      (or any GPIO)\n  USART2 -> keyboard   TX PA2 p16 / RX PA3 p17   AF7\n  I2C1   -> keyboard   SCL PB6 p58 / SDA PB7 p59 AF4\n\nON THIS SHEET  (Clock / Programming / DisplayIF merged in here)\n  SWD   PA13/PA14 (+ PB3 SWO)      -> J4 Tag-Connect (+ NRST)\n  LSE   PC14/PC15 OSC32            -> Y1 + C24/C25\n  DISP  SPI1 + DISP_IRQ/NRST/BOOT  -> J3 FFC ; J7 VSYS outlet\n\nOFF-SHEET\n  USB   PA11/PA12                     -> PSU ESD (U3)\n  KBD   I2C1+USART2+KB_IRQ/NRST/BOOT0 -> KeyboardIF J5/J6\n  QSPI  OCTOSPI1 CLK/NCS/IO0-3        -> QSPIFlash U7\n\nKB_IRQ must land on a WKUP pin (keypress wake from Stop) -- still open."
+	(text "MCU CORE  -  U1  STM32U575RGT6   (LQFP-64, Cortex-M33)\nSmaller pkg now the key matrix scans on the keyboard G0, not here.\n\nPOWER\n  VDD (each pin) -> +3V3   C12-C16 100nF + C17 10uF bulk\n                           (LQFP-64 has fewer VDD than the 5 caps;\n                            spares are extra bypass, trim @ layout)\n  VDDA / VREF+   -> +3V3   C18 1uF + C19 100nF\n  VDDUSB         -> +3V3   C20 100nF\n  VSS / EP       -> GND\n  VCORE          -> LDO or internal SMPS (SMPS: L on VLXSMPS + VDD12);\n                    C22/C23 = VCAP placeholders (set per mode)\nRESET / BOOT\n  NRST -> C21 100nF          BOOT0 -> R8 10k to GND\n\nPIN MAP  (verified vs the ST CubeMX pin DB for LQFP-64)\n  OCTOSPI1 -> U7      OCTOSPIM Port 1; IO0-3 forced, 1 pin each\n    CLK  PB10 AF10 p29      IO0  PB1  AF10 p27\n    NCS  PA4  AF3  p20      IO1  PB0  AF10 p26\n                            IO2  PA7  AF10 p23\n                            IO3  PA6  AF10 p22\n  SPI1 -> display J3  (PA6/PA7 are QSPI now; the FFC has no MISO)\n    SCK  PA5  AF5  p21      MOSI PB5  AF5  p57\n    CS   PA8       p41      (plain GPIO -- MOVED off PA15, now UCPD1_CC1)\n  UCPD1  -> USB-C CC   CC1 PA15 p50 / CC2 PB15 p63   (dedicated analog, NO AF\n                       alt -- this is why SPI1 CS had to move.  Rd is INTERNAL:\n                       no 5.1k parts.  DBCC1/DBCC2 UNUSED -- the TCPP01 DB/ pin\n                       is a plain GPIO -- so PB5 stays SPI1 MOSI.)\n                       UCPD BMC PHY also runs the 12V PD sink negotiation.\n  USART2 -> keyboard   TX PA2 p16 / RX PA3 p17   AF7\n  I2C1   -> keyboard + CHARGER + FUEL GAUGE   SCL PB6 p58 / SDA PB7 p59 AF4\n                       (shared bus: BQ25601 = 0x6B, MAX17048 = 0x36, kbd G0 --\n                        no address clashes)\n\nON THIS SHEET  (Clock / Programming / DisplayIF merged in here)\n  SWD   PA13/PA14 (+ PB3 SWO)      -> J4 Tag-Connect (+ NRST)\n  LSE   PC14/PC15 OSC32            -> Y1 + C24/C25\n  DISP  SPI1 + DISP_IRQ/NRST/BOOT  -> J3 FFC ; J7 VSYS outlet\n\nOFF-SHEET\n  USB   PA11/PA12                     -> PSU ESD (U3)\n  CC    PA15/PB15 (UCPD1)             -> PSU TCPP01 (U5) -> USB-C CC1/CC2\n  TCPP  TCPP01_EN / TCPP01_DB / TCPP01_FLT / VBUS_SENSE(ADC) -> PSU U5\n  CHG   I2C1 + CHG_INT/CHG_PG/CHG_CE  -> PSU charger U4\n  GAUGE I2C1 + GAUGE_ALRT (WKUP)      -> PSU MAX17048 U6 -> LOWBAT annunciator\n  KBD   I2C1+USART2+KB_IRQ/NRST/BOOT0 -> KeyboardIF J5/J6\n  QSPI  OCTOSPI1 CLK/NCS/IO0-3        -> QSPIFlash U7\n\nKB_IRQ must land on a WKUP pin (keypress wake from Stop) -- still open."
 		(exclude_from_sim no)
 		(at 15 168.4 0)

Commit message: Wire mainboard and keypad schematics and verify expanded nets
Connect hierarchical interfaces, power/control circuits, debug links, matrix and RGB chains. Correct MCU package pins, diode polarity and power configuration; add bypass components and repeatable KiCad netlist/ERC checks. Document pin maps and remaining physical validation.
Parts:
- added R13, R14: 4.7k, Resistor_SMD:R_0402_1005Metric, symbol Device:R
- C22, C23: value 2.2uF -> 2.2uF 10V low ESR
Connections:
- net VDD is gone; now on net +3V3: U1.13 (VDDA), U1.19 (VDD), U1.32 (VDD), U1.64 (VDD)
- net VDDUSB is gone; now on net +3V3: C20.1, U1.48 (VDDUSB)
- net GND: now also C12.2, C13.2, C14.2, C15.2, C16.2, C17.2, C18.2, C19.2, C21.2, C22.2, C23.2, C24.2, C25.2, J3.12 (Pin_12), J3.3 (Pin_3), J3.4 (Pin_4), J4.5 (GND), J7.2 (Pin_2), R8.2
- net +3V3: now reaches C12.1
- net +3V3: now also C13.1, C14.1, C15.1, C16.1, C17.1, C18.1, C19.1, J3.5 (Pin_5), J4.1 (VCC), U1.1 (VBAT), R13.1, R14.1
- net LSE_IN: now reaches C24.1
- net LSE_IN: now also U1.3 (PC14), Y1.1
- net VSYS: now reaches J3.1 (Pin_1)
- net VSYS: now also J3.2 (Pin_2), J7.1 (Pin_1)
- net DISP_NRST: now reaches J3.10 (Pin_10)
- net DISP_NRST: now also U1.39 (PC8)
- net DISP_BOOT: now reaches J3.11 (Pin_11)
- net DISP_BOOT: now also U1.40 (PC9)
- net SPI_SCLK: now reaches J3.6 (Pin_6)
- net SPI_SCLK: now also U1.21 (PA5)
- net SPI_MOSI: now reaches J3.7 (Pin_7)
- net SPI_MOSI: now also U1.57 (PB5)
- net SPI_CS: now reaches J3.8 (Pin_8)
- net SPI_CS: now also U1.41 (PA8)
- net DISP_IRQ: now reaches J3.9 (Pin_9)
- net DISP_IRQ: now also U1.33 (PB12)
- net LSE_OUT: now reaches C25.1
- net LSE_OUT: now also U1.4 (PC15), Y1.2
- net VCAP: now reaches C23.1
- net VCAP: now also C22.1, U1.30 (VCAP)
- net CHG_INT: now reaches U1.10 (PC2)
- net TCPP01_FLT: now reaches U1.11 (PC3)
- net KB_IRQ: now reaches U1.14 (PA0)
- net UART_TX: now reaches U1.16 (PA2)
- net UART_RX: now reaches U1.17 (PA3)
- net GAUGE_ALRT: now reaches U1.2 (PC13)
- net QSPI_NCS: now reaches U1.20 (PA4)
- net QSPI_IO3: now reaches U1.22 (PA6)
- net QSPI_IO2: now reaches U1.23 (PA7)
- net CHG_PG: now reaches U1.24 (PC4)
- net CHG_CE: now reaches U1.25 (PC5)
- net QSPI_IO1: now reaches U1.26 (PB0)
- net QSPI_IO0: now reaches U1.27 (PB1)
- net QSPI_CLK: now reaches U1.29 (PB10)
- net UCPD_CC2: now reaches U1.36 (PB15)
- net TCPP01_EN: now reaches U1.37 (PC6)
- net TCPP01_DB: now reaches U1.38 (PC7)
- net USB_DM: now reaches U1.44 (PA11)
- net USB_DP: now reaches U1.45 (PA12)
- net SWDIO: now reaches U1.46 (PA13)
- net SWDIO: now also J4.2 (SWDIO)
- net SWCLK: now reaches U1.49 (PA14)
- net SWCLK: now also J4.4 (SWCLK)
- net UCPD_CC1: now reaches U1.50 (PA15)
- net KB_NRST: now reaches U1.51 (PC10)
- net KB_BOOT0: now reaches U1.52 (PC11)
- net SWO: now reaches U1.55 (PB3)
- net SWO: now also J4.6 (SWO)
- net I2C_SCL: now reaches U1.58 (PB6)
- net I2C_SCL: now also R13.2
- net I2C_SDA: now reaches U1.59 (PB7)
- net I2C_SDA: now also R14.2
- net BOOT0: now reaches U1.60 (PH3)
- net BOOT0: now also R8.1
- net NRST: now reaches U1.7 (NRST)
- net NRST: now also C21.1, J4.3 (~{RESET})
- net VBUS_SENSE: now reaches U1.8 (PC0)
- net BAT_SENSE: now reaches U1.9 (PC1)
- no-connect marks 0 -> 13
Other:
- note added: "LSE 32.768 kHz; fit load capacitors for crystal CL + PCB stray."
- note added: "PB15 = pin 36 (CC2); pin 63 is VSS. KB_IRQ PA0/WKUP1; gauge PC13/WKUP2. CHG_INT PC2, TCPP_FLT PC3, DISP_IRQ PB12: distinct EXTI lines. VBAT uses regulated 3V3, never the raw 4.2V cell. Only R13/R14 pull up the shared I2C bus."
- note added: "STM32U575RGT6 / LQFP64 / LDO core supply"
- note added: "VCAP: 2 x 2.2uF, >=10V, combined ESR <20mohm at 3MHz. No 3V3 connection."
- note removed: "CLOCK - LSE 32.768 kHz (Y1 Q13FC13500004, LCSC C32346) Y1.1 -> OSC32_IN (PC14) Y1.2 -> OSC32_OUT (PC15) C24 / C25 -> LSE load caps to GND (12pF shown) Load caps: CL match = 2*(CL - Cstray); trim with the RTC SMOOTHCALIB. Drives the RTC for sleep timing."
- note removed: "MCU CORE - U1 STM32U575RGT6 (LQFP-64, Cortex-M33) Smaller pkg now the key matrix scans on the keyboard G0, not here. POWER VDD (each pin) -> +3V3 C12-C16 100nF + C17 10uF bulk (LQFP-64 has fewer VDD than the 5 caps; spares are extra bypass, trim @ layout) VDDA / VREF+ -> +3V3 C18 1uF + C19 100nF VDDUSB -> +3V3 C20 100nF VSS / EP -> GND VCORE -> LDO or internal SMPS (SMPS: L on VLXSMPS + VDD12); C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"
- note removed: "SWD PROGRAMMING - J4 Tag-Connect TC2030-NL (no-legs pogo pad) Bare land, no part mounted. PIN SIGNAL 1 +3V3 (VTref) 2 SWDIO (PA13) 3 NRST 4 SWCLK (PA14) 5 GND 6 SWO (PB3, opt)"
- note removed: "UNIFIED DISPLAY-MODULE INTERFACE J3 = 0.5mm 12-pos FFC to the display module (AFC01-S12FCA-00, C262661). SAME pinout on BOTH display boards (7-seg + RGB matrix) -> interchangeable. Technology-agnostic: power + SPI 'display intent' + reset/boot. The module MCU (STM32G031 on 7-seg / RP2040 on the matrix) is the SPI slave + renders locally; 5V + any level-shifting are generated ON the module now. PI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"
- title: Calcumaker 16 — MCU — MCU core (STM32U575) -> Calcumaker 16 / mcu / mcu
- moved on the sheet: C12, C13, C14, C15, C16, C17, C18, C19, C20, C21, C22, C23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
