File: hardware/calcumaker-mcu/display_if.kicad_sch (KiCad schematic)
At the start: 12 parts, among them J3 TO DISPLAY, U5 TPS61022RWUR, U6 74HCT125

Commit message: hardware: 3-board split (MCU + keyboard + display), wired display, real connectors (#1)
* hardware: 3-board split (MCU + keyboard + display), wired display, real connectors

Split the single logic board into three, wire the display as a KiCad
multi-channel design, and settle every interconnect on real, in-stock parts.

Three-board split (was two):
- Rename calcumaker-main -> calcumaker-mcu (brain/PSU logic board).
- New calcumaker-keyboard board: 50-key Cherry MX matrix + its own
  STM32G031K8U6 scanner (LCSC C432207, UFQFPN-32) + annunciator LEDs,
  mezzanine-stacked above the MCU board. Keyscanning is off the main board;
  only an I2C + UART link + KB_IRQ wake + power cross the mezzanine.

Display board (calcumaker-display):
- Corrected FJ5161AH to a SINGLE-digit 0.56" common-cathode part (C8093) --
  it is NOT a 4-digit module; 48 single digits (16/row x 3), authored symbol
  + 0.56" LTS6760 land. The old 4-digit CC56-12 mapping (and its 3D model)
  was the phantom "clock colon".
- Rebuilt as a KiCad multi-channel design: one reusable display_row.kicad_sch
  (1 TM1640 + 16 digits, fully wired) instantiated x3. Extended kschgen.py
  with wiring primitives + reused-sheet (multi-channel) support.

Connectors (real, verified LCSC / DigiKey parts):
- Display link -> 0.5mm 12P FFC: AFC01-S12FCA-00 (LCSC C262661) on both
  boards; cable = GCT FFC05-TIN 05-12-A-<len>-A-4-06-4-T (DigiKey accessory,
  length TBD). +5V/GND conductors doubled for the display LED current.
- Keyboard mezzanine -> low-profile Hirose DF40 (0.4mm, 2x5, 1.5mm stack):
  DF40C-10DS (C424636) + DF40C-10DP (C424635) -- dedicated KiCad footprint
  + 3D model, unlike the datasheet-less generic parts first considered.

Low-power & wake documented (two Stop domains; keypress -> G0 EXTI wake ->
KB_IRQ -> U575 WKUP; G0 also wakes on I2C address-match). calcumaker-core
is unchanged -- App still consumes (row,col).

All three boards generate + pass the structure check (mcu 52 / keyboard 119 /
display 60 compo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
Parts:
- removed J3: TO DISPLAY, Connector_PinHeader_2.54mm:PinHeader_1x10_P2.54mm_Vertical, symbol Connector_Generic:Conn_01x10
- added J3: TO DISPLAY (FFC), Connector_FFC-FPC:Hirose_FH12-12S-0.5SH_1x12-1MP_P0.50mm_Horizontal, symbol Connector_Generic:Conn_01x12
Other:
- note added: "Calcumaker 16 MCU board — Display 5V rail + interface. 5V BOOST U5 TPS61022 (C915088, EN-gated): VIN<-VSYS (3.0-4.7V), L2 1uH (C5832342), Cin C8 10uF, Cout C9/C10 2x22uF; FB R6/R7 divider -> +5V (Vref 0.6V); EN<-MCU DISP_PWR_EN (low in sleep). LEVEL SHIFT U6 74HCT125 @ +5V (VIH=2V accepts 3V3): IN<-MCU CLK,DIN1,DIN2,DIN3 (3V3); OUT-> J3 at 5V logic; C11 100nF; tie all 4 /OE low. J3 = 0.5mm 12P FF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"
- note removed: "Calcumaker 16 main — Display 5V rail + interface. 5V BOOST U5 TPS61022 (C915088, EN-gated): VIN<-VSYS (3.0-4.7V), L2 1uH (C5832342), Cin C8 10uF, Cout C9/C10 2x22uF; FB R6/R7 divider -> +5V (Vref 0.6V); EN<-MCU DISP_PWR_EN (low in sleep). LEVEL SHIFT U6 74HCT125 @ +5V (VIH=2V accepts 3V3): IN<-MCU CLK,DIN1,DIN2,DIN3 (3V3); OUT-> J3 at 5V logic; C11 100nF; tie all 4 /OE low. J3 to display (MUST ma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"
- title: Calcumaker 16 — Main — Display 5V rail (TPS61022) + 74HCT125 level shifter + interconnect -> Calcumaker 16 — MCU — Display 5V rail (TPS61022) + 74HCT125 level shifter + interconnect
Changed lines of the file:
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@@
 	(paper "A3")
 	(title_block
-		(title "Calcumaker 16 — Main — Display 5V rail (TPS61022) + 74HCT125 level shifter + interconnect")
-		(date "2026-06-21")
-		(rev "0.1")
+		(title "Calcumaker 16 — MCU — Display 5V rail (TPS61022) + 74HCT125 level shifter + interconnect")
+		(date "2026-07-05")
+		(rev "0.2")
 		(company "calcumaker authors")
 	)
@@
 		(pin "7")
 		(instances
-			(project "calcumaker-main"
-				(path "/ca1c0000-0000-4000-8000-00000000ma01/5a080947-7cc4-4e41-bc3c-27cf4b2ace01"
+			(project "calcumaker-mcu"
+				(path "/ca1c0000-0000-4000-8000-00000000ma01/882301f2-c62c-4450-8afe-fd55e1916916"
 					(reference "U5")
 					(unit 1)
@@
 		(pin "14")
 		(instances
-			(project "calcumaker-main"
-				(path "/ca1c0000-0000-4000-8000-00000000ma01/5a080947-7cc4-4e41-bc3c-27cf4b2ace01"
+			(project "calcumaker-mcu"
+				(path "/ca1c0000-0000-4000-8000-00000000ma01/882301f2-c62c-4450-8afe-fd55e1916916"
 					(reference "U6")
 					(unit 1)
@@
 	)
 	(symbol
-		(lib_id "Connector_Generic:Conn_01x10")
+		(lib_id "Connector_Generic:Conn_01x12")
 		(at 238.7600 55.8800 0)
 		(unit 1)
@@
 			(effects (font (size 1.27 1.27)) (justify left))
 		)
-		(property "Value" "TO DISPLAY"
+		(property "Value" "TO DISPLAY (FFC)"
 			(at 242.5700 58.4200 0)
 			(effects (font (size 1.27 1.27)) (justify left))
 		)
-		(property "Footprint" "Connector_PinHeader_2.54mm:PinHeader_1x10_P2.54mm_Vertical"
+		(property "Footprint" "Connector_FFC-FPC:Hirose_FH12-12S-0.5SH_1x12-1MP_P0.50mm_Horizontal"
 			(at 238.7600 55.8800 0)
 			(effects (font (size 1.27 1.27))) (hide yes)
@@
 			(effects (font (size 1.27 1.27))) (hide yes)
 		)
-		(property "LCSC" "C492409"
+		(property "LCSC" "C262661"
 			(at 238.7600 55.8800 0)
 			(effects (font (size 1.27 1.27))) (hide yes)
 		)
-		(property "MPN" "PZ254V-11-10P"
+		(property "MPN" "AFC01-S12FCA-00"
 			(at 238.7600 55.8800 0)
 			(effects (font (size 1.27 1.27))) (hide yes)
 		)
-		(property "Manufacturer" "XKB"
+		(property "Manufacturer" "JUSHUO"
 			(at 238.7600 55.8800 0)
 			(effects (font (size 1.27 1.27))) (hide yes)
@@
 		(pin "9")
 		(pin "10")
-		(instances
-			(project "calcumaker-main"
-				(path "/ca1c0000-0000-4000-8000-00000000ma01/5a080947-7cc4-4e41-bc3c-27cf4b2ace01"
+		(pin "11")
+		(pin "12")
+		(instances
+			(project "calcumaker-mcu"
+				(path "/ca1c0000-0000-4000-8000-00000000ma01/882301f2-c62c-4450-8afe-fd55e1916916"
 					(reference "J3")
 					(unit 1)
@@
 		(pin "2")
 		(instances
-			(project "calcumaker-main"
-				(path "/ca1c0000-0000-4000-8000-00000000ma01/5a080947-7cc4-4e41-bc3c-27cf4b2ace01"
+			(project "calcumaker-mcu"
+				(path "/ca1c0000-0000-4000-8000-00000000ma01/882301f2-c62c-4450-8afe-fd55e1916916"
 					(reference "L2")
 					(unit 1)
@@
 		(pin "2")
 		(instances
-			(project "calcumaker-main"
-				(path "/ca1c0000-0000-4000-8000-00000000ma01/5a080947-7cc4-4e41-bc3c-27cf4b2ace01"
+			(project "calcumaker-mcu"
+				(path "/ca1c0000-0000-4000-8000-00000000ma01/882301f2-c62c-4450-8afe-fd55e1916916"
 					(reference "C8")
 					(unit 1)
@@
 		(pin "2")
 		(instances
-			(project "calcumaker-main"
-				(path "/ca1c0000-0000-4000-8000-00000000ma01/5a080947-7cc4-4e41-bc3c-27cf4b2ace01"
+			(project "calcumaker-mcu"
+				(path "/ca1c0000-0000-4000-8000-00000000ma01/882301f2-c62c-4450-8afe-fd55e1916916"
 					(reference "C9")
 					(unit 1)
@@
 		(pin "2")
 		(instances
-			(project "calcumaker-main"
-				(path "/ca1c0000-0000-4000-8000-00000000ma01/5a080947-7cc4-4e41-bc3c-27cf4b2ace01"
+			(project "calcumaker-mcu"
+				(path "/ca1c0000-0000-4000-8000-00000000ma01/882301f2-c62c-4450-8afe-fd55e1916916"
 					(reference "C10")
 					(unit 1)
@@
 		(pin "2")
 		(instances
-			(project "calcumaker-main"
-				(path "/ca1c0000-0000-4000-8000-00000000ma01/5a080947-7cc4-4e41-bc3c-27cf4b2ace01"
+			(project "calcumaker-mcu"
+				(path "/ca1c0000-0000-4000-8000-00000000ma01/882301f2-c62c-4450-8afe-fd55e1916916"
 					(reference "C11")
 					(unit 1)
@@
 		(pin "2")
 		(instances
-			(project "calcumaker-main"
-				(path "/ca1c0000-0000-4000-8000-00000000ma01/5a080947-7cc4-4e41-bc3c-27cf4b2ace01"
+			(project "calcumaker-mcu"
+				(path "/ca1c0000-0000-4000-8000-00000000ma01/882301f2-c62c-4450-8afe-fd55e1916916"
 					(reference "R6")
 					(unit 1)
@@
 		(pin "2")
 		(instances
-			(project "calcumaker-main"
-				(path "/ca1c0000-0000-4000-8000-00000000ma01/5a080947-7cc4-4e41-bc3c-27cf4b2ace01"
+			(project "calcumaker-mcu"
+				(path "/ca1c0000-0000-4000-8000-00000000ma01/882301f2-c62c-4450-8afe-fd55e1916916"
 					(reference "R7")
 					(unit 1)
@@
 		(pin "2")
 		(instances
-			(project "calcumaker-main"
-				(path "/ca1c0000-0000-4000-8000-00000000ma01/5a080947-7cc4-4e41-bc3c-27cf4b2ace01"
+			(project "calcumaker-mcu"
+				(path "/ca1c0000-0000-4000-8000-00000000ma01/882301f2-c62c-4450-8afe-fd55e1916916"
 					(reference "R14")
 					(unit 1)
@@
 		(pin "2")
 		(instances
-			(project "calcumaker-main"
-				(path "/ca1c0000-0000-4000-8000-00000000ma01/5a080947-7cc4-4e41-bc3c-27cf4b2ace01"
+			(project "calcumaker-mcu"
+				(path "/ca1c0000-0000-4000-8000-00000000ma01/882301f2-c62c-4450-8afe-fd55e1916916"
 					(reference "R15")
 					(unit 1)
@@
 		)
 	)
-	(text "Calcumaker 16 main — Display 5V rail + interface. 5V BOOST U5 TPS61022 (C915088, EN-gated): VIN<-VSYS (3.0-4.7V), L2 1uH (C5832342), Cin C8 10uF, Cout C9/C10 2x22uF; FB R6/R7 divider -> +5V (Vref 0.6V); EN<-MCU DISP_PWR_EN (low in sleep). LEVEL SHIFT U6 74HCT125 @ +5V (VIH=2V accepts 3V3): IN<-MCU CLK,DIN1,DIN2,DIN3 (3V3); OUT-> J3 at 5V logic; C11 100nF; tie all 4 /OE low. J3 to display (MUST match calcumaker-display J1): 1=+5V, 2=GND, 3=CLK, 4=DIN1, 5=DIN2, 6=DIN3, 7=GND, 8=spare. Wide +5V/GND (LED current). See DESIGN.md Power Tree / Board Partition."
+	(text "Calcumaker 16 MCU board — Display 5V rail + interface. 5V BOOST U5 TPS61022 (C915088, EN-gated): VIN<-VSYS (3.0-4.7V), L2 1uH (C5832342), Cin C8 10uF, Cout C9/C10 2x22uF; FB R6/R7 divider -> +5V (Vref 0.6V); EN<-MCU DISP_PWR_EN (low in sleep). LEVEL SHIFT U6 74HCT125 @ +5V (VIH=2V accepts 3V3): IN<-MCU CLK,DIN1,DIN2,DIN3 (3V3); OUT-> J3 at 5V logic; C11 100nF; tie all 4 /OE low. J3 = 0.5mm 12P FFC to display (AFC01-S12FCA-00 C262661; cable = GCT FFC05-TIN 05-12-A-<len>-A-4-06-4-T, DigiKey, length TBD). Pinout (MUST match calcumaker-display J1): 1=+5V, 2=+5V, 3=GND, 4=CLK, 5=DIN1, 6=DIN2, 7=DIN3, 8=GND, 9=+3V3, 10=SDA, 11=SCL, 12=GND. +5V/GND DOUBLED for LED current (0.5mm FFC conductor ~0.4A). Pins 9-11 = the DNP aux OLED I2C. See DESIGN.md Power Tree / Board Partition."
 		(exclude_from_sim no)
 		(at 15.00 110.00 0)
@@
 	(sheet_instances
 		(path "/"
-			(page "7")
-		)
-	)
+			(page "6")
+		)
+	)
