File: hardware/calcumaker-mcu/display_if.kicad_sch (KiCad schematic)
At the start: 12 parts, among them J3 TO DISPLAY, U5 TPS61022RWUR, U6 74HCT125

Commit message: hardware: 3-board split (MCU + keyboard + display), wired display, real connectors
Split the single logic board into three, wire the display as a KiCad
multi-channel design, and settle every interconnect on real, in-stock parts.

Three-board split (was two):
- Rename calcumaker-main -> calcumaker-mcu (brain/PSU logic board).
- New calcumaker-keyboard board: 50-key Cherry MX matrix + its own
  STM32G031K8U6 scanner (LCSC C432207, UFQFPN-32) + annunciator LEDs,
  mezzanine-stacked above the MCU board. Keyscanning is off the main board;
  only an I2C + UART link + KB_IRQ wake + power cross the mezzanine.

Display board (calcumaker-display):
- Corrected FJ5161AH to a SINGLE-digit 0.56" common-cathode part (C8093) --
  it is NOT a 4-digit module; 48 single digits (16/row x 3), authored symbol
  + 0.56" LTS6760 land. The old 4-digit CC56-12 mapping (and its 3D model)
  was the phantom "clock colon".
- Rebuilt as a KiCad multi-channel design: one reusable display_row.kicad_sch
  (1 TM1640 + 16 digits, fully wired) instantiated x3. Extended kschgen.py
  with wiring primitives + reused-sheet (multi-channel) support.

Connectors (real, verified LCSC / DigiKey parts):
- Display link -> 0.5mm 12P FFC: AFC01-S12FCA-00 (LCSC C262661) on both
  boards; cable = GCT FFC05-TIN 05-12-A-<len>-A-4-06-4-T (DigiKey accessory,
  length TBD). +5V/GND conductors doubled for the display LED current.
- Keyboard mezzanine -> low-profile Hirose DF40 (0.4mm, 2x5, 1.5mm stack):
  DF40C-10DS (C424636) + DF40C-10DP (C424635) -- dedicated KiCad footprint
  + 3D model, unlike the datasheet-less generic parts first considered.

Low-power & wake documented (two Stop domains; keypress -> G0 EXTI wake ->
KB_IRQ -> U575 WKUP; G0 also wakes on I2C address-match). calcumaker-core
is unchanged -- App still consumes (row,col).

All three boards generate + pass the structure check (mcu 52 / keyboard 119 /
display 60 components, all footprints assigned, no duplicate refs). Docs
(DESIGN.md, PARTS.md incl. a Non-B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
Parts:
- removed J3: TO DISPLAY, Connector_PinHeader_2.54mm:PinHeader_1x10_P2.54mm_Vertical, symbol Connector_Generic:Conn_01x10
- added J3: TO DISPLAY (FFC), Connector_FFC-FPC:Hirose_FH12-12S-0.5SH_1x12-1MP_P0.50mm_Horizontal, symbol Connector_Generic:Conn_01x12
Other:
- note added: "Calcumaker 16 main — Display 5V rail + interface. 5V BOOST U5 TPS61022 (C915088, EN-gated): VIN<-VSYS (3.0-4.7V), L2 1uH (C5832342), Cin C8 10uF, Cout C9/C10 2x22uF; FB R6/R7 divider -> +5V (Vref 0.6V); EN<-MCU DISP_PWR_EN (low in sleep). LEVEL SHIFT U6 74HCT125 @ +5V (VIH=2V accepts 3V3): IN<-MCU CLK,DIN1,DIN2,DIN3 (3V3); OUT-> J3 at 5V logic; C11 100nF; tie all 4 /OE low. J3 = 0.5mm 12P FFC to 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"
- note removed: "Calcumaker 16 main — Display 5V rail + interface. 5V BOOST U5 TPS61022 (C915088, EN-gated): VIN<-VSYS (3.0-4.7V), L2 1uH (C5832342), Cin C8 10uF, Cout C9/C10 2x22uF; FB R6/R7 divider -> +5V (Vref 0.6V); EN<-MCU DISP_PWR_EN (low in sleep). LEVEL SHIFT U6 74HCT125 @ +5V (VIH=2V accepts 3V3): IN<-MCU CLK,DIN1,DIN2,DIN3 (3V3); OUT-> J3 at 5V logic; C11 100nF; tie all 4 /OE low. J3 to display (MUST ma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"
- title: Calcumaker 16 — Main — Display 5V rail (TPS61022) + 74HCT125 level shifter + interconnect -> Calcumaker 16 — MCU — Display 5V rail (TPS61022) + 74HCT125 level shifter + interconnect
Changed lines of the file:
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@@
 	(paper "A3")
 	(title_block
-		(title "Calcumaker 16 — Main — Display 5V rail (TPS61022) + 74HCT125 level shifter + interconnect")
-		(date "2026-06-21")
-		(rev "0.1")
+		(title "Calcumaker 16 — MCU — Display 5V rail (TPS61022) + 74HCT125 level shifter + interconnect")
+		(date "2026-07-05")
+		(rev "0.2")
 		(company "calcumaker authors")
 	)
@@
 		(pin "7")
 		(instances
-			(project "calcumaker-main"
-				(path "/ca1c0000-0000-4000-8000-00000000ma01/5a080947-7cc4-4e41-bc3c-27cf4b2ace01"
+			(project "calcumaker-mcu"
+				(path "/ca1c0000-0000-4000-8000-00000000ma01/882301f2-c62c-4450-8afe-fd55e1916916"
 					(reference "U5")
 					(unit 1)
@@
 		(pin "14")
 		(instances
-			(project "calcumaker-main"
-				(path "/ca1c0000-0000-4000-8000-00000000ma01/5a080947-7cc4-4e41-bc3c-27cf4b2ace01"
+			(project "calcumaker-mcu"
+				(path "/ca1c0000-0000-4000-8000-00000000ma01/882301f2-c62c-4450-8afe-fd55e1916916"
 					(reference "U6")
 					(unit 1)
@@
 	)
 	(symbol
-		(lib_id "Connector_Generic:Conn_01x10")
+		(lib_id "Connector_Generic:Conn_01x12")
 		(at 238.7600 55.8800 0)
 		(unit 1)
@@
 			(effects (font (size 1.27 1.27)) (justify left))
 		)
-		(property "Value" "TO DISPLAY"
+		(property "Value" "TO DISPLAY (FFC)"
 			(at 242.5700 58.4200 0)
 			(effects (font (size 1.27 1.27)) (justify left))
 		)
-		(property "Footprint" "Connector_PinHeader_2.54mm:PinHeader_1x10_P2.54mm_Vertical"
+		(property "Footprint" "Connector_FFC-FPC:Hirose_FH12-12S-0.5SH_1x12-1MP_P0.50mm_Horizontal"
 			(at 238.7600 55.8800 0)
 			(effects (font (size 1.27 1.27))) (hide yes)
@@
 			(effects (font (size 1.27 1.27))) (hide yes)
 		)
-		(property "LCSC" "C492409"
+		(property "LCSC" "C262661"
 			(at 238.7600 55.8800 0)
 			(effects (font (size 1.27 1.27))) (hide yes)
 		)
-		(property "MPN" "PZ254V-11-10P"
+		(property "MPN" "AFC01-S12FCA-00"
 			(at 238.7600 55.8800 0)
 			(effects (font (size 1.27 1.27))) (hide yes)
 		)
-		(property "Manufacturer" "XKB"
+		(property "Manufacturer" "JUSHUO"
 			(at 238.7600 55.8800 0)
 			(effects (font (size 1.27 1.27))) (hide yes)
@@
 		(pin "9")
 		(pin "10")
-		(instances
-			(project "calcumaker-main"
-				(path "/ca1c0000-0000-4000-8000-00000000ma01/5a080947-7cc4-4e41-bc3c-27cf4b2ace01"
+		(pin "11")
+		(pin "12")
+		(instances
+			(project "calcumaker-mcu"
+				(path "/ca1c0000-0000-4000-8000-00000000ma01/882301f2-c62c-4450-8afe-fd55e1916916"
 					(reference "J3")
 					(unit 1)
@@
 		(pin "2")
 		(instances
-			(project "calcumaker-main"
-				(path "/ca1c0000-0000-4000-8000-00000000ma01/5a080947-7cc4-4e41-bc3c-27cf4b2ace01"
+			(project "calcumaker-mcu"
+				(path "/ca1c0000-0000-4000-8000-00000000ma01/882301f2-c62c-4450-8afe-fd55e1916916"
 					(reference "L2")
 					(unit 1)
@@
 		(pin "2")
 		(instances
-			(project "calcumaker-main"
-				(path "/ca1c0000-0000-4000-8000-00000000ma01/5a080947-7cc4-4e41-bc3c-27cf4b2ace01"
+			(project "calcumaker-mcu"
+				(path "/ca1c0000-0000-4000-8000-00000000ma01/882301f2-c62c-4450-8afe-fd55e1916916"
 					(reference "C8")
 					(unit 1)
@@
 		(pin "2")
 		(instances
-			(project "calcumaker-main"
-				(path "/ca1c0000-0000-4000-8000-00000000ma01/5a080947-7cc4-4e41-bc3c-27cf4b2ace01"
+			(project "calcumaker-mcu"
+				(path "/ca1c0000-0000-4000-8000-00000000ma01/882301f2-c62c-4450-8afe-fd55e1916916"
 					(reference "C9")
 					(unit 1)
@@
 		(pin "2")
 		(instances
-			(project "calcumaker-main"
-				(path "/ca1c0000-0000-4000-8000-00000000ma01/5a080947-7cc4-4e41-bc3c-27cf4b2ace01"
+			(project "calcumaker-mcu"
+				(path "/ca1c0000-0000-4000-8000-00000000ma01/882301f2-c62c-4450-8afe-fd55e1916916"
 					(reference "C10")
 					(unit 1)
@@
 		(pin "2")
 		(instances
-			(project "calcumaker-main"
-				(path "/ca1c0000-0000-4000-8000-00000000ma01/5a080947-7cc4-4e41-bc3c-27cf4b2ace01"
+			(project "calcumaker-mcu"
+				(path "/ca1c0000-0000-4000-8000-00000000ma01/882301f2-c62c-4450-8afe-fd55e1916916"
 					(reference "C11")
 					(unit 1)
@@
 		(pin "2")
 		(instances
-			(project "calcumaker-main"
-				(path "/ca1c0000-0000-4000-8000-00000000ma01/5a080947-7cc4-4e41-bc3c-27cf4b2ace01"
+			(project "calcumaker-mcu"
+				(path "/ca1c0000-0000-4000-8000-00000000ma01/882301f2-c62c-4450-8afe-fd55e1916916"
 					(reference "R6")
 					(unit 1)
@@
 		(pin "2")
 		(instances
-			(project "calcumaker-main"
-				(path "/ca1c0000-0000-4000-8000-00000000ma01/5a080947-7cc4-4e41-bc3c-27cf4b2ace01"
+			(project "calcumaker-mcu"
+				(path "/ca1c0000-0000-4000-8000-00000000ma01/882301f2-c62c-4450-8afe-fd55e1916916"
 					(reference "R7")
 					(unit 1)
@@
 		(pin "2")
 		(instances
-			(project "calcumaker-main"
-				(path "/ca1c0000-0000-4000-8000-00000000ma01/5a080947-7cc4-4e41-bc3c-27cf4b2ace01"
+			(project "calcumaker-mcu"
+				(path "/ca1c0000-0000-4000-8000-00000000ma01/882301f2-c62c-4450-8afe-fd55e1916916"
 					(reference "R14")
 					(unit 1)
@@
 		(pin "2")
 		(instances
-			(project "calcumaker-main"
-				(path "/ca1c0000-0000-4000-8000-00000000ma01/5a080947-7cc4-4e41-bc3c-27cf4b2ace01"
+			(project "calcumaker-mcu"
+				(path "/ca1c0000-0000-4000-8000-00000000ma01/882301f2-c62c-4450-8afe-fd55e1916916"
 					(reference "R15")
 					(unit 1)
@@
 		)
 	)
-	(text "Calcumaker 16 main — Display 5V rail + interface. 5V BOOST U5 TPS61022 (C915088, EN-gated): VIN<-VSYS (3.0-4.7V), L2 1uH (C5832342), Cin C8 10uF, Cout C9/C10 2x22uF; FB R6/R7 divider -> +5V (Vref 0.6V); EN<-MCU DISP_PWR_EN (low in sleep). LEVEL SHIFT U6 74HCT125 @ +5V (VIH=2V accepts 3V3): IN<-MCU CLK,DIN1,DIN2,DIN3 (3V3); OUT-> J3 at 5V logic; C11 100nF; tie all 4 /OE low. J3 to display (MUST match calcumaker-display J1): 1=+5V, 2=GND, 3=CLK, 4=DIN1, 5=DIN2, 6=DIN3, 7=GND, 8=spare. Wide +5V/GND (LED current). See DESIGN.md Power Tree / Board Partition."
+	(text "Calcumaker 16 main — Display 5V rail + interface. 5V BOOST U5 TPS61022 (C915088, EN-gated): VIN<-VSYS (3.0-4.7V), L2 1uH (C5832342), Cin C8 10uF, Cout C9/C10 2x22uF; FB R6/R7 divider -> +5V (Vref 0.6V); EN<-MCU DISP_PWR_EN (low in sleep). LEVEL SHIFT U6 74HCT125 @ +5V (VIH=2V accepts 3V3): IN<-MCU CLK,DIN1,DIN2,DIN3 (3V3); OUT-> J3 at 5V logic; C11 100nF; tie all 4 /OE low. J3 = 0.5mm 12P FFC to display (AFC01-S12FCA-00 C262661; cable = GCT FFC05-TIN 05-12-A-<len>-A-4-06-4-T, DigiKey, length TBD). Pinout (MUST match calcumaker-display J1): 1=+5V, 2=+5V, 3=GND, 4=CLK, 5=DIN1, 6=DIN2, 7=DIN3, 8=GND, 9=+3V3, 10=SDA, 11=SCL, 12=GND. +5V/GND DOUBLED for LED current (0.5mm FFC conductor ~0.4A). Pins 9-11 = the DNP aux OLED I2C. See DESIGN.md Power Tree / Board Partition."
 		(exclude_from_sim no)
 		(at 15.00 110.00 0)
@@
 	(sheet_instances
 		(path "/"
-			(page "7")
-		)
-	)
+			(page "6")
+		)
+	)

Commit message: docs: accuracy cleanup across README/DESIGN/PARTS + firmware/schgen comments
Sweep the docs and code comments to the three-board reality. Reviewed for
accuracy against the schematics/parts — no factual fixes were needed; this
also corrected several stale spots left over from the split:

- README / DESIGN.md / PARTS.md / reference: three-board split, 0.5mm FFC
  display link, Hirose DF40 mezzanine, STM32G0 keyboard scanner; drop stale
  "main board" phrasing; populate reference/README.md's datasheet table with
  the real parts (STM32G031K8U6, TM1640, FJ5161AH, AFC01-S12FCA-00 + GCT FFC,
  DF40C-10DS/DP).
- DESIGN.md Annunciators corrected to the keyboard board (D51-55 / R1-5,
  driven by the keyboard G0); Open Questions renumbered sequentially.
- firmware comments (keypad.rs / main.rs / Cargo.toml / README): keyboard-event
  intake over the mezzanine link + wake on KB_IRQ; fixed the wrong "host-tested
  with rug" note (it is the gmp-mpfr-nostd FFI). Comment-only, no logic change.
- schgen + .kicad_sch notes: "main" -> "MCU board", FFC/mezzanine references,
  TPS61022/MCU "no custom symbol".

All three boards still pass the structure check (mcu 52 / keyboard 119 /
display 60 components, no duplicate refs); the generator still compiles.

Co-Authored-By: Claude Opus 4.8 (1M context) <noreply@anthropic.com>
Other:
- note added: "Calcumaker 16 MCU board — Display 5V rail + interface. 5V BOOST U5 TPS61022 (C915088, EN-gated): VIN<-VSYS (3.0-4.7V), L2 1uH (C5832342), Cin C8 10uF, Cout C9/C10 2x22uF; FB R6/R7 divider -> +5V (Vref 0.6V); EN<-MCU DISP_PWR_EN (low in sleep). LEVEL SHIFT U6 74HCT125 @ +5V (VIH=2V accepts 3V3): IN<-MCU CLK,DIN1,DIN2,DIN3 (3V3); OUT-> J3 at 5V logic; C11 100nF; tie all 4 /OE low. J3 = 0.5mm 12P FF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"
- note removed: "Calcumaker 16 main — Display 5V rail + interface. 5V BOOST U5 TPS61022 (C915088, EN-gated): VIN<-VSYS (3.0-4.7V), L2 1uH (C5832342), Cin C8 10uF, Cout C9/C10 2x22uF; FB R6/R7 divider -> +5V (Vref 0.6V); EN<-MCU DISP_PWR_EN (low in sleep). LEVEL SHIFT U6 74HCT125 @ +5V (VIH=2V accepts 3V3): IN<-MCU CLK,DIN1,DIN2,DIN3 (3V3); OUT-> J3 at 5V logic; C11 100nF; tie all 4 /OE low. J3 = 0.5mm 12P FFC to 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"
Changed lines of the file:
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@@
 		)
 	)
-	(text "Calcumaker 16 main — Display 5V rail + interface. 5V BOOST U5 TPS61022 (C915088, EN-gated): VIN<-VSYS (3.0-4.7V), L2 1uH (C5832342), Cin C8 10uF, Cout C9/C10 2x22uF; FB R6/R7 divider -> +5V (Vref 0.6V); EN<-MCU DISP_PWR_EN (low in sleep). LEVEL SHIFT U6 74HCT125 @ +5V (VIH=2V accepts 3V3): IN<-MCU CLK,DIN1,DIN2,DIN3 (3V3); OUT-> J3 at 5V logic; C11 100nF; tie all 4 /OE low. J3 = 0.5mm 12P FFC to display (AFC01-S12FCA-00 C262661; cable = GCT FFC05-TIN 05-12-A-<len>-A-4-06-4-T, DigiKey, length TBD). Pinout (MUST match calcumaker-display J1): 1=+5V, 2=+5V, 3=GND, 4=CLK, 5=DIN1, 6=DIN2, 7=DIN3, 8=GND, 9=+3V3, 10=SDA, 11=SCL, 12=GND. +5V/GND DOUBLED for LED current (0.5mm FFC conductor ~0.4A). Pins 9-11 = the DNP aux OLED I2C. See DESIGN.md Power Tree / Board Partition."
+	(text "Calcumaker 16 MCU board — Display 5V rail + interface. 5V BOOST U5 TPS61022 (C915088, EN-gated): VIN<-VSYS (3.0-4.7V), L2 1uH (C5832342), Cin C8 10uF, Cout C9/C10 2x22uF; FB R6/R7 divider -> +5V (Vref 0.6V); EN<-MCU DISP_PWR_EN (low in sleep). LEVEL SHIFT U6 74HCT125 @ +5V (VIH=2V accepts 3V3): IN<-MCU CLK,DIN1,DIN2,DIN3 (3V3); OUT-> J3 at 5V logic; C11 100nF; tie all 4 /OE low. J3 = 0.5mm 12P FFC to display (AFC01-S12FCA-00 C262661; cable = GCT FFC05-TIN 05-12-A-<len>-A-4-06-4-T, DigiKey, length TBD). Pinout (MUST match calcumaker-display J1): 1=+5V, 2=+5V, 3=GND, 4=CLK, 5=DIN1, 6=DIN2, 7=DIN3, 8=GND, 9=+3V3, 10=SDA, 11=SCL, 12=GND. +5V/GND DOUBLED for LED current (0.5mm FFC conductor ~0.4A). Pins 9-11 = the DNP aux OLED I2C. See DESIGN.md Power Tree / Board Partition."
 		(exclude_from_sim no)
 		(at 15.00 110.00 0)

Commit message: hardware: MCU -> STM32U575RGT6 (LQFP-64) + 4MB QSPI flash; monospace wiring notes
MCU package + external flash
- Swap U1 STM32U575ZGT6 (LQFP-144) -> STM32U575RGT6 (LQFP-64, LCSC C5270980).
  The firmware links at ~323 KB so 1 MB flash is ample (~3x headroom), and with
  the key matrix scanned off-board the LQFP-64 has enough GPIO — smaller/cheaper.
- Correct the flash size everywhere: the STM32 `G` code = 1 MB (not 2 MB; the
  `I` parts are 2 MB). memory.x FLASH 2048K -> 1024K; .cargo runner -> RGTx.
- Add U7 W25Q32JVSSIQ, a 4 MB (32 Mbit) quad-SPI NOR (LCSC C179173, SOIC-8) on
  OCTOSPI1 as a new QSPIFlash sheet (+ R9 CS# pull-up + C26 decoupling) for
  memory-mapped (XIP) constants + state/program storage.
- mcu board 52 -> 55 components / 7 sheets. Docs (DESIGN.md, PARTS.md, READMEs,
  CLAUDE/AGENTS) updated; availability ladder now lists RGT6/VGT6/ZGT6.

Monospace, multi-line schematic wiring notes
- kschgen text_note() now renders notes in a monospace font (Courier New) so
  tables/columns line up; add note_block() + pin_table() helpers.
- Reformat all 14 per-sheet notes into titled, multi-line, aligned blocks —
  connector pinouts as PIN/SIGNAL tables, power/MCU sheets as wiring blocks.

The regenerated schematics carry both changes, so this is one commit. All three
boards regenerate + pass the structure check (mcu 55 / keyboard 119 / display
60, no duplicate refs).

Co-Authored-By: Claude Opus 4.8 (1M context) <noreply@anthropic.com>
Other:
- note added: "DISPLAY 5V RAIL + INTERFACE 5V BOOST U5 TPS61022 (C915088, EN-gated) VIN<-VSYS (3.0-4.7V), L2 1uH (C5832342), Cin C8 10uF, Cout C9/C10 2x22uF FB R6/R7 divider -> +5V (Vref 0.6V); EN<-MCU DISP_PWR_EN (low in sleep) LEVEL SHIFT U6 74HCT125 @ +5V (VIH=2V accepts 3V3) IN<-MCU CLK,DIN1,DIN2,DIN3 (3V3); OUT-> J3 @ 5V logic; C11 100nF; tie all 4 /OE low J3 = 0.5mm 12-pos FFC to display (AFC01-S12FCA-00,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"
- note removed: "Calcumaker 16 MCU board — Display 5V rail + interface. 5V BOOST U5 TPS61022 (C915088, EN-gated): VIN<-VSYS (3.0-4.7V), L2 1uH (C5832342), Cin C8 10uF, Cout C9/C10 2x22uF; FB R6/R7 divider -> +5V (Vref 0.6V); EN<-MCU DISP_PWR_EN (low in sleep). LEVEL SHIFT U6 74HCT125 @ +5V (VIH=2V accepts 3V3): IN<-MCU CLK,DIN1,DIN2,DIN3 (3V3); OUT-> J3 at 5V logic; C11 100nF; tie all 4 /OE low. J3 = 0.5mm 12P FF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"
Changed lines of the file:
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@@
 	(title_block
 		(title "Calcumaker 16 — MCU — Display 5V rail (TPS61022) + 74HCT125 level shifter + interconnect")
-		(date "2026-07-05")
-		(rev "0.2")
+		(date "2026-07-06")
+		(rev "0.3")
 		(company "calcumaker authors")
 	)
@@
 		(instances
 			(project "calcumaker-mcu"
-				(path "/ca1c0000-0000-4000-8000-00000000ma01/882301f2-c62c-4450-8afe-fd55e1916916"
+				(path "/ca1c0000-0000-4000-8000-00000000ma01/66273e88-92ab-499d-8908-57ce43e17319"
 					(reference "U5")
 					(unit 1)
@@
 		(instances
 			(project "calcumaker-mcu"
-				(path "/ca1c0000-0000-4000-8000-00000000ma01/882301f2-c62c-4450-8afe-fd55e1916916"
+				(path "/ca1c0000-0000-4000-8000-00000000ma01/66273e88-92ab-499d-8908-57ce43e17319"
 					(reference "U6")
 					(unit 1)
@@
 		(instances
 			(project "calcumaker-mcu"
-				(path "/ca1c0000-0000-4000-8000-00000000ma01/882301f2-c62c-4450-8afe-fd55e1916916"
+				(path "/ca1c0000-0000-4000-8000-00000000ma01/66273e88-92ab-499d-8908-57ce43e17319"
 					(reference "J3")
 					(unit 1)
@@
 		(instances
 			(project "calcumaker-mcu"
-				(path "/ca1c0000-0000-4000-8000-00000000ma01/882301f2-c62c-4450-8afe-fd55e1916916"
+				(path "/ca1c0000-0000-4000-8000-00000000ma01/66273e88-92ab-499d-8908-57ce43e17319"
 					(reference "L2")
 					(unit 1)
@@
 		(instances
 			(project "calcumaker-mcu"
-				(path "/ca1c0000-0000-4000-8000-00000000ma01/882301f2-c62c-4450-8afe-fd55e1916916"
+				(path "/ca1c0000-0000-4000-8000-00000000ma01/66273e88-92ab-499d-8908-57ce43e17319"
 					(reference "C8")
 					(unit 1)
@@
 		(instances
 			(project "calcumaker-mcu"
-				(path "/ca1c0000-0000-4000-8000-00000000ma01/882301f2-c62c-4450-8afe-fd55e1916916"
+				(path "/ca1c0000-0000-4000-8000-00000000ma01/66273e88-92ab-499d-8908-57ce43e17319"
 					(reference "C9")
 					(unit 1)
@@
 		(instances
 			(project "calcumaker-mcu"
-				(path "/ca1c0000-0000-4000-8000-00000000ma01/882301f2-c62c-4450-8afe-fd55e1916916"
+				(path "/ca1c0000-0000-4000-8000-00000000ma01/66273e88-92ab-499d-8908-57ce43e17319"
 					(reference "C10")
 					(unit 1)
@@
 		(instances
 			(project "calcumaker-mcu"
-				(path "/ca1c0000-0000-4000-8000-00000000ma01/882301f2-c62c-4450-8afe-fd55e1916916"
+				(path "/ca1c0000-0000-4000-8000-00000000ma01/66273e88-92ab-499d-8908-57ce43e17319"
 					(reference "C11")
 					(unit 1)
@@
 		(instances
 			(project "calcumaker-mcu"
-				(path "/ca1c0000-0000-4000-8000-00000000ma01/882301f2-c62c-4450-8afe-fd55e1916916"
+				(path "/ca1c0000-0000-4000-8000-00000000ma01/66273e88-92ab-499d-8908-57ce43e17319"
 					(reference "R6")
 					(unit 1)
@@
 		(instances
 			(project "calcumaker-mcu"
-				(path "/ca1c0000-0000-4000-8000-00000000ma01/882301f2-c62c-4450-8afe-fd55e1916916"
+				(path "/ca1c0000-0000-4000-8000-00000000ma01/66273e88-92ab-499d-8908-57ce43e17319"
 					(reference "R7")
 					(unit 1)
@@
 		(instances
 			(project "calcumaker-mcu"
-				(path "/ca1c0000-0000-4000-8000-00000000ma01/882301f2-c62c-4450-8afe-fd55e1916916"
+				(path "/ca1c0000-0000-4000-8000-00000000ma01/66273e88-92ab-499d-8908-57ce43e17319"
 					(reference "R14")
 					(unit 1)
@@
 		(instances
 			(project "calcumaker-mcu"
-				(path "/ca1c0000-0000-4000-8000-00000000ma01/882301f2-c62c-4450-8afe-fd55e1916916"
+				(path "/ca1c0000-0000-4000-8000-00000000ma01/66273e88-92ab-499d-8908-57ce43e17319"
 					(reference "R15")
 					(unit 1)
@@
 		)
 	)
-	(text "Calcumaker 16 MCU board — Display 5V rail + interface. 5V BOOST U5 TPS61022 (C915088, EN-gated): VIN<-VSYS (3.0-4.7V), L2 1uH (C5832342), Cin C8 10uF, Cout C9/C10 2x22uF; FB R6/R7 divider -> +5V (Vref 0.6V); EN<-MCU DISP_PWR_EN (low in sleep). LEVEL SHIFT U6 74HCT125 @ +5V (VIH=2V accepts 3V3): IN<-MCU CLK,DIN1,DIN2,DIN3 (3V3); OUT-> J3 at 5V logic; C11 100nF; tie all 4 /OE low. J3 = 0.5mm 12P FFC to display (AFC01-S12FCA-00 C262661; cable = GCT FFC05-TIN 05-12-A-<len>-A-4-06-4-T, DigiKey, length TBD). Pinout (MUST match calcumaker-display J1): 1=+5V, 2=+5V, 3=GND, 4=CLK, 5=DIN1, 6=DIN2, 7=DIN3, 8=GND, 9=+3V3, 10=SDA, 11=SCL, 12=GND. +5V/GND DOUBLED for LED current (0.5mm FFC conductor ~0.4A). Pins 9-11 = the DNP aux OLED I2C. See DESIGN.md Power Tree / Board Partition."
+	(text "DISPLAY 5V RAIL + INTERFACE\n\n5V BOOST  U5 TPS61022 (C915088, EN-gated)\n  VIN<-VSYS (3.0-4.7V), L2 1uH (C5832342), Cin C8 10uF, Cout C9/C10 2x22uF\n  FB R6/R7 divider -> +5V (Vref 0.6V);  EN<-MCU DISP_PWR_EN (low in sleep)\nLEVEL SHIFT  U6 74HCT125 @ +5V (VIH=2V accepts 3V3)\n  IN<-MCU CLK,DIN1,DIN2,DIN3 (3V3);  OUT-> J3 @ 5V logic;\n  C11 100nF;  tie all 4 /OE low\n\nJ3 = 0.5mm 12-pos FFC to display (AFC01-S12FCA-00, C262661).\nPinout MUST match calcumaker-display J1:\n\n  PIN  SIGNAL    PIN  SIGNAL\n    1  +5V         7  DIN3  \n    2  +5V         8  GND   \n    3  GND         9  +3V3  \n    4  CLK        10  SDA   \n    5  DIN1       11  SCL   \n    6  DIN2       12  GND\n\n+5V/GND doubled for LED current (a 0.5mm FFC conductor is ~0.4A).\nPins 9-11 = the DNP aux OLED I2C.\nCABLE (non-BOM): GCT FFC05-TIN 05-12-A-<len>-A-4-06-4-T (DigiKey; len TBD).\nSee DESIGN.md Power Tree / Board Partition."
 		(exclude_from_sim no)
 		(at 15.00 110.00 0)
-		(effects (font (size 1.5 1.5)) (justify left top))
+		(effects (font (face "Courier New") (size 1.27 1.27)) (justify left top))
 	)
 	(sheet_instances
