File: hardware/calcumaker-mcu/psu.kicad_sch (KiCad schematic)
At the start: 21 parts, among them J1 USB-C, J2 BAT 1S Li-ion, Q1 AO3401A, U2 TPS63900DSKR, U3 USBLC6-2SC6, U4 MCP73831-2-OT

Commit message: Checkpoint
Parts:
- removed D1: B5819W, Diode_SMD:D_SOD-123, symbol Device:D_Schottky
- removed Q1: AO3401A, Package_TO_SOT_SMD:SOT-23, symbol Transistor_FET:Q_PMOS_GSD
- removed U4: MCP73831-2-OT, Package_TO_SOT_SMD:SOT-23-5, symbol Battery_Management:MCP73831-2-OT
- added C10, C8, C9: 10uF, Capacitor_SMD:C_0603_1608Metric, symbol Device:C
- added C11: 4.7uF, Capacitor_SMD:C_0603_1608Metric, symbol Device:C
- added C27: 47nF, Capacitor_SMD:C_0402_1005Metric, symbol Device:C
- added C28, C29: 150pF, Capacitor_SMD:C_0402_1005Metric, symbol Device:C
- added C30: 100nF 50V X7R, Capacitor_SMD:C_0603_1608Metric, symbol Device:C
- added C31, C32: 100nF, Capacitor_SMD:C_0402_1005Metric, symbol Device:C
- added L2: 2.2uH, Inductor_SMD:L_Changjiang_FNR4020S, symbol Device:L
- added Q1: AO3400A, Package_TO_SOT_SMD:SOT-23, symbol Transistor_FET:Q_NMOS_GSD
- added R10: 40.2k, Resistor_SMD:R_0402_1005Metric, symbol Device:R
- added R11, R12: 100k, Resistor_SMD:R_0402_1005Metric, symbol Device:R
- added R6: 10k, Resistor_SMD:R_0402_1005Metric, symbol Device:R
- added R7: 976R, Resistor_SMD:R_0402_1005Metric, symbol Device:R
- added U4: BQ25601RTWR, Package_DFN_QFN:Texas_RTW_WQFN-24-1EP_4x4mm_P0.5mm_EP2.7x2.7mm_ThermalVias, symbol Battery_Management:BQ25601
- added U5: TCPP01-M12, Package_DFN_QFN:QFN-12-1EP_3x3mm_P0.5mm_EP1.45x1.45mm_ThermalVias, symbol calcumaker:TCPP01-M12
- added U6: MAX17048G+T10, Package_DFN_QFN:TDFN-8-1EP_2x2mm_P0.5mm_EP0.8x1.2mm, symbol calcumaker:MAX17048
- C1: value 10uF -> 1uF 50V; LCSC (none) -> C15849; MPN (none) -> CL10A105KB8NNNC; Manufacturer (none) -> Samsung
- C2, C6: value 10uF -> 10uF 50V; footprint Capacitor_SMD:C_0603_1608Metric -> Capacitor_SMD:C_0805_2012Metric; LCSC (none) -> C440198; MPN (none) -> GRM21BR61H106KE43L; Manufacturer (none) -> Murata
- R1: value 5.1k -> 100k; LCSC C25905 -> C25741
- R2: value 5.1k -> 5.23k; LCSC C25905 -> (none)
- R3: value 4.7k -> 30.1k; LCSC C25900 -> (none)
- R4: value 100k -> 200k; LCSC C25741 -> (none)
Connections:
- new net: U4.13 (BAT), U4.14 (BAT)
- new net: U4.15 (SYS), U4.16 (SYS)
- new net: U4.17 (GND), U4.18 (GND), U4.25 (GND)
- new net: U4.19 (SW), U4.20 (SW)
Other:
- note added: "POWER - USB-C -> BQ25601 (3A buck + NVDC power path) -> buck-boost 3V3 PLACED, not wired. See DESIGN.md Power / Power Tree. USB-C J1 D+/D- -> U3 ESD -> MCU USB. (TCPP01 covers VBUS+CC, not data.) TCPP01 U5 ST Type-C port protection -- the companion chip to STM32 UCPD. VBUS PATH (U5 gate-drives Q1; VBUS passes THROUGH the FET): J1 VBUS -> C30 (ESD cap, 50V X7R, keep CLOSE to U5) -> IN_GD(8) IN_GD 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"
- note removed: "POWER - USB-C -> charge -> load-share -> buck-boost 3V3 PLACED, not wired. See DESIGN.md Power Tree. USB-C J1 CC1->R1, CC2->R2 (5.1k sink); D+/D- -> U3 ESD -> MCU USB; VBUS bulk C6. CHARGER U4 MCP73831: VDD<-VBUS, VBAT->BAT+, PROG R3 (size to cell), STAT->D2+R5; C1/C2 in/out. LOAD-SHR Q1 AO3401A: src=BAT+, drn=VSYS, gate<-VBUS via R4; D1 B5819W VBUS->VSYS. BUCK-BST U2 TPS63900: VIN<-VSYS, L1 2.2u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"
- title: Calcumaker 16 — MCU — USB-C / Li-ion charge / load-share / buck-boost -> Calcumaker 16 — MCU — USB-C / CC sense / BQ25601 charger (NVDC power path) / buck-boost 3V3
