File: hardware/calcumaker-mcu/psu.kicad_sch (KiCad schematic)
At the start: 38 parts, among them J1 USB-C, J2 BAT 1S Li-ion, Q1 AO3400A, U2 TPS63900DSKR, U3 USBLC6-2SC6, U4 BQ25601RTWR, U5 TCPP01-M12, U6 MAX17048G+T10

Commit message: Wire mainboard and keypad schematics and verify expanded nets
Connect hierarchical interfaces, power/control circuits, debug links, matrix and RGB chains. Correct MCU package pins, diode polarity and power configuration; add bypass components and repeatable KiCad netlist/ERC checks. Document pin maps and remaining physical validation.
Parts:
- added C33: 100nF, Capacitor_SMD:C_0402_1005Metric, symbol Device:C
- added J8: PACK NTC 10k 103AT-2, Connector_JST:JST_PH_S2B-PH-K_1x02_P2.00mm_Horizontal, symbol Connector_Generic:Conn_01x02
- added J9: SHIP WAKE (short to wake), Connector_PinHeader_2.54mm:PinHeader_1x02_P2.54mm_Vertical, symbol Connector_Generic:Conn_01x02
- added R15, R16: 10k, Resistor_SMD:R_0402_1005Metric, symbol Device:R
- added R17: 100k, Resistor_SMD:R_0402_1005Metric, symbol Device:R
- added R18: 36.5k 1%, Resistor_SMD:R_0402_1005Metric, symbol Device:R
- added R19: 16.2k 1%, Resistor_SMD:R_0402_1005Metric, symbol Device:R
- added R20, R21: 1M 1%, Resistor_SMD:R_0402_1005Metric, symbol Device:R
- C11: value 4.7uF -> 4.7uF 10V
Connections:
- net BAT+: now reaches C10.1
- net BAT+: now also C32.1, J2.1 (Pin_1), U4.13 (BAT), U4.14 (BAT), U6.2 (CELL), U6.3 (VDD), R20.1
- net GND: now reaches C10.2
- net GND: now also C1.2, C11.2, C2.2, C28.2, C29.2, C3.2, C30.2, C31.2, C32.2, C4.2, C5.2, C6.2, C7.2, C8.2, C9.2, J1.A1 (GND), J1.A12 (GND), J1.B1 (GND), J1.B12 (GND), J1.SH (SHIELD), J2.2 (Pin_2), R10.2, R3.2, R7.2, U2.11 (GND), U2.2 (SEL), U2.4 (CFG2), U2.8 (GND), U3.2 (GND), U4.17 (GND), U4.18 (GND), U4.25 (GND), U5.13 (EP), U5.2 (GND), U6.1 (CTG), U6.4 (GND), U6.6 (QSTRT), U6.9 (EP), C33.2, J8.2 (Pin_2), J9.2 (Pin_2), R18.2, R19.2, R21.2
- net +3V3: now reaches R12.1
- net +3V3: now also C4.1, C5.1, C7.1, R11.1, R5.1, U2.6 (VOUT), U3.5 (VBUS), R15.1, R16.1, R17.1
- net GAUGE_ALRT: now reaches R12.2
- net GAUGE_ALRT: now also U6.5 (ALRT)
- net VBUS_IN: now reaches R6.1
- net VBUS_IN: now also C30.1, J1.A4 (VBUS), J1.A9 (VBUS), J1.B4 (VBUS), J1.B9 (VBUS), Q1.3 (D), R4.1, U5.8 (IN_GD)
- net VBUS_CTRL: now reaches R6.2
- net VBUS_CTRL: now also R7.1, U5.6 (VBUS_CTRL)
- net LX1: now reaches L1.1
- net LX1: now also U2.9 (LX1)
- net LX2: now reaches L1.2
- net LX2: now also U2.7 (LX2)
- net VSYS: now reaches C3.1
- net VSYS: now also C8.1, C9.1, L2.2, U2.1 (EN), U2.10 (VIN), U4.15 (SYS), U4.16 (SYS)
- net CC1_CONN: now reaches J1.A5 (CC1)
- net CC1_CONN: now also C28.1, U5.7 (CC1c)
- net USB_DP_CONN: now reaches J1.A6 (D+)
- net USB_DP_CONN: now also J1.B6 (D+), U3.1 (I/O1)
- net USB_DM_CONN: now reaches J1.A7 (D-)
- net USB_DM_CONN: now also J1.B7 (D-), U3.3 (I/O2)
- net CC2_CONN: now reaches J1.B5 (CC2)
- net CC2_CONN: now also C29.1, U5.9 (CC2c)
- net TCPP01_FLT: now reaches R11.2
- net TCPP01_FLT: now also U5.11 (FLT)
- net VBUS_SENSE: now reaches R4.2
- net VBUS_SENSE: now also R10.1
- net CHG_TS: now reaches R3.1
- net CHG_TS: now also R2.2, U4.11 (TS), J8.1 (Pin_1)
- net VBUS_GATE: now reaches Q1.1 (G)
- net VBUS_GATE: now also U5.5 (GATE)
- net VBUS_PROT: now reaches Q1.2 (S)
- net VBUS_PROT: now also C1.1, C6.1, U4.1 (VAC), U4.24 (VBUS), U5.4 (SOURCE)
- net I2C_SCL: now reaches U6.7 (SCL)
- net I2C_SCL: now also U4.5 (SCL)
- net I2C_SDA: now reaches U6.8 (SDA)
- net I2C_SDA: now also U4.6 (SDA)
- net CHG_QON: now reaches U4.12 (~{QON})
- net CHG_QON: now also J9.1 (Pin_1)
- net CHG_SW: now reaches U4.19 (SW), U4.20 (SW)
- net CHG_SW: now also C27.2, L2.1
- net PSEL: now reaches U4.2 (PSEL)
- net PSEL: now also R1.2
- net CHG_BTST: now reaches U4.21 (BTST)
- net CHG_BTST: now also C27.1
- net REGN: now reaches U4.22 (REGN)
- net REGN: now also C11.1, R1.1, R2.1
- net PMID: now reaches U4.23 (PMID)
- net PMID: now also C2.1
- net CHG_PG: now reaches U4.3 (~{PG})
- net CHG_PG: now also R16.2
- net CHG_STAT: now reaches U4.4 (STAT)
- net CHG_STAT: now also D2.1 (K)
- net CHG_INT: now reaches U4.7 (~{INT})
- net CHG_INT: now also R15.2
- net CHG_CE: now reaches U4.9 (~{CE})
- net CHG_CE: now also R17.2
- net CHG_LED_A: now reaches D2.2 (A)
- net CHG_LED_A: now also R5.2
- net UCPD_CC2: now reaches U5.1 (CC2)
- net TCPP01_DB: now reaches U5.10 (DB)
- net TCPP01_EN: now reaches U5.12 (VCC)
- net TCPP01_EN: now also C31.1
- net UCPD_CC1: now reaches U5.3 (CC1)
- net USB_DM: now reaches U3.4 (I/O2)
- net USB_DP: now reaches U3.6 (I/O1)
- net CFG1: now reaches U2.3 (CFG1)
- net CFG1: now also R18.1
- net CFG3: now reaches U2.5 (CFG3)
- net CFG3: now also R19.1
- new net BAT_SENSE: C33.1, R20.2, R21.1
- no-connect marks 0 -> 4
Other:
- note added: "BQ25601 @ 0x6B: VAC tied to protected VBUS. PSEL pull-up goes to REGN (<7V), never 12V VBUS. R17 inhibits charging until firmware configures the cell and pulls CE low. R2/R3 require an external 10k pack NTC on J8 (not a fixed-temperature bypass). Program 14V charger OVP before requesting a 12V PD contract. Set IINDPM from CC/PD policy; service or disable the watchdog deliberately. J9 connects QON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"
- note added: "MAX17048 @ 0x36 stays on the raw cell. BAT_SENSE = cell / 2; allow ADC settling for 1M divider. Gauge alert is open-drain. EP is connected to GND."
- note added: "TCPP01: enable VCC, enable UCPD Rd, then release DB. No external CC Rd: the dead-battery clamp hands over to UCPD. R6/R7 set OVP about 13.5-15.1V; C30 is 50V X7R at U5. U3 pin 5 = 3V3 (USB data clamp), NEVER the 12V PD rail."
- note added: "TPS63900: SEL=0, CFG3=16.2k gives 3V3. CFG1=36.5k, CFG2=0: 3V3 alternate setting / unlimited input mode. L1 >=2A saturation; verify effective Cout >=10uF at 3V3."
- note added: "USB-C + NVDC POWER PATH / 3V3 / FUEL GAUGE"
- note removed: "POWER - USB-C -> BQ25601 (3A buck + NVDC power path) -> buck-boost 3V3 PLACED, not wired. See DESIGN.md Power / Power Tree. USB-C J1 D+/D- -> U3 ESD -> MCU USB. (TCPP01 covers VBUS+CC, not data.) TCPP01 U5 ST Type-C port protection -- the companion chip to STM32 UCPD. VBUS PATH (U5 gate-drives Q1; VBUS passes THROUGH the FET): J1 VBUS -> C30 (ESD cap, 50V X7R, keep CLOSE to U5) -> IN_GD(8) IN_GD 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"
- title: Calcumaker 16 — MCU — USB-C / CC sense / BQ25601 charger (NVDC power path) / buck-boost 3V3 -> Calcumaker 16 / mcu / psu
- moved on the sheet: C1, C10, C11, C2, C27, C28, C29, C3, C30, C31, C32, C4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
