File: hardware/calcumaker-keyboard/keypad.kicad_sch (KiCad schematic)
At the start: 100 parts, among them SW1 MX, SW10 MX, SW11 MX, SW12 MX, SW13 MX, SW14 MX, SW15 MX, SW16 MX, SW17 MX, SW18 MX, SW19 MX, SW2 MX, SW20 MX, SW21 MX, SW22 MX, SW23 MX, SW24 MX, SW25 MX, SW26 MX, SW27 MX, SW28 MX, SW29 MX, SW3 MX, SW30 MX, SW31 MX, SW32 MX, SW33 MX, SW34 MX, SW35 MX, SW36 MX, SW37 MX, SW38 MX, SW39 MX, SW4 MX, SW40 MX, SW41 MX, SW42 MX, SW43 MX, SW44 MX, SW45 MX, SW46 MX, SW47 MX, SW48 MX, SW49 MX, SW5 MX, SW50 MX, SW6 MX, SW7 MX, SW8 MX, SW9 MX

Commit message: hardware: 3-board split (MCU + keyboard + display), wired display, real connectors
Split the single logic board into three, wire the display as a KiCad
multi-channel design, and settle every interconnect on real, in-stock parts.

Three-board split (was two):
- Rename calcumaker-main -> calcumaker-mcu (brain/PSU logic board).
- New calcumaker-keyboard board: 50-key Cherry MX matrix + its own
  STM32G031K8U6 scanner (LCSC C432207, UFQFPN-32) + annunciator LEDs,
  mezzanine-stacked above the MCU board. Keyscanning is off the main board;
  only an I2C + UART link + KB_IRQ wake + power cross the mezzanine.

Display board (calcumaker-display):
- Corrected FJ5161AH to a SINGLE-digit 0.56" common-cathode part (C8093) --
  it is NOT a 4-digit module; 48 single digits (16/row x 3), authored symbol
  + 0.56" LTS6760 land. The old 4-digit CC56-12 mapping (and its 3D model)
  was the phantom "clock colon".
- Rebuilt as a KiCad multi-channel design: one reusable display_row.kicad_sch
  (1 TM1640 + 16 digits, fully wired) instantiated x3. Extended kschgen.py
  with wiring primitives + reused-sheet (multi-channel) support.

Connectors (real, verified LCSC / DigiKey parts):
- Display link -> 0.5mm 12P FFC: AFC01-S12FCA-00 (LCSC C262661) on both
  boards; cable = GCT FFC05-TIN 05-12-A-<len>-A-4-06-4-T (DigiKey accessory,
  length TBD). +5V/GND conductors doubled for the display LED current.
- Keyboard mezzanine -> low-profile Hirose DF40 (0.4mm, 2x5, 1.5mm stack):
  DF40C-10DS (C424636) + DF40C-10DP (C424635) -- dedicated KiCad footprint
  + 3D model, unlike the datasheet-less generic parts first considered.

Low-power & wake documented (two Stop domains; keypress -> G0 EXTI wake ->
KB_IRQ -> U575 WKUP; G0 also wakes on I2C address-match). calcumaker-core
is unchanged -- App still consumes (row,col).

All three boards generate + pass the structure check (mcu 52 / keyboard 119 /
display 60 components, all footprints assigned, no duplicate refs). Docs
(DESIGN.md, PARTS.md incl. a Non-B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
Parts:
- removed D51, D52, D53, D54, D55, D56, D57, D58, D59, D60: 1N4148W, Diode_SMD:D_SOD-123, symbol Device:D
- added D1, D10, D2, D3, D4, D5, D6, D7, D8, D9: 1N4148W, Diode_SMD:D_SOD-123, symbol Device:D
Other:
- note added: "Calcumaker 16 keyboard — Keypad: 50 Cherry MX keys in a 5x10 scanned matrix (wide HP-16C layout + f/g shifts; keymap in DESIGN.md). PLACED, not wired. WIRING: ROW1..ROW5 + COL1..COL10 go to the on-board STM32G0 (U1, KbdMCU sheet) — ROWs = G0 GPIO outputs; COLs = G0 GPIO inputs with INTERNAL pull-ups (no external R, kept in Stop). Each key SWn in series with Dn (anode at switch, cathode to its COL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"
- note removed: "Calcumaker 16 main — Keypad: 50 Cherry MX keys in a 5x10 scanned matrix (wide HP-16C layout + f/g shifts; keymap in DESIGN.md). PLACED, not wired. WIRING: ROW1..ROW5 = GPIO outputs; COL1..COL10 = GPIO inputs with INTERNAL pull-ups (no external R; STM32U5 keeps pull-ups in Stop). Each key SWn in series with Dn (anode at switch, cathode to its COL) for n-key rollover. Key (row r, col c): SW#=(r-1)*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"
- title: Calcumaker 16 — Main — Cherry MX key matrix (5x10, 50 keys) -> Calcumaker 16 — Keyboard — Cherry MX key matrix (5x10, 50 keys)

Commit message: hardware: MCU -> STM32U575RGT6 (LQFP-64) + 4MB QSPI flash; monospace wiring notes
MCU package + external flash
- Swap U1 STM32U575ZGT6 (LQFP-144) -> STM32U575RGT6 (LQFP-64, LCSC C5270980).
  The firmware links at ~323 KB so 1 MB flash is ample (~3x headroom), and with
  the key matrix scanned off-board the LQFP-64 has enough GPIO — smaller/cheaper.
- Correct the flash size everywhere: the STM32 `G` code = 1 MB (not 2 MB; the
  `I` parts are 2 MB). memory.x FLASH 2048K -> 1024K; .cargo runner -> RGTx.
- Add U7 W25Q32JVSSIQ, a 4 MB (32 Mbit) quad-SPI NOR (LCSC C179173, SOIC-8) on
  OCTOSPI1 as a new QSPIFlash sheet (+ R9 CS# pull-up + C26 decoupling) for
  memory-mapped (XIP) constants + state/program storage.
- mcu board 52 -> 55 components / 7 sheets. Docs (DESIGN.md, PARTS.md, READMEs,
  CLAUDE/AGENTS) updated; availability ladder now lists RGT6/VGT6/ZGT6.

Monospace, multi-line schematic wiring notes
- kschgen text_note() now renders notes in a monospace font (Courier New) so
  tables/columns line up; add note_block() + pin_table() helpers.
- Reformat all 14 per-sheet notes into titled, multi-line, aligned blocks —
  connector pinouts as PIN/SIGNAL tables, power/MCU sheets as wiring blocks.

The regenerated schematics carry both changes, so this is one commit. All three
boards regenerate + pass the structure check (mcu 55 / keyboard 119 / display
60, no duplicate refs).

Co-Authored-By: Claude Opus 4.8 (1M context) <noreply@anthropic.com>
Other:
- note added: "KEYPAD - 50 Cherry MX keys in a 5x10 scanned matrix Wide HP-16C layout + f/g shifts (keymap in DESIGN.md). PLACED, not wired. WIRING ROW1..ROW5 -> G0 GPIO outputs (U1, KbdMCU sheet) COL1..COL10 -> G0 GPIO inputs, INTERNAL pull-ups (no ext R, kept in Stop) each key SWn + series Dn (anode@switch, cathode->COL) for n-key rollover key (row r, col c): SW# = D# = (r-1)*10 + c SCAN G0 drives one ROW low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"
- note removed: "Calcumaker 16 keyboard — Keypad: 50 Cherry MX keys in a 5x10 scanned matrix (wide HP-16C layout + f/g shifts; keymap in DESIGN.md). PLACED, not wired. WIRING: ROW1..ROW5 + COL1..COL10 go to the on-board STM32G0 (U1, KbdMCU sheet) — ROWs = G0 GPIO outputs; COLs = G0 GPIO inputs with INTERNAL pull-ups (no external R, kept in Stop). Each key SWn in series with Dn (anode at switch, cathode to its COL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"

Commit message: hardware: per-key RGB hint lighting on the keyboard board (50x SK6805 on gated VSYS) (#4)
Add addressable RGB accent lighting that hints key positions / presses -- one
SK6805-EC15 (1.5x1.5mm, the smallest serial RGB with a KiCad footprint + real
LCSC stock, C2890035) beside each of the 50 keys, single-wire daisy chain off
one STM32G0 pin.

Power: the LEDs are ~5V parts and the keyboard rail is only 3.3V, so they run
off VSYS (the MCU board's load-shared battery/USB rail, ~3.7-4.7V) brought up a
WIDENED 12-pin mezzanine (10 -> 12: +VSYS +GND). A high-side P-FET load switch
(Q1 AO3401A + Q2 2N7002) gates the whole LED rail off in sleep (G0 LED_EN) to
protect battery life, and a 74LVC1G125 (powered from the gated rail) level-shifts
the 3.3V data up to the LED VIH.

- calcumaker-keyboard: new KeyLighting sheet (50x SK6805 D56-D105 + U2 shifter +
  Q1/Q2 load switch + R7-R10 / C6-C7); J1 mezzanine -> 12-pin DF40C-12DP
  (C6224952). 119 -> 178 components.
- calcumaker-mcu: J5 mezzanine -> 12-pin DF40B-12DS (C3641147); route VSYS.
- DF40 stack: the receptacle SUFFIX sets the mated height (none = 1.5mm,
  (2.0) = 2.0mm, H-series = 2.5-4.0mm), NOT the B/C letter; the DF40C plug is the
  common header -- so DF40C-12DP x DF40B-12DS is a valid 1.5mm stack, same as the
  original 10-pin (DF40C-12DS just isn't LCSC-stocked).
- DESIGN.md / PARTS.md / memory: RGB subsystem, 12-pin pinout, BOM rows, the
  sleep-gate + current-cap notes (firmware must cap total brightness; 50x
  full-white ~0.75A would exceed the DF40 / VSYS budget).

All three boards regenerate + pass the structure check (mcu 55 / keyboard 178 /
display 60, no duplicate refs).

Co-authored-by: Claude Opus 4.8 (1M context) <noreply@anthropic.com>
Changed lines of the file:
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@@
 	(title_block
 		(title "Calcumaker 16 — Keyboard — Cherry MX key matrix (5x10, 50 keys)")
-		(date "2026-07-05")
-		(rev "0.2")
+		(date "2026-07-06")
+		(rev "0.3")
 		(company "calcumaker authors")
 	)
@@
 	(text "KEYPAD  -  50 Cherry MX keys in a 5x10 scanned matrix\nWide HP-16C layout + f/g shifts (keymap in DESIGN.md).  PLACED, not wired.\n\nWIRING\n  ROW1..ROW5   -> G0 GPIO outputs  (U1, KbdMCU sheet)\n  COL1..COL10  -> G0 GPIO inputs, INTERNAL pull-ups (no ext R, kept in Stop)\n  each key SWn + series Dn (anode@switch, cathode->COL) for n-key rollover\n  key (row r, col c):  SW# = D# = (r-1)*10 + c\n\nSCAN  G0 drives one ROW low, reads COLs; reports (row,col) to U575 via I2C.\nWAKE  G0 holds all ROWs low + EXTI on COLs -> any keypress wakes the G0\n      from Stop, which asserts KB_IRQ to wake the U575.\nOptional Kailh hot-swap sockets.  See DESIGN.md Low-power & wake."
 		(exclude_from_sim no)
-		(at 15.00 130.00 0)
+		(at 15.00 259.84 0)
 		(effects (font (face "Courier New") (size 1.27 1.27)) (justify left top))
 	)
