File: hardware/calcumaker-keyboard/annunc.kicad_sch (KiCad schematic)
At the start: 10 parts

Commit message: hardware: 3-board split (MCU + keyboard + display), wired display, real connectors
Split the single logic board into three, wire the display as a KiCad
multi-channel design, and settle every interconnect on real, in-stock parts.

Three-board split (was two):
- Rename calcumaker-main -> calcumaker-mcu (brain/PSU logic board).
- New calcumaker-keyboard board: 50-key Cherry MX matrix + its own
  STM32G031K8U6 scanner (LCSC C432207, UFQFPN-32) + annunciator LEDs,
  mezzanine-stacked above the MCU board. Keyscanning is off the main board;
  only an I2C + UART link + KB_IRQ wake + power cross the mezzanine.

Display board (calcumaker-display):
- Corrected FJ5161AH to a SINGLE-digit 0.56" common-cathode part (C8093) --
  it is NOT a 4-digit module; 48 single digits (16/row x 3), authored symbol
  + 0.56" LTS6760 land. The old 4-digit CC56-12 mapping (and its 3D model)
  was the phantom "clock colon".
- Rebuilt as a KiCad multi-channel design: one reusable display_row.kicad_sch
  (1 TM1640 + 16 digits, fully wired) instantiated x3. Extended kschgen.py
  with wiring primitives + reused-sheet (multi-channel) support.

Connectors (real, verified LCSC / DigiKey parts):
- Display link -> 0.5mm 12P FFC: AFC01-S12FCA-00 (LCSC C262661) on both
  boards; cable = GCT FFC05-TIN 05-12-A-<len>-A-4-06-4-T (DigiKey accessory,
  length TBD). +5V/GND conductors doubled for the display LED current.
- Keyboard mezzanine -> low-profile Hirose DF40 (0.4mm, 2x5, 1.5mm stack):
  DF40C-10DS (C424636) + DF40C-10DP (C424635) -- dedicated KiCad footprint
  + 3D model, unlike the datasheet-less generic parts first considered.

Low-power & wake documented (two Stop domains; keypress -> G0 EXTI wake ->
KB_IRQ -> U575 WKUP; G0 also wakes on I2C address-match). calcumaker-core
is unchanged -- App still consumes (row,col).

All three boards generate + pass the structure check (mcu 52 / keyboard 119 /
display 60 components, all footprints assigned, no duplicate refs). Docs
(DESIGN.md, PARTS.md incl. a Non-B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
Parts:
- removed D61: f (yellow), LED_SMD:LED_0603_1608Metric, symbol Device:LED
- removed D62: g (blue), LED_SMD:LED_0603_1608Metric, symbol Device:LED
- removed D63: C (red), LED_SMD:LED_0603_1608Metric, symbol Device:LED
- removed D64: G (red), LED_SMD:LED_0603_1608Metric, symbol Device:LED
- removed D65: LOWBAT (red), LED_SMD:LED_0603_1608Metric, symbol Device:LED
- removed R10, R11, R12, R13, R9: 470, Resistor_SMD:R_0402_1005Metric, symbol Device:R
- added D51: f (yellow), LED_SMD:LED_0603_1608Metric, symbol Device:LED
- added D52: g (blue), LED_SMD:LED_0603_1608Metric, symbol Device:LED
- added D53: C (red), LED_SMD:LED_0603_1608Metric, symbol Device:LED
- added D54: G (red), LED_SMD:LED_0603_1608Metric, symbol Device:LED
- added D55: LOWBAT (red), LED_SMD:LED_0603_1608Metric, symbol Device:LED
- added R1, R2, R3, R4, R5: 470, Resistor_SMD:R_0402_1005Metric, symbol Device:R
Other:
- note added: "Calcumaker 16 keyboard — Annunciator LEDs (DESIGN.md status-line mapping). PLACED, not wired. Five drive lines from the ON-BOARD STM32G0 (U1, active high), each -> Rn 470R -> LED -> GND: D51 'f' yellow + D52 'g' blue mounted BESIDE the f/g keys; D53 'C' carry, D54 'G' overflow, D55 low-battery along the top edge under the display bezel. +3V3 feeds the resistors; GND is the return. 470R = ~1.3-2.8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"
- note removed: "Calcumaker 16 main — Annunciator LEDs (DESIGN.md status-line mapping). PLACED, not wired. Five MCU GPIOs (active high), each -> Rn 470R -> LED -> GND: D61 'f' yellow + D62 'g' blue mounted BESIDE the f/g keys; D63 'C' carry, D64 'G' overflow, D65 low-battery along the top edge under the display bezel. 470R @3V3 = ~1.3-2.8mA; adjust per color at bring-up. Firmware: calcumaker-core App drives f/g f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"
- title: Calcumaker 16 — Main — Annunciator LEDs (f g C G low-batt) -> Calcumaker 16 — Keyboard — Annunciator LEDs (f g C G low-batt)
Changed lines of the file:
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@@
 	(paper "A3")
 	(title_block
-		(title "Calcumaker 16 — Main — Annunciator LEDs (f g C G low-batt)")
-		(date "2026-06-21")
-		(rev "0.1")
+		(title "Calcumaker 16 — Keyboard — Annunciator LEDs (f g C G low-batt)")
+		(date "2026-07-05")
+		(rev "0.2")
 		(company "calcumaker authors")
 	)
@@
 		(on_board yes)
 		(dnp no)
-		(property "Reference" "D61"
+		(property "Reference" "D51"
 			(at 34.2900 38.1000 0)
 			(effects (font (size 1.27 1.27)) (justify left))
@@
 		(pin "2")
 		(instances
-			(project "calcumaker-main"
-				(path "/ca1c0000-0000-4000-8000-00000000ma01/09ef021e-eba5-4a51-ac3b-4585f8d3f3ef"
-					(reference "D61")
+			(project "calcumaker-keyboard"
+				(path "/ca1c0000-0000-4000-8000-00000000eb01/e123962d-af1f-484c-976e-978d59e057ae"
+					(reference "D51")
 					(unit 1)
 				)
@@
 		(on_board yes)
 		(dnp no)
-		(property "Reference" "D62"
+		(property "Reference" "D52"
 			(at 72.3900 38.1000 0)
 			(effects (font (size 1.27 1.27)) (justify left))
@@
 		(pin "2")
 		(instances
-			(project "calcumaker-main"
-				(path "/ca1c0000-0000-4000-8000-00000000ma01/09ef021e-eba5-4a51-ac3b-4585f8d3f3ef"
-					(reference "D62")
+			(project "calcumaker-keyboard"
+				(path "/ca1c0000-0000-4000-8000-00000000eb01/e123962d-af1f-484c-976e-978d59e057ae"
+					(reference "D52")
 					(unit 1)
 				)
@@
 		(on_board yes)
 		(dnp no)
-		(property "Reference" "D63"
+		(property "Reference" "D53"
 			(at 110.4900 38.1000 0)
 			(effects (font (size 1.27 1.27)) (justify left))
@@
 		(pin "2")
 		(instances
-			(project "calcumaker-main"
-				(path "/ca1c0000-0000-4000-8000-00000000ma01/09ef021e-eba5-4a51-ac3b-4585f8d3f3ef"
-					(reference "D63")
+			(project "calcumaker-keyboard"
+				(path "/ca1c0000-0000-4000-8000-00000000eb01/e123962d-af1f-484c-976e-978d59e057ae"
+					(reference "D53")
 					(unit 1)
 				)
@@
 		(on_board yes)
 		(dnp no)
-		(property "Reference" "D64"
+		(property "Reference" "D54"
 			(at 148.5900 38.1000 0)
 			(effects (font (size 1.27 1.27)) (justify left))
@@
 		(pin "2")
 		(instances
-			(project "calcumaker-main"
-				(path "/ca1c0000-0000-4000-8000-00000000ma01/09ef021e-eba5-4a51-ac3b-4585f8d3f3ef"
-					(reference "D64")
+			(project "calcumaker-keyboard"
+				(path "/ca1c0000-0000-4000-8000-00000000eb01/e123962d-af1f-484c-976e-978d59e057ae"
+					(reference "D54")
 					(unit 1)
 				)
@@
 		(on_board yes)
 		(dnp no)
-		(property "Reference" "D65"
+		(property "Reference" "D55"
 			(at 186.6900 38.1000 0)
 			(effects (font (size 1.27 1.27)) (justify left))
@@
 		(pin "2")
 		(instances
-			(project "calcumaker-main"
-				(path "/ca1c0000-0000-4000-8000-00000000ma01/09ef021e-eba5-4a51-ac3b-4585f8d3f3ef"
-					(reference "D65")
+			(project "calcumaker-keyboard"
+				(path "/ca1c0000-0000-4000-8000-00000000eb01/e123962d-af1f-484c-976e-978d59e057ae"
+					(reference "D55")
 					(unit 1)
 				)
@@
 		(on_board yes)
 		(dnp no)
-		(property "Reference" "R9"
+		(property "Reference" "R1"
 			(at 224.7900 38.1000 0)
 			(effects (font (size 1.27 1.27)) (justify left))
@@
 		(pin "2")
 		(instances
-			(project "calcumaker-main"
-				(path "/ca1c0000-0000-4000-8000-00000000ma01/09ef021e-eba5-4a51-ac3b-4585f8d3f3ef"
-					(reference "R9")
+			(project "calcumaker-keyboard"
+				(path "/ca1c0000-0000-4000-8000-00000000eb01/e123962d-af1f-484c-976e-978d59e057ae"
+					(reference "R1")
 					(unit 1)
 				)
@@
 		(on_board yes)
 		(dnp no)
-		(property "Reference" "R10"
+		(property "Reference" "R2"
 			(at 262.8900 38.1000 0)
 			(effects (font (size 1.27 1.27)) (justify left))
@@
 		(pin "2")
 		(instances
-			(project "calcumaker-main"
-				(path "/ca1c0000-0000-4000-8000-00000000ma01/09ef021e-eba5-4a51-ac3b-4585f8d3f3ef"
-					(reference "R10")
+			(project "calcumaker-keyboard"
+				(path "/ca1c0000-0000-4000-8000-00000000eb01/e123962d-af1f-484c-976e-978d59e057ae"
+					(reference "R2")
 					(unit 1)
 				)
@@
 		(on_board yes)
 		(dnp no)
-		(property "Reference" "R11"
+		(property "Reference" "R3"
 			(at 300.9900 38.1000 0)
 			(effects (font (size 1.27 1.27)) (justify left))
@@
 		(pin "2")
 		(instances
-			(project "calcumaker-main"
-				(path "/ca1c0000-0000-4000-8000-00000000ma01/09ef021e-eba5-4a51-ac3b-4585f8d3f3ef"
-					(reference "R11")
+			(project "calcumaker-keyboard"
+				(path "/ca1c0000-0000-4000-8000-00000000eb01/e123962d-af1f-484c-976e-978d59e057ae"
+					(reference "R3")
 					(unit 1)
 				)
@@
 		(on_board yes)
 		(dnp no)
-		(property "Reference" "R12"
+		(property "Reference" "R4"
 			(at 339.0900 38.1000 0)
 			(effects (font (size 1.27 1.27)) (justify left))
@@
 		(pin "2")
 		(instances
-			(project "calcumaker-main"
-				(path "/ca1c0000-0000-4000-8000-00000000ma01/09ef021e-eba5-4a51-ac3b-4585f8d3f3ef"
-					(reference "R12")
+			(project "calcumaker-keyboard"
+				(path "/ca1c0000-0000-4000-8000-00000000eb01/e123962d-af1f-484c-976e-978d59e057ae"
+					(reference "R4")
 					(unit 1)
 				)
@@
 		(on_board yes)
 		(dnp no)
-		(property "Reference" "R13"
+		(property "Reference" "R5"
 			(at 377.1900 38.1000 0)
 			(effects (font (size 1.27 1.27)) (justify left))
@@
 		(pin "2")
 		(instances
-			(project "calcumaker-main"
-				(path "/ca1c0000-0000-4000-8000-00000000ma01/09ef021e-eba5-4a51-ac3b-4585f8d3f3ef"
-					(reference "R13")
-					(unit 1)
-				)
-			)
-		)
-	)
-	(text "Calcumaker 16 main — Annunciator LEDs (DESIGN.md status-line mapping). PLACED, not wired. Five MCU GPIOs (active high), each -> Rn 470R -> LED -> GND: D61 'f' yellow + D62 'g' blue mounted BESIDE the f/g keys; D63 'C' carry, D64 'G' overflow, D65 low-battery along the top edge under the display bezel. 470R @3V3 = ~1.3-2.8mA; adjust per color at bring-up. Firmware: calcumaker-core App drives f/g from keys::Shift, C/G from Calc::carry()/overflow(); LOWBAT from the battery ADC (PSU). Radix/STATUS/errors render in the digits."
+			(project "calcumaker-keyboard"
+				(path "/ca1c0000-0000-4000-8000-00000000eb01/e123962d-af1f-484c-976e-978d59e057ae"
+					(reference "R5")
+					(unit 1)
+				)
+			)
+		)
+	)
+	(text "Calcumaker 16 keyboard — Annunciator LEDs (DESIGN.md status-line mapping). PLACED, not wired. Five drive lines from the ON-BOARD STM32G0 (U1, active high), each -> Rn 470R -> LED -> GND: D51 'f' yellow + D52 'g' blue mounted BESIDE the f/g keys; D53 'C' carry, D54 'G' overflow, D55 low-battery along the top edge under the display bezel. +3V3 feeds the resistors; GND is the return. 470R = ~1.3-2.8mA; adjust per color at bring-up. Firmware: the U575's calcumaker-core App drives f/g from keys::Shift, C/G from Calc::carry()/overflow(), LOWBAT from the battery ADC, and pushes the 5-bit state to the G0 over I2C; the G0 sets the pins. Radix/STATUS/errors render in the 7-seg digits."
 		(exclude_from_sim no)
 		(at 15.00 105.00 0)
@@
 	(sheet_instances
 		(path "/"
-			(page "8")
-		)
-	)
+			(page "3")
+		)
+	)

Commit message: hardware: MCU -> STM32U575RGT6 (LQFP-64) + 4MB QSPI flash; monospace wiring notes
MCU package + external flash
- Swap U1 STM32U575ZGT6 (LQFP-144) -> STM32U575RGT6 (LQFP-64, LCSC C5270980).
  The firmware links at ~323 KB so 1 MB flash is ample (~3x headroom), and with
  the key matrix scanned off-board the LQFP-64 has enough GPIO — smaller/cheaper.
- Correct the flash size everywhere: the STM32 `G` code = 1 MB (not 2 MB; the
  `I` parts are 2 MB). memory.x FLASH 2048K -> 1024K; .cargo runner -> RGTx.
- Add U7 W25Q32JVSSIQ, a 4 MB (32 Mbit) quad-SPI NOR (LCSC C179173, SOIC-8) on
  OCTOSPI1 as a new QSPIFlash sheet (+ R9 CS# pull-up + C26 decoupling) for
  memory-mapped (XIP) constants + state/program storage.
- mcu board 52 -> 55 components / 7 sheets. Docs (DESIGN.md, PARTS.md, READMEs,
  CLAUDE/AGENTS) updated; availability ladder now lists RGT6/VGT6/ZGT6.

Monospace, multi-line schematic wiring notes
- kschgen text_note() now renders notes in a monospace font (Courier New) so
  tables/columns line up; add note_block() + pin_table() helpers.
- Reformat all 14 per-sheet notes into titled, multi-line, aligned blocks —
  connector pinouts as PIN/SIGNAL tables, power/MCU sheets as wiring blocks.

The regenerated schematics carry both changes, so this is one commit. All three
boards regenerate + pass the structure check (mcu 55 / keyboard 119 / display
60, no duplicate refs).

Co-Authored-By: Claude Opus 4.8 (1M context) <noreply@anthropic.com>
Other:
- note added: "ANNUNCIATOR LEDs (DESIGN.md status-line mapping) PLACED, not wired. 5 drive lines from the on-board STM32G0 (active high), each -> Rn 470R -> LED -> GND. +3V3 feeds the resistors; GND returns. D51 f yellow beside the f key D52 g blue beside the g key D53 C red carry ] top edge, under D54 G red overflow ] the display bezel D55 LOWBAT red low-battery 470R = ~1.3-2.8mA (adjust per color at bring-up)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"
- note removed: "Calcumaker 16 keyboard — Annunciator LEDs (DESIGN.md status-line mapping). PLACED, not wired. Five drive lines from the ON-BOARD STM32G0 (U1, active high), each -> Rn 470R -> LED -> GND: D51 'f' yellow + D52 'g' blue mounted BESIDE the f/g keys; D53 'C' carry, D54 'G' overflow, D55 low-battery along the top edge under the display bezel. +3V3 feeds the resistors; GND is the return. 470R = ~1.3-2.8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"
Changed lines of the file:
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@@
 		(instances
 			(project "calcumaker-keyboard"
-				(path "/ca1c0000-0000-4000-8000-00000000eb01/e123962d-af1f-484c-976e-978d59e057ae"
+				(path "/ca1c0000-0000-4000-8000-00000000eb01/4e94bd18-e5fe-49a6-ae02-b46fd6d77075"
 					(reference "D51")
 					(unit 1)
@@
 		(instances
 			(project "calcumaker-keyboard"
-				(path "/ca1c0000-0000-4000-8000-00000000eb01/e123962d-af1f-484c-976e-978d59e057ae"
+				(path "/ca1c0000-0000-4000-8000-00000000eb01/4e94bd18-e5fe-49a6-ae02-b46fd6d77075"
 					(reference "D52")
 					(unit 1)
@@
 		(instances
 			(project "calcumaker-keyboard"
-				(path "/ca1c0000-0000-4000-8000-00000000eb01/e123962d-af1f-484c-976e-978d59e057ae"
+				(path "/ca1c0000-0000-4000-8000-00000000eb01/4e94bd18-e5fe-49a6-ae02-b46fd6d77075"
 					(reference "D53")
 					(unit 1)
@@
 		(instances
 			(project "calcumaker-keyboard"
-				(path "/ca1c0000-0000-4000-8000-00000000eb01/e123962d-af1f-484c-976e-978d59e057ae"
+				(path "/ca1c0000-0000-4000-8000-00000000eb01/4e94bd18-e5fe-49a6-ae02-b46fd6d77075"
 					(reference "D54")
 					(unit 1)
@@
 		(instances
 			(project "calcumaker-keyboard"
-				(path "/ca1c0000-0000-4000-8000-00000000eb01/e123962d-af1f-484c-976e-978d59e057ae"
+				(path "/ca1c0000-0000-4000-8000-00000000eb01/4e94bd18-e5fe-49a6-ae02-b46fd6d77075"
 					(reference "D55")
 					(unit 1)
@@
 		(instances
 			(project "calcumaker-keyboard"
-				(path "/ca1c0000-0000-4000-8000-00000000eb01/e123962d-af1f-484c-976e-978d59e057ae"
+				(path "/ca1c0000-0000-4000-8000-00000000eb01/4e94bd18-e5fe-49a6-ae02-b46fd6d77075"
 					(reference "R1")
 					(unit 1)
@@
 		(instances
 			(project "calcumaker-keyboard"
-				(path "/ca1c0000-0000-4000-8000-00000000eb01/e123962d-af1f-484c-976e-978d59e057ae"
+				(path "/ca1c0000-0000-4000-8000-00000000eb01/4e94bd18-e5fe-49a6-ae02-b46fd6d77075"
 					(reference "R2")
 					(unit 1)
@@
 		(instances
 			(project "calcumaker-keyboard"
-				(path "/ca1c0000-0000-4000-8000-00000000eb01/e123962d-af1f-484c-976e-978d59e057ae"
+				(path "/ca1c0000-0000-4000-8000-00000000eb01/4e94bd18-e5fe-49a6-ae02-b46fd6d77075"
 					(reference "R3")
 					(unit 1)
@@
 		(instances
 			(project "calcumaker-keyboard"
-				(path "/ca1c0000-0000-4000-8000-00000000eb01/e123962d-af1f-484c-976e-978d59e057ae"
+				(path "/ca1c0000-0000-4000-8000-00000000eb01/4e94bd18-e5fe-49a6-ae02-b46fd6d77075"
 					(reference "R4")
 					(unit 1)
@@
 		(instances
 			(project "calcumaker-keyboard"
-				(path "/ca1c0000-0000-4000-8000-00000000eb01/e123962d-af1f-484c-976e-978d59e057ae"
+				(path "/ca1c0000-0000-4000-8000-00000000eb01/4e94bd18-e5fe-49a6-ae02-b46fd6d77075"
 					(reference "R5")
 					(unit 1)
@@
 		)
 	)
-	(text "Calcumaker 16 keyboard — Annunciator LEDs (DESIGN.md status-line mapping). PLACED, not wired. Five drive lines from the ON-BOARD STM32G0 (U1, active high), each -> Rn 470R -> LED -> GND: D51 'f' yellow + D52 'g' blue mounted BESIDE the f/g keys; D53 'C' carry, D54 'G' overflow, D55 low-battery along the top edge under the display bezel. +3V3 feeds the resistors; GND is the return. 470R = ~1.3-2.8mA; adjust per color at bring-up. Firmware: the U575's calcumaker-core App drives f/g from keys::Shift, C/G from Calc::carry()/overflow(), LOWBAT from the battery ADC, and pushes the 5-bit state to the G0 over I2C; the G0 sets the pins. Radix/STATUS/errors render in the 7-seg digits."
+	(text "ANNUNCIATOR LEDs   (DESIGN.md status-line mapping)\nPLACED, not wired.  5 drive lines from the on-board STM32G0 (active high),\neach -> Rn 470R -> LED -> GND.  +3V3 feeds the resistors; GND returns.\n\n  D51  f  yellow    beside the f key\n  D52  g  blue      beside the g key\n  D53  C  red       carry     ] top edge, under\n  D54  G  red       overflow  ] the display bezel\n  D55  LOWBAT red   low-battery\n\n470R = ~1.3-2.8mA (adjust per color at bring-up).\nFW: the U575 App drives f/g from keys::Shift, C/G from Calc carry/overflow,\nLOWBAT from the battery ADC, pushing the 5-bit state to the G0 over I2C.\nRadix / STATUS / errors render in the 7-seg digits."
 		(exclude_from_sim no)
 		(at 15.00 105.00 0)
-		(effects (font (size 1.5 1.5)) (justify left top))
+		(effects (font (face "Courier New") (size 1.27 1.27)) (justify left top))
 	)
 	(sheet_instances
