File: hardware/calcumaker-keyboard/calcumaker-keyboard.kicad_sch (KiCad schematic)
At the start: 0 parts

Commit message: Wire mainboard and keypad schematics and verify expanded nets
Connect hierarchical interfaces, power/control circuits, debug links, matrix and RGB chains. Correct MCU package pins, diode polarity and power configuration; add bypass components and repeatable KiCad netlist/ERC checks. Document pin maps and remaining physical validation.
Connections:
- no-connect marks 0 -> 1
Other:
- sheet Annunciators ports: added ANN_CARRY, ANN_F, ANN_G, ANN_LOWBAT, ANN_OVERFLOW; removed none
- sheet KbdMCU ports: added ANN_CARRY, ANN_F, ANN_G, ANN_LOWBAT, ANN_OVERFLOW, I2C_SCL, I2C_SDA, KB_BOOT0, KB_IRQ, KB_NRST, KB_ROW1, KB_ROW2, KB_ROW3, KB_ROW4, KB_ROW5, LED_EN, LED_RAW, UART_RX, UART_TX; removed none
- sheet MainIF ports: added I2C_SCL, I2C_SDA, KB_BOOT0, KB_IRQ, KB_NRST, UART_RX, UART_TX; removed none
- sheet RGBPower ports: added KB_LED_DATA, LED_EN, LED_RAW; removed none
- note added: "CALCUMAKER 16 / KEYBOARD / 49 switches + 49 RGB LEDs"
- note added: "Columns COL1..10, VLED and GND are shared global nets inside the row/scanner sheets. Rows and serial interfaces cross explicit sheet pins. RGB data is wired in order down the right edge. Row4 is the 9-key variant: COL6 is omitted for the 2U ENTER. Final DOUT is deliberately unused."
- note removed: "Calcumaker 16 - Keyboard (MULTI-CHANNEL). Row1/2/3/5 = four instances of the reusable 10-key sheet key_row.kicad_sch. Row4 = key_row_9.kicad_sch: 9 keys, no switch/diode/RGB at COL6 -- that is the upper half of the 2U ENTER cap (switch lives in Row5/COL6). 49 keys. (MX switch + diode + SK6812MINI-E RGB per key). Shared buses on global nets COL1..COL10 / VLED / GND; each row's ROW line = a hier pi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"
- title: Calcumaker 16 — Keyboard -> Calcumaker 16 / keyboard / calcumaker-keyboard
