File: hardware/calcumaker-matrix/rp2040.kicad_sch (KiCad schematic)
At the start: 22 parts, among them J4 USB-C (BOOTSEL), SW1 BOOTSEL, U1 RP2040, U2 W25Q32JVSSIQ, U3 USBLC6-2SC6, Y1 12MHz

Commit message: Floorplan both display PCBs and verify their schematic nets
Parts:
- added C19: 1uF, Capacitor_SMD:C_0402_1005Metric, symbol Device:C
- added C20, C21, C22, C23: 100nF, Capacitor_SMD:C_0402_1005Metric, symbol Device:C
- added J5: SWD TC2030-NL, Connector:Tag-Connect_TC2030-IDC-NL_2x03_P1.27mm_Vertical, symbol Connector:Conn_ARM_SWD_TagConnect_TC2030-NL
- added R10, R11: 1k, Resistor_SMD:R_0402_1005Metric, symbol Device:R
- added R12: 10k, Resistor_SMD:R_0402_1005Metric, symbol Device:R
- added R8, R9: 5.1k, Resistor_SMD:R_0402_1005Metric, symbol Device:R
- Y1: value 12MHz -> 12MHz 3225 CL10pF (verify BOM); footprint Crystal:Crystal_SMD_3225-2Pin_3.2x2.5mm -> Crystal:Crystal_SMD_3225-4Pin_3.2x2.5mm; symbol Device:Crystal -> Device:Crystal_GND24
Connections:
- net +3V3: now also C19.1, C22.1, C23.1, J5.1 (VCC), R12.1
- net DISP_NRST: now also J5.3 (~{RESET}), R12.2
- net DVDD: now also C20.1, C21.1
- net GND: now also J4.SH (SHIELD), Y1.2 (G), Y1.4 (G), C19.2, C20.2, C21.2, C22.2, C23.2, J5.5 (GND), R8.2, R9.2
- net QSPI_CS: now also R10.1, R11.1; no longer SW1.1
- net SWCLK: now also J5.4 (SWCLK)
- net SWDIO: now also J5.2 (SWDIO)
- net USB_DM_C: now also J4.B7 (D-), U3.4 (I/O2)
- net USB_DP_C: now also J4.B6 (D+), U3.6 (I/O1)
- net XOSC: now also Y1.3; no longer Y1.2
- net USB_CC1: now reaches J4.A5 (CC1)
- net USB_CC1: now also R8.1
- net USB_CC2: now reaches J4.B5 (CC2)
- net USB_CC2: now also R9.1
- new net BOOTSEL_N: R10.2, SW1.1
- new net DISP_BOOT: R11.2
- no-connect marks 0 -> 23
Other:
- note added: "C1..C6: six IOVDD bypasses; C7: flash. C8: VREG_OUT; C19: VREG_IN, both 1uF. C20/C21: DVDD pins 23/50. C22: ADC_AVDD. C23: USB_VDD (shares nearby IOVDD). USB requires module 3V3 from the main board; VBUS is for ESD clamping only, not a power source. BOOTSEL_N and DISP_BOOT are ACTIVE LOW. Main host must assert LOW for matrix boot, and release to high impedance for operation; STM32 display BOOT0 i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"
- note added: "RP2040 / SPI slave / 3 x PIO LED chains / USB programming"
- note removed: "RP2040 MIN-SYSTEM (WIRED) - U1 RP2040 (C2040, QFN-56). PIO drives WS2812. POWER IOVDD/VREG_VIN/USB_VDD/ADC_AVDD -> +3V3 (C1-C6); VREG_VOUT+DVDD = 1.1V core -> C8 1uF; C9/C10 10uF bulk. GND pad + TESTEN -> GND. CLOCK Y1 12MHz (XIN..R1..XOUT), C11/C12 15pF loads. FLASH U2 W25Q32 on QSPI (SD0-3/SCLK/CS); R4 10k CS pull-up; SW1 BOOTSEL pulls CS low. USB U1 D+/D- -> R2/R3 27R -> U3 USBLC6 ESD -> J4 US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"
- title: Calcumaker 16 — RGB Matrix — RP2040 min-system (MCU + QSPI flash + USB BOOTSEL) — wired -> Calcumaker 16 / matrix / rp2040
- moved on the sheet: C1, C10, C11, C12, C2, C3, C4, C5, C6, C7, C8, C9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
